File: RJG/Drums.sch (KiCad schematic (older format))
At the start: 9 parts, among them U101 4520

Commit message: Small improvements
Parts:
- renumbered U101 to U102
Changed lines of the file:
@@
 AR Path="/5F439237" Ref="U?"  Part="1"
 AR Path="/5F425067/5F439237" Ref="U?"  Part="1"
-AR Path="/5F42563C/5F439237" Ref="U101"  Part="1"
-F 0 "U101" H 2200 1417 50  0000 C CNN
+AR Path="/5F42563C/5F439237" Ref="U102"  Part="1"
+F 0 "U102" H 2200 1417 50  0000 C CNN
 F 1 "4520" H 2200 1326 50  0000 C CNN
 F 2 "Package_DIP:DIP-16_W7.62mm_LongPads" H 2200 1050 50  0001 C CNN

Commit message: Schematic done
Other:
- note added: "Simple drum pattern"
Changed lines of the file:
@@
 Text HLabel 850  1150 0    50   Input ~ 0
 Rst
+Text Notes 1850 1500 0    50   ~ 0
+Simple drum pattern
 $EndSCHEMATC

Commit message: First layout fit
Parts:
- added D? (x4): LED, LED_THT:LED_D3.0mm, symbol Device:LED
- added R? (x4): 1k, Resistor_THT:R_Axial_DIN0204_L3.6mm_D1.6mm_P7.62mm_Horizontal, symbol Device:R
Connections:
- net GND: now also D?.1 (K), D?.1 (K), D?.1 (K), D?.1 (K)
- net at C501.1, U102.3 (Q1): now also R?.1
- net at C502.1, U102.4 (Q2): now also R?.1
- net at C503.2, U102.5 (Q3): now also R?.1
- net at C504.2, U102.6 (Q4): now also R?.1
- new net: D?.2 (A), R?.2 (x4)
Other:
- moved on the sheet: C501, C502, C503, C504, R501, R502, R503, R504

Commit message: Layout improvment
Parts:
- D501, D502, D503, D504: renamed from D?; footprint LED_THT:LED_D3.0mm -> LED_SMD:LED_1206_3216Metric_ReverseMount_Hole1.8x2.4mm
- R505, R506, R507, R508: renamed from R?; footprint Resistor_THT:R_Axial_DIN0204_L3.6mm_D1.6mm_P7.62mm_Horizontal -> Resistor_SMD:R_1206_3216Metric_Pad1.42x1.75mm_HandSolder
Changed lines of the file:
@@
 U 1 1 604F6F5E
 P 3150 2500
-F 0 "D?" V 3189 2383 50  0000 R CNN
+AR Path="/604F6F5E" Ref="D?"  Part="1"
+AR Path="/5F42563C/604F6F5E" Ref="D502"  Part="1"
+F 0 "D502" V 3189 2383 50  0000 R CNN
 F 1 "LED" V 3098 2383 50  0000 R CNN
-F 2 "LED_THT:LED_D3.0mm" H 3150 2500 50  0001 C CNN
+F 2 "LED_SMD:LED_1206_3216Metric_ReverseMount_Hole1.8x2.4mm" H 3150 2500 50  0001 C CNN
 F 3 "~" H 3150 2500 50  0001 C CNN
 	1    3150 2500
@@
 U 1 1 604F6F64
 P 3150 2650
-F 0 "#PWR?" H 3150 2400 50  0001 C CNN
+AR Path="/604F6F64" Ref="#PWR?"  Part="1"
+AR Path="/5F42563C/604F6F64" Ref="#PWR0507"  Part="1"
+F 0 "#PWR0507" H 3150 2400 50  0001 C CNN
 F 1 "GND" H 3155 2477 50  0000 C CNN
 F 2 "" H 3150 2650 50  0001 C CNN
@@
 U 1 1 604F6F71
 P 3500 2500
-F 0 "D?" V 3539 2383 50  0000 R CNN
+AR Path="/604F6F71" Ref="D?"  Part="1"
+AR Path="/5F42563C/604F6F71" Ref="D503"  Part="1"
+F 0 "D503" V 3539 2383 50  0000 R CNN
 F 1 "LED" V 3448 2383 50  0000 R CNN
-F 2 "LED_THT:LED_D3.0mm" H 3500 2500 50  0001 C CNN
+F 2 "LED_SMD:LED_1206_3216Metric_ReverseMount_Hole1.8x2.4mm" H 3500 2500 50  0001 C CNN
 F 3 "~" H 3500 2500 50  0001 C CNN
 	1    3500 2500
@@
 U 1 1 604F6F77
 P 3500 2650
-F 0 "#PWR?" H 3500 2400 50  0001 C CNN
+AR Path="/604F6F77" Ref="#PWR?"  Part="1"
+AR Path="/5F42563C/604F6F77" Ref="#PWR0508"  Part="1"
+F 0 "#PWR0508" H 3500 2400 50  0001 C CNN
 F 1 "GND" H 3505 2477 50  0000 C CNN
 F 2 "" H 3500 2650 50  0001 C CNN
@@
 U 1 1 604F6F84
 P 3850 2500
-F 0 "D?" V 3889 2383 50  0000 R CNN
+AR Path="/604F6F84" Ref="D?"  Part="1"
+AR Path="/5F42563C/604F6F84" Ref="D504"  Part="1"
+F 0 "D504" V 3889 2383 50  0000 R CNN
 F 1 "LED" V 3798 2383 50  0000 R CNN
-F 2 "LED_THT:LED_D3.0mm" H 3850 2500 50  0001 C CNN
+F 2 "LED_SMD:LED_1206_3216Metric_ReverseMount_Hole1.8x2.4mm" H 3850 2500 50  0001 C CNN
 F 3 "~" H 3850 2500 50  0001 C CNN
 	1    3850 2500
@@
 U 1 1 604F6F8A
 P 3850 2650
-F 0 "#PWR?" H 3850 2400 50  0001 C CNN
+AR Path="/604F6F8A" Ref="#PWR?"  Part="1"
+AR Path="/5F42563C/604F6F8A" Ref="#PWR0509"  Part="1"
+F 0 "#PWR0509" H 3850 2400 50  0001 C CNN
 F 1 "GND" H 3855 2477 50  0000 C CNN
 F 2 "" H 3850 2650 50  0001 C CNN
@@
 U 1 1 604F6F97
 P 2800 2500
-F 0 "D?" V 2839 2383 50  0000 R CNN
+AR Path="/604F6F97" Ref="D?"  Part="1"
+AR Path="/5F42563C/604F6F97" Ref="D501"  Part="1"
+F 0 "D501" V 2839 2383 50  0000 R CNN
 F 1 "LED" V 2748 2383 50  0000 R CNN
-F 2 "LED_THT:LED_D3.0mm" H 2800 2500 50  0001 C CNN
+F 2 "LED_SMD:LED_1206_3216Metric_ReverseMount_Hole1.8x2.4mm" H 2800 2500 50  0001 C CNN
 F 3 "~" H 2800 2500 50  0001 C CNN
 	1    2800 2500
@@
 U 1 1 604F6F9D
 P 2800 2650
-F 0 "#PWR?" H 2800 2400 50  0001 C CNN
+AR Path="/604F6F9D" Ref="#PWR?"  Part="1"
+AR Path="/5F42563C/604F6F9D" Ref="#PWR0502"  Part="1"
+F 0 "#PWR0502" H 2800 2400 50  0001 C CNN
 F 1 "GND" H 2805 2477 50  0000 C CNN
 F 2 "" H 2800 2650 50  0001 C CNN
@@
 P 2800 2200
 AR Path="/604F6FA3" Ref="R?"  Part="1"
-AR Path="/5F42563C/604F6FA3" Ref="R?"  Part="1"
-F 0 "R?" H 2870 2246 50  0000 L CNN
+AR Path="/5F42563C/604F6FA3" Ref="R505"  Part="1"
+F 0 "R505" H 2870 2246 50  0000 L CNN
 F 1 "1k" V 2800 2150 50  0000 L CNN
-F 2 "Resistor_THT:R_Axial_DIN0204_L3.6mm_D1.6mm_P7.62mm_Horizontal" V 2730 2200 50  0001 C CNN
+F 2 "Resistor_SMD:R_1206_3216Metric_Pad1.42x1.75mm_HandSolder" V 2730 2200 50  0001 C CNN
 F 3 "~" H 2800 2200 50  0001 C CNN
 	1    2800 2200
@@
 P 3150 2200
 AR Path="/604FE354" Ref="R?"  Part="1"
-AR Path="/5F42563C/604FE354" Ref="R?"  Part="1"
-F 0 "R?" H 3220 2246 50  0000 L CNN
+AR Path="/5F42563C/604FE354" Ref="R506"  Part="1"
+F 0 "R506" H 3220 2246 50  0000 L CNN
 F 1 "1k" V 3150 2150 50  0000 L CNN
-F 2 "Resistor_THT:R_Axial_DIN0204_L3.6mm_D1.6mm_P7.62mm_Horizontal" V 3080 2200 50  0001 C CNN
+F 2 "Resistor_SMD:R_1206_3216Metric_Pad1.42x1.75mm_HandSolder" V 3080 2200 50  0001 C CNN
 F 3 "~" H 3150 2200 50  0001 C CNN
 	1    3150 2200
@@
 P 3500 2200
 AR Path="/604FE71B" Ref="R?"  Part="1"
-AR Path="/5F42563C/604FE71B" Ref="R?"  Part="1"
-F 0 "R?" H 3570 2246 50  0000 L CNN
+AR Path="/5F42563C/604FE71B" Ref="R507"  Part="1"
+F 0 "R507" H 3570 2246 50  0000 L CNN
 F 1 "1k" V 3500 2150 50  0000 L CNN
-F 2 "Resistor_THT:R_Axial_DIN0204_L3.6mm_D1.6mm_P7.62mm_Horizontal" V 3430 2200 50  0001 C CNN
+F 2 "Resistor_SMD:R_1206_3216Metric_Pad1.42x1.75mm_HandSolder" V 3430 2200 50  0001 C CNN
 F 3 "~" H 3500 2200 50  0001 C CNN
 	1    3500 2200
@@
 P 3850 2200
 AR Path="/604FEA36" Ref="R?"  Part="1"
-AR Path="/5F42563C/604FEA36" Ref="R?"  Part="1"
-F 0 "R?" H 3920 2246 50  0000 L CNN
+AR Path="/5F42563C/604FEA36" Ref="R508"  Part="1"
+F 0 "R508" H 3920 2246 50  0000 L CNN
 F 1 "1k" V 3850 2150 50  0000 L CNN
-F 2 "Resistor_THT:R_Axial_DIN0204_L3.6mm_D1.6mm_P7.62mm_Horizontal" V 3780 2200 50  0001 C CNN
+F 2 "Resistor_SMD:R_1206_3216Metric_Pad1.42x1.75mm_HandSolder" V 3780 2200 50  0001 C CNN
 F 3 "~" H 3850 2200 50  0001 C CNN
 	1    3850 2200

Commit message: Minor tweaks; added BOM
Parts:
- U102: value 4520 -> 74HCT4520
Changed lines of the file:
@@
 AR Path="/5F42563C/5F439237" Ref="U102"  Part="1"
 F 0 "U102" H 2200 1417 50  0000 C CNN
-F 1 "4520" H 2200 1326 50  0000 C CNN
+F 1 "74HCT4520" H 2200 1326 50  0000 C CNN
 F 2 "Package_DIP:DIP-16_W7.62mm_LongPads" H 2200 1050 50  0001 C CNN
 F 3 "http://www.intersil.com/content/dam/Intersil/documents/cd45/cd4518bms-20bms.pdf" H 2200 1050 50  0001 C CNN
