File: RJG/Random Jazz Generator.sch (KiCad schematic (older format))
At the start: 36 parts, among them J101 EuroPower, J102 CV, J103 RND, J104 Gate, J105 Trig1, J106 Trig2, J107 Clock, J108 Trig3, J109 Trig4, Q101 BC557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

Commit message: Finished graphics
Parts:
- added D102, D103, D104, D105: LED, LED_SMD:LED_1206_3216Metric_Castellated, symbol Device:LED
- added H104: Mounting_Holes, Kosmo_panel:Kosmo_Panel_Dual_Mounting_Holes, symbol Kosmo:Mounting_Holes
- added R102, R103, R104, R113: 1k, Resistor_SMD:R_1206_3216Metric_Pad1.42x1.75mm_HandSolder, symbol Device:R
Connections:
- net +5V: now also R102.1, R103.1, R104.1, R113.1
- net GND: now also D102.1 (K), D103.1 (K), D104.1 (K), D105.1 (K), H104.1
- new net: D102.2 (A), R102.2
- new net: D103.2 (A), R103.2
- new net: D104.2 (A), R104.2
- new net: D105.2 (A), R113.2
Other:
- moved on the sheet: H101, H102, H103

Commit message: Minor tweaks; added BOM
Parts:
- U102: value 4520 -> 74HCT4520
Changed lines of the file:
@@
 AR Path="/5F642777" Ref="U102"  Part="3"
 AR Path="/5F425067/5F642777" Ref="U?"  Part="3"
-F 0 "U102" H 1780 2746 50  0000 L CNN
-F 1 "4520" H 1780 2655 50  0000 L CNN
+F 0 "U102" H 1550 3150 50  0000 L CNN
+F 1 "74HCT4520" H 1550 3050 50  0000 L CNN
 F 2 "Package_DIP:DIP-16_W7.62mm_LongPads" H 1550 2700 50  0001 C CNN
 F 3 "http://www.intersil.com/content/dam/Intersil/documents/cd45/cd4518bms-20bms.pdf" H 1550 2700 50  0001 C CNN
@@
 $EndComp
 $Comp
-L power:GND #PWR?
+L power:GND #PWR0151
 U 1 1 60F6C69A
 P 1850 7200
-AR Path="/60F6C69A" Ref="#PWR?"  Part="1"
+AR Path="/60F6C69A" Ref="#PWR0151"  Part="1"
 AR Path="/5F345A0C/60F6C69A" Ref="#PWR?"  Part="1"
-F 0 "#PWR?" H 1850 6950 50  0001 C CNN
+F 0 "#PWR0151" H 1850 6950 50  0001 C CNN
 F 1 "GND" H 1855 7027 50  0000 C CNN
 F 2 "" H 1850 7200 50  0001 C CNN
