File: RJG/Random Jazz Generator.sch (KiCad schematic (older format))
At the start: 45 parts, among them J101 EuroPower, J102 CV, J103 RND, J104 Gate, J105 Trig1, J106 Trig2, J107 Clock, J108 Trig3, J109 Trig4, Q101 BC557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

Commit message: Small tweak
Parts:
- LOGO1: symbol Graphic:Logo_Open_Hardware_Small -> logo:Logo_telec
Changed lines of the file:
@@
 Gate
 $Comp
-L Graphic:Logo_Open_Hardware_Small LOGO1
+L logo:Logo_telec LOGO1
 U 1 1 60E67084
 P 3350 6950

Commit message: RJG done !
Parts:
- added D106: 1N4148, Diode_THT:D_DO-35_SOD27_P7.62mm_Horizontal, symbol Diode:1N4148
Connections:
- net GND: now also D106.2 (A)
- net at Q102.2 (B), R110.1: now also D106.1 (K)
Other:
- moved on the sheet: J107, R110
Changed lines of the file:
@@
 L Connector:AudioJack3_Switch J107
 U 1 1 5F0BD040
-P 3350 5200
-F 0 "J107" H 3332 5625 50  0000 C CNN
-F 1 "Clock" H 3332 5534 50  0000 C CNN
-F 2 "telec:JackHole" H 3350 5200 50  0001 C CNN
-F 3 "~" H 3350 5200 50  0001 C CNN
-	1    3350 5200
+P 3150 5200
+F 0 "J107" H 3132 5625 50  0000 C CNN
+F 1 "Clock" H 3132 5534 50  0000 C CNN
+F 2 "telec:JackHole" H 3150 5200 50  0001 C CNN
+F 3 "~" H 3150 5200 50  0001 C CNN
+	1    3150 5200
 	1    0    0    -1
 $EndComp
@@
 	0    1    1    0
 $EndComp
-NoConn ~ 3550 5300
-NoConn ~ 3550 5200
-NoConn ~ 3550 5100
+NoConn ~ 3350 5300
+NoConn ~ 3350 5200
+NoConn ~ 3350 5100
 $Comp
 L power:GND #PWR0123
 U 1 1 5F63005B
-P 3550 5000
-F 0 "#PWR0123" H 3550 4750 50  0001 C CNN
-F 1 "GND" V 3555 4872 50  0000 R CNN
-F 2 "" H 3550 5000 50  0001 C CNN
-F 3 "" H 3550 5000 50  0001 C CNN
-	1    3550 5000
+P 3350 5000
+F 0 "#PWR0123" H 3350 4750 50  0001 C CNN
+F 1 "GND" V 3355 4872 50  0000 R CNN
+F 2 "" H 3350 5000 50  0001 C CNN
+F 3 "" H 3350 5000 50  0001 C CNN
+	1    3350 5000
 	0    -1   1    0
 $EndComp
@@
 L power:GND #PWR0125
 U 1 1 5F6304F3
-P 3550 5500
-F 0 "#PWR0125" H 3550 5250 50  0001 C CNN
-F 1 "GND" V 3555 5372 50  0000 R CNN
-F 2 "" H 3550 5500 50  0001 C CNN
-F 3 "" H 3550 5500 50  0001 C CNN
-	1    3550 5500
+P 3350 5500
+F 0 "#PWR0125" H 3350 5250 50  0001 C CNN
+F 1 "GND" V 3355 5372 50  0000 R CNN
+F 2 "" H 3350 5500 50  0001 C CNN
+F 3 "" H 3350 5500 50  0001 C CNN
+	1    3350 5500
 	0    -1   1    0
 $EndComp
@@
 L power:GND #PWR0135
 U 1 1 603B9D4E
-P 4450 5600
+P 4450 5750
 AR Path="/603B9D4E" Ref="#PWR0135"  Part="1"
 AR Path="/5F42563C/603B9D4E" Ref="#PWR?"  Part="1"
 AR Path="/5F425067/603B9D4E" Ref="#PWR?"  Part="1"
-F 0 "#PWR0135" H 4450 5350 50  0001 C CNN
-F 1 "GND" H 4455 5427 50  0000 C CNN
-F 2 "" H 4450 5600 50  0001 C CNN
-F 3 "" H 4450 5600 50  0001 C CNN
-	1    4450 5600
+F 0 "#PWR0135" H 4450 5500 50  0001 C CNN
+F 1 "GND" H 4455 5577 50  0000 C CNN
+F 2 "" H 4450 5750 50  0001 C CNN
+F 3 "" H 4450 5750 50  0001 C CNN
+	1    4450 5750
 	-1   0    0    -1
 $EndComp
@@
 L Device:R R110
 U 1 1 603B9D54
-P 4000 5400
+P 3800 5400
 AR Path="/603B9D54" Ref="R110"  Part="1"
 AR Path="/5F42563C/603B9D54" Ref="R?"  Part="1"
 AR Path="/5F425067/603B9D54" Ref="R?"  Part="1"
-F 0 "R110" V 3900 5300 50  0000 L CNN
-F 1 "100k" V 4000 5300 50  0000 L CNN
-F 2 "Resistor_THT:R_Axial_DIN0204_L3.6mm_D1.6mm_P7.62mm_Horizontal" V 3930 5400 50  0001 C CNN
-F 3 "~" H 4000 5400 50  0001 C CNN
-	1    4000 5400
+F 0 "R110" V 3700 5300 50  0000 L CNN
+F 1 "100k" V 3800 5300 50  0000 L CNN
+F 2 "Resistor_THT:R_Axial_DIN0204_L3.6mm_D1.6mm_P7.62mm_Horizontal" V 3730 5400 50  0001 C CNN
+F 3 "~" H 3800 5400 50  0001 C CNN
+	1    3800 5400
 	0    1    -1   0
 $EndComp
@@
 L power:GND #PWR0136
 U 1 1 603C03D3
-P 5250 5600
+P 5250 5750
 AR Path="/603C03D3" Ref="#PWR0136"  Part="1"
 AR Path="/5F42563C/603C03D3" Ref="#PWR?"  Part="1"
 AR Path="/5F425067/603C03D3" Ref="#PWR?"  Part="1"
-F 0 "#PWR0136" H 5250 5350 50  0001 C CNN
-F 1 "GND" H 5255 5427 50  0000 C CNN
-F 2 "" H 5250 5600 50  0001 C CNN
-F 3 "" H 5250 5600 50  0001 C CNN
-	1    5250 5600
+F 0 "#PWR0136" H 5250 5500 50  0001 C CNN
+F 1 "GND" H 5255 5577 50  0000 C CNN
+F 2 "" H 5250 5750 50  0001 C CNN
+F 3 "" H 5250 5750 50  0001 C CNN
+	1    5250 5750
 	-1   0    0    -1
 $EndComp
@@
 Connection ~ 6050 5400
 Wire Wire Line
-	3850 5400 3550 5400
+	3650 5400 3350 5400
 $Comp
 L Transistor_BJT:BC557 Q101
@@
 	5250 5150 5250 5200
 Wire Wire Line
-	5250 5550 5250 5600
+	5250 5550 5250 5750
 $Comp
 L Device:R R109
@@
 	-1   0    0    -1
 $EndComp
+Wire Wire Line
+	3950 5400 4050 5400
+$Comp
+L Diode:1N4148 D106
+U 1 1 63804C31
+P 4050 5600
+F 0 "D106" V 4004 5679 50  0000 L CNN
+F 1 "1N4148" V 4095 5679 50  0000 L CNN
+F 2 "Diode_THT:D_DO-35_SOD27_P7.62mm_Horizontal" H 4050 5425 50  0001 C CNN
+F 3 "https://assets.nexperia.com/documents/data-sheet/1N4148_1N4448.pdf" H 4050 5600 50  0001 C CNN
+	1    4050 5600
+	0    1    1    0
+$EndComp
+$Comp
+L power:GND #PWR?
+U 1 1 63807A13
+P 4050 5750
+AR Path="/63807A13" Ref="#PWR?"  Part="1"
+AR Path="/5F42563C/63807A13" Ref="#PWR?"  Part="1"
+AR Path="/5F425067/63807A13" Ref="#PWR?"  Part="1"
+F 0 "#PWR?" H 4050 5500 50  0001 C CNN
+F 1 "GND" H 4055 5577 50  0000 C CNN
+F 2 "" H 4050 5750 50  0001 C CNN
+F 3 "" H 4050 5750 50  0001 C CNN
+	1    4050 5750
+	-1   0    0    -1
+$EndComp
+Wire Wire Line
+	4050 5450 4050 5400
+Connection ~ 4050 5400
+Wire Wire Line
+	4050 5400 4150 5400
+Wire Wire Line
+	4450 5600 4450 5750
 Wire Bus Line
 	6100 2050 6100 2800

Commit message: fix stuffs
Parts:
- added Q?: BC557, Package_TO_SOT_THT:TO-92_Inline_Wide, symbol Transistor_BJT:BC557
- added R?: 10k, Resistor_THT:R_Axial_DIN0204_L3.6mm_D1.6mm_P7.62mm_Horizontal, symbol Device:R
Connections:
- net +5V: now also Q?.3 (E); no longer R102.1, R103.1, R104.1, R113.1
- new net: Q?.1 (C), R102.1, R103.1, R104.1, R113.1
- new net: Q?.2 (B), R?.2
- new net ~Chorus~\Impro: R?.1
Other:
- moved on the sheet: C105, D102, D103, D104, D105, J104, R102, R103, R104, R107, R112, R113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
