File: RJG/Duration.sch (KiCad schematic (older format))
At the start: 29 parts, among them Q401 BC547, Q402 BC547, SW401 Duration Length, SW402 Reload, U102 74HCT4520, U401 74HCT4520, U402 74HCT74, U403 74HCT85, U404 74HCT157, U405 SST39SF010, U406 74HCT173

Commit message: fix stuffs
Parts:
- added C?: 2n, Capacitor_THT:C_Disc_D7.0mm_W2.5mm_P5.00mm, symbol Device:C
- R401, R403: value 100k -> 10k
- R404: value 100k -> 47k
Connections:
- net +5V: now also R401.1, R403.1; no longer R401.2, R403.2
- net GND: now also C?.1
- net Gate: now also C?.2
- net at Q402.1 (C), U402.1 (~R): now also R403.2; no longer R403.1
- net at Q401.1 (C), U402.3 (C): now also R401.2; no longer R401.1
Other:
- note added: "Duration pattern\ncounter"
- note added: "Note step\ncounter"
- note removed: "Duration pattern counter"
- note removed: "Note step counter"
- moved on the sheet: D401, D402, R404
