File: RJG/RandomByteGenerator.sch (KiCad schematic (older format))
At the start: 12 parts, among them Q201 BC547, Q202 BC547, U201 74LS04, U202 74LS595

Commit message: Small improvements
Parts:
- added C201, C202: 100n, Capacitor_THT:C_Disc_D7.0mm_W2.5mm_P5.00mm, symbol Device:C
- renumbered C201 to C203, C202 to C204, C203 to C205
Connections:
- net +5V: now also C201.2, C202.2
- net GND: now also C201.1, C202.1
- net Rb: no longer R202.2
- net at C204.1, U201.11: now also R202.1
- net at U201.10, U201.9: now also R202.2; no longer R202.1
Other:
- moved on the sheet: C203, C204, C205, Q201, Q202, R201, R202, R203, R204, R205, U201A, U201B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

Commit message: Schematic done
Other:
- note added: "Clock from spare components"
- note added: "Latch must be eight times\nslower than Fclk\n=> <10Hz"
- note added: "Random bit generator"
- note added: "Random bytes"
Changed lines of the file:
@@
 Wire Wire Line
 	4550 2700 3750 2700
-Text Notes 6250 1650 0    50   ~ 0
+Text Notes 6400 1800 0    50   ~ 0
 Untested
-Text Notes 6250 2600 0    50   ~ 0
+Text Notes 6450 2750 0    50   ~ 0
 Untested
 $Comp
@@
 Wire Bus Line
 	4650 3000 4650 3800
+Text Notes 5900 1650 0    50   ~ 0
+Random bit generator
+Text Notes 5800 2600 0    50   ~ 0
+Clock from spare components
+Text Notes 2250 3500 0    50   ~ 0
+Latch must be eight times\nslower than Fclk\n=> <10Hz
+Text Notes 5250 3150 0    50   ~ 0
+Random bytes
 $EndSCHEMATC

Commit message: Minor tweaks; added BOM
Parts:
- U201: value 74LS04 -> 74HCT04
- U202: value 74LS595 -> 74ACHT595
Changed lines of the file:
@@
 P 4150 2200
 F 0 "U201" H 4150 2517 50  0000 C CNN
-F 1 "74LS04" H 4150 2426 50  0000 C CNN
+F 1 "74HCT04" H 4150 2426 50  0000 C CNN
 F 2 "Package_DIP:DIP-14_W7.62mm_LongPads" H 4150 2200 50  0001 C CNN
 F 3 "http://www.ti.com/lit/gpn/sn74LS04" H 4150 2200 50  0001 C CNN
@@
 P 4950 2200
 F 0 "U201" H 4950 2517 50  0000 C CNN
-F 1 "74LS04" H 4950 2426 50  0000 C CNN
+F 1 "74HCT04" H 4950 2426 50  0000 C CNN
 F 2 "Package_DIP:DIP-14_W7.62mm_LongPads" H 4950 2200 50  0001 C CNN
 F 3 "http://www.ti.com/lit/gpn/sn74LS04" H 4950 2200 50  0001 C CNN
 	2    4950 2200
-	1    0    0    -1
-$EndComp
-$Comp
-L 74xx:74LS04 U201
-U 3 1 5F3626E8
-P 5750 2200
-F 0 "U201" H 5750 2517 50  0000 C CNN
-F 1 "74LS04" H 5750 2426 50  0000 C CNN
-F 2 "Package_DIP:DIP-14_W7.62mm_LongPads" H 5750 2200 50  0001 C CNN
-F 3 "http://www.ti.com/lit/gpn/sn74LS04" H 5750 2200 50  0001 C CNN
-	3    5750 2200
 	1    0    0    -1
 $EndComp
@@
 $Comp
 L 74xx:74LS04 U201
-U 4 1 5F3A371B
-P 5750 1350
-F 0 "U201" H 5750 1667 50  0000 C CNN
-F 1 "74LS04" H 5750 1576 50  0000 C CNN
-F 2 "Package_DIP:DIP-14_W7.62mm_LongPads" H 5750 1350 50  0001 C CNN
-F 3 "http://www.ti.com/lit/gpn/sn74LS04" H 5750 1350 50  0001 C CNN
-	4    5750 1350
-	1    0    0    -1
-$EndComp
-$Comp
-L 74xx:74LS04 U201
-U 5 1 5F3A653F
-P 5050 1350
-F 0 "U201" H 5050 1667 50  0000 C CNN
-F 1 "74LS04" H 5050 1576 50  0000 C CNN
-F 2 "Package_DIP:DIP-14_W7.62mm_LongPads" H 5050 1350 50  0001 C CNN
-F 3 "http://www.ti.com/lit/gpn/sn74LS04" H 5050 1350 50  0001 C CNN
-	5    5050 1350
-	1    0    0    -1
-$EndComp
-$Comp
-L 74xx:74LS04 U201
-U 6 1 5F3A7507
-P 3950 1350
-F 0 "U201" H 3950 1667 50  0000 C CNN
-F 1 "74LS04" H 3950 1576 50  0000 C CNN
-F 2 "Package_DIP:DIP-14_W7.62mm_LongPads" H 3950 1350 50  0001 C CNN
-F 3 "http://www.ti.com/lit/gpn/sn74LS04" H 3950 1350 50  0001 C CNN
-	6    3950 1350
-	1    0    0    -1
-$EndComp
-$Comp
-L 74xx:74LS04 U201
 U 7 1 5F3A843F
 P 1600 1250
-F 0 "U201" H 1830 1296 50  0000 L CNN
-F 1 "74LS04" H 1830 1205 50  0000 L CNN
+F 0 "U201" H 1600 1700 50  0000 L CNN
+F 1 "74HCT04" H 1600 1600 50  0000 L CNN
 F 2 "Package_DIP:DIP-14_W7.62mm_LongPads" H 1600 1250 50  0001 C CNN
 F 3 "http://www.ti.com/lit/gpn/sn74LS04" H 1600 1250 50  0001 C CNN
@@
 P 4000 3600
 F 0 "U202" H 4150 4250 50  0000 C CNN
-F 1 "74LS595" H 4200 4150 50  0000 C CNN
+F 1 "74ACHT595" H 4200 4150 50  0000 C CNN
 F 2 "Package_DIP:DIP-16_W7.62mm_LongPads" H 4000 3600 50  0001 C CNN
 F 3 "http://www.ti.com/lit/gpn/sn74ls595" H 4000 3600 50  0001 C CNN
@@
 Text Notes 5250 3150 0    50   ~ 0
 Random bytes
+$Comp
+L 74xx:74LS04 U201
+U 6 1 5F3A7507
+P 3950 1350
+F 0 "U201" H 3950 1667 50  0000 C CNN
+F 1 "74HCT04" H 3950 1576 50  0000 C CNN
+F 2 "Package_DIP:DIP-14_W7.62mm_LongPads" H 3950 1350 50  0001 C CNN
+F 3 "http://www.ti.com/lit/gpn/sn74LS04" H 3950 1350 50  0001 C CNN
+	6    3950 1350
+	1    0    0    -1
+$EndComp
+$Comp
+L 74xx:74LS04 U201
+U 5 1 5F3A653F
+P 5050 1350
+F 0 "U201" H 5050 1667 50  0000 C CNN
+F 1 "74HCT04" H 5050 1576 50  0000 C CNN
+F 2 "Package_DIP:DIP-14_W7.62mm_LongPads" H 5050 1350 50  0001 C CNN
+F 3 "http://www.ti.com/lit/gpn/sn74LS04" H 5050 1350 50  0001 C CNN
+	5    5050 1350
+	1    0    0    -1
+$EndComp
+$Comp
+L 74xx:74LS04 U201
+U 4 1 5F3A371B
+P 5750 1350
+F 0 "U201" H 5750 1667 50  0000 C CNN
+F 1 "74HCT04" H 5750 1576 50  0000 C CNN
+F 2 "Package_DIP:DIP-14_W7.62mm_LongPads" H 5750 1350 50  0001 C CNN
+F 3 "http://www.ti.com/lit/gpn/sn74LS04" H 5750 1350 50  0001 C CNN
+	4    5750 1350
+	1    0    0    -1
+$EndComp
+$Comp
+L 74xx:74LS04 U201
+U 3 1 5F3626E8
+P 5750 2200
+F 0 "U201" H 5750 2517 50  0000 C CNN
+F 1 "74HCT04" H 5750 2426 50  0000 C CNN
+F 2 "Package_DIP:DIP-14_W7.62mm_LongPads" H 5750 2200 50  0001 C CNN
+F 3 "http://www.ti.com/lit/gpn/sn74LS04" H 5750 2200 50  0001 C CNN
+	3    5750 2200
+	1    0    0    -1
+$EndComp
 $EndSCHEMATC

Commit message: fix stuffs
Parts:
- C205: value 220n -> 100n
Other:
- note added: "150Hz"
- note added: "Tested - OK"
- note removed: "Untested"
Changed lines of the file:
@@
 AR Path="/5F345A0C/5F3D3D6C" Ref="C205"  Part="1"
 F 0 "C205" V 5500 2450 50  0000 C CNN
-F 1 "220n" V 5600 2450 50  0000 C CNN
+F 1 "100n" V 5600 2450 50  0000 C CNN
 F 2 "Capacitor_THT:C_Disc_D7.0mm_W2.5mm_P5.00mm" H 5388 2300 50  0001 C CNN
 F 3 "~" H 5350 2450 50  0001 C CNN
@@
 	4550 2700 3750 2700
 Text Notes 6400 1800 0    50   ~ 0
-Untested
+Tested - OK
 Text Notes 6450 2750 0    50   ~ 0
-Untested
+Tested - OK
 $Comp
 L Device:C C?
@@
 	1    0    0    -1
 $EndComp
-Wire Bus Line
-	4650 3000 4650 3800
 Text Notes 5900 1650 0    50   ~ 0
 Random bit generator
@@
 	1    0    0    -1
 $EndComp
+Text Notes 6100 2300 0    50   ~ 0
+150Hz
+Wire Bus Line
+	4650 3000 4650 3800
 $EndSCHEMATC
