File: VCA/VCA.kicad_pcb (KiCad board)
At the start: 2 copper layers, 40 x 200 mm, 55 parts, among them J1 EuroPower, J2 CV1, J3 IN1, J4 OUT1, J5 CV2, J6 IN2, J7 OUT2, U1 LM13700, U2 TL082, U3 TL082, U4 TL082, U5 TL082

Commit message: VCA done !
Parts:
- removed the D5 at (61.2, 106.2)
- removed the R11 at (60.8, 118.0)
- removed the R12 at (56.2, 99.8)
- removed the R13 at (60.8, 112.0)
- added D1: LED, LED_SMD:LED_1206_3216Metric_ReverseMount_Hole1.8x2.4mm, B.Cu at (33.9, 70.3)
- added D2: LED, LED_SMD:LED_1206_3216Metric_ReverseMount_Hole1.8x2.4mm, B.Cu at (37.0, 70.3)
- added R15: 2k2, Resistor_SMD:R_1206_3216Metric_Pad1.42x1.75mm_HandSolder, B.Cu at (33.9, 163.9)
- added R16: 2k2, Resistor_SMD:R_1206_3216Metric_Pad1.42x1.75mm_HandSolder, B.Cu at (37.1, 163.9)
- added R24: 1k5, Resistor_SMD:R_1206_3216Metric_Pad1.42x1.75mm_HandSolder, B.Cu at (33.1, 115.2)
- added R6: 47k, Resistor_SMD:R_1206_3216Metric_Pad1.42x1.75mm_HandSolder, F.Cu at (32.1, 56.0)
- D3, D4: footprint LED_SMD:LED_1206_3216Metric_Castellated -> LED_SMD:LED_1206_3216Metric_ReverseMount_Hole1.8x2.4mm; moved to B.Cu
- D5: renamed from D1; moved to B.Cu
- D6: renamed from D2; moved to B.Cu
- R23: renamed from R10; moved to B.Cu
- R4: value 47k -> 2k2; moved to B.Cu
- R5: renamed from R14; value 1k -> 2k2; moved to B.Cu
- RV3, RV6: footprint Potentiometer_THT:Potentiometer_Bourns_3339P_Vertical -> telec:Potentiometer_P3.81mmx5.12mm_Vertical
- moved D3 61.2 mm to (33.9, 168.8), turned to 270 degrees
- moved D4 54.4 mm to (37.1, 168.8)
- moved R23 48.7 mm to (14.5, 109.0), turned to 270 degrees
- moved D5 42.9 mm to (14.5, 115.1)
- moved R5 41.1 mm to (37.0, 65.4), turned to 270 degrees
- moved D6 27.6 mm to (33.1, 109.1)
- moved R4 9.56 mm to (33.9, 65.4), turned to 270 degrees
- moved RV6 1.96 mm to (44.5, 127.7)
- moved RV3 1.77 mm to (29.2, 131.5)
- renumbered R8 to R10, R9 to R11, R15 to R12, R16 to R13, R17 to R14, R18 to R17, R19 to R18, R20 to R19, R21 to R20, R22 to R21, R23 to R22, R5 to R7, R6 to R8, R7 to R9
Connections:
- D3 pad 1: GND -> Net-(D3-Pad1)
- D3 pad 2: Net-(D3-Pad2) -> GND
- D6 pad 1: GND -> Net-(D6-Pad1)
- D6 pad 2: Net-(D2-Pad2) (its old number) -> +12V
- R4 pad 1: /CV1 -> /Gain1
- R4 pad 2: Net-(R4-Pad2) -> Net-(D1-Pad1)
- R5 pad 1: /Clk -> /Gain1
- RV2 pad 1: Net-(R4-Pad2) -> Net-(R6-Pad2)
- RV2 pad 2: Net-(R4-Pad2) -> Net-(R6-Pad2)
- U1 pad 8: GND -> Net-(U1-Pad8)
- U1 pad 9: GND -> Net-(U1-Pad9)
- U2 pad 2: Net-(R4-Pad2) -> Net-(R6-Pad2)
Routing:
- net +12V: track 209.8 -> 244.5 mm, vias 9 -> 11
- net Net-(R6-Pad2): track 0.00 -> 30.6 mm
- net Net-(R4-Pad2): track 30.6 -> 0.00 mm
- net /Gain1: track 7.90 -> 15.5 mm, vias 0 -> 1
- net /Gain2: track 11.0 -> 18.6 mm, vias 0 -> 1
- net Net-(D5-Pad2): track 0.00 -> 3.18 mm
- net Net-(D6-Pad1): track 0.00 -> 3.17 mm
- net GND: track 6.13 -> 3.61 mm, vias 29 -> 27
- net Net-(R10-Pad2): track 71.0 -> 68.8 mm
- net Net-(D1-Pad1): track 0.00 -> 1.91 mm
- net Net-(D2-Pad2): track 0.00 -> 1.89 mm
- net Net-(D4-Pad2): track 0.00 -> 1.81 mm
- net Net-(D3-Pad1): track 0.00 -> 1.81 mm
- net Net-(RV6-Pad3): track 12.0 -> 10.2 mm
- net Net-(RV3-Pad1): track 11.1 -> 9.93 mm
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Other:
- board text added: "+12V"
- board text added: "- +"
- board text added: "-12V"
- board text added: "Attenu"
- board text added: "CV"
- board text added: "GAIN"
- board text added: "GND"
- board text added: "IN"
- board text added: "O"
- board text added: "OUT"
- board text added: "Offset 1"
- board text added: "Offset 2"
- board text added: "VCA"
- board text added: "ation"
- board text added: "e"
- board text added: "f"
- board text added: "s"
- board text added: "t"
- board text added: "telec"

Commit message: Added PCB ref stamp and send to prod!
Other:
- board text added: "Design by telec"
- board text added: "PCB ref here:"
- board text removed: "telec"
Changed lines of the file:
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@@
   (general
     (thickness 1.6)
-    (drawings 125)
+    (drawings 154)
     (tracks 360)
     (zones 0)
@@
     )
   )
+  (gr_line (start 12.3 202.8) (end 32.1 202.8) (layer F.SilkS) (width 0.5))
+  (gr_line (start 32.1 180.4) (end 12.3 180.4) (layer F.SilkS) (width 0.5))
+  (gr_line (start 12.3 180.4) (end 12.3 202.8) (layer F.SilkS) (width 0.5))
+  (gr_line (start 12.3 104.4) (end 32.1 104.4) (layer F.SilkS) (width 0.5))
+  (gr_line (start 12.3 82) (end 12.3 104.4) (layer F.SilkS) (width 0.5))
+  (gr_line (start 32.1 82) (end 12.3 82) (layer F.SilkS) (width 0.5))
+  (gr_line (start 40.2 17.8) (end 41.7 12.1) (layer F.SilkS) (width 0.15))
+  (gr_line (start 38.9 12.5) (end 40.2 17.8) (layer F.SilkS) (width 0.15))
+  (gr_line (start 37.9 17.4) (end 38.9 12.5) (layer F.SilkS) (width 0.15))
+  (gr_line (start 36.5 12.9) (end 37.9 17.4) (layer F.SilkS) (width 0.15))
+  (gr_line (start 35.1 17) (end 36.5 12.9) (layer F.SilkS) (width 0.15))
+  (gr_line (start 33.5 13.3) (end 35.1 17) (layer F.SilkS) (width 0.15))
+  (gr_line (start 32.4 16.6) (end 33.5 13.3) (layer F.SilkS) (width 0.15))
+  (gr_line (start 30.9 13.7) (end 32.4 16.6) (layer F.SilkS) (width 0.15))
+  (gr_line (start 29.7 16.2) (end 30.9 13.7) (layer F.SilkS) (width 0.15))
+  (gr_line (start 29 14) (end 29.7 16.2) (layer F.SilkS) (width 0.15))
+  (gr_line (start 27.8 15.9) (end 29 14) (layer F.SilkS) (width 0.15))
+  (gr_line (start 27 14.3) (end 27.8 15.9) (layer F.SilkS) (width 0.15))
+  (gr_line (start 25.9 15.6) (end 27 14.3) (layer F.SilkS) (width 0.15))
+  (gr_line (start 25 14.6) (end 25.9 15.6) (layer F.SilkS) (width 0.15))
+  (gr_line (start 24.1 15.3) (end 25 14.6) (layer F.SilkS) (width 0.15))
+  (gr_line (start 23.8 14.8) (end 24.1 15.3) (layer F.SilkS) (width 0.15))
+  (gr_line (start 22 15) (end 42 18.1) (layer F.SilkS) (width 0.15))
+  (gr_line (start 22 15) (end 42 12) (layer F.SilkS) (width 0.15))
+  (gr_text "PCB ref here:" (at 23.3 48.3) (layer B.SilkS)
+    (effects (font (size 1 1) (thickness 0.15)) (justify mirror))
+  )
+  (gr_line (start 14.9 47.4) (end 14.9 51.7) (layer B.SilkS) (width 0.15))
+  (gr_line (start 29.1 47.4) (end 14.9 47.4) (layer B.SilkS) (width 0.15))
+  (gr_line (start 29.1 51.7) (end 29.1 47.4) (layer B.SilkS) (width 0.15))
+  (gr_line (start 14.9 51.7) (end 29.1 51.7) (layer B.SilkS) (width 0.15))
+  (gr_text "Design by\ntelec" (at 32.4 209.1) (layer B.SilkS)
+    (effects (font (size 1.5 1.5) (thickness 0.3)) (justify mirror))
+  )
   (gr_line (start 51.3 121.7) (end 51.3 116.1) (layer F.SilkS) (width 0.15))
   (gr_line (start 50.5 122.5) (end 51.3 121.7) (layer F.SilkS) (width 0.15))
@@
     (effects (font (size 2 2.8) (thickness 0.5)) (justify left mirror))
   )
-  (gr_text telec (at 32.5 15) (layer F.SilkS)
-    (effects (font (size 2 2) (thickness 0.3)))
-  )
   (gr_poly (pts (xy 52 104.6) (xy 32.1 104.6) (xy 32.1 81.8) (xy 52 81.8)) (layer F.SilkS) (width 0.1))
