File: VCA/VCA.sch (KiCad schematic (older format))
At the start: 55 parts, among them J1 EuroPower, J2 CV1, J3 IN1, J4 OUT1, J5 CV2, J6 IN2, J7 OUT2, U1 LM13700, U2 TL082, U3 TL082, U4 TL082, U5 TL082

Commit message: VCA done !
Parts:
- removed R12, R13: 1k5, Resistor_SMD:R_1206_3216Metric_Pad1.42x1.75mm_HandSolder, symbol Device:R
- added D1: LED, LED_SMD:LED_1206_3216Metric_ReverseMount_Hole1.8x2.4mm, symbol Device:LED
- added R15, R16, R4: 2k2, Resistor_SMD:R_1206_3216Metric_Pad1.42x1.75mm_HandSolder, symbol Device:R
- D3, D4: footprint LED_SMD:LED_1206_3216Metric_Castellated -> LED_SMD:LED_1206_3216Metric_ReverseMount_Hole1.8x2.4mm
- R5: renamed from R14; value 1k -> 2k2
- RV3, RV6: footprint Potentiometer_THT:Potentiometer_Bourns_3339P_Vertical -> telec:Potentiometer_P3.81mmx5.12mm_Vertical
- renumbered D5 to D2, D1 to D5, D2 to D6, R8 to R10, R9 to R11, R15 to R12, R16 to R13, R17 to R14, R18 to R17, R19 to R18, R20 to R19, R21 to R20, R22 to R21, R23 to R22, R10 to R23, R11 to R24, R4 to R6, R5 to R7, R6 to R8, R7 to R9
Connections:
- net Clk is gone; now on net Gain1: R5.1
- net +12V: now also D6.2 (A); no longer R24.1
- net GND: now also D3.2 (A), R24.2, D1.2 (A); no longer D3.1 (K), D6.1 (K), U1.8, U1.9
- net Gain1: now also R4.1
- net Gain2: now also R15.1, R16.1
- net at D4.2 (A): now also R16.2
- new net: D1.1 (K), R4.2
- new net: D3.1 (K), R15.2
- new net: D6.1 (K), R24.1
- no-connect marks 20 -> 22
Other:
- note added: "Front Panel"
- moved on the sheet: C1, C2, D2, D5, D6, R23, R24, R5, U1E

Commit message: updated footprints on VCA
Parts:
- J2, J3, J4, J5, J6, J7: footprint telec:JackHole -> telec:Jack_Hole_Square; symbol Connector:AudioJack3_Switch -> Connector:AudioJack3_SwitchTR
- RV1, RV2, RV4, RV5: footprint Potentiometer_THT:Potentiometer_Piher_T-16L_Single_Vertical_Hole -> telec:Potentiometer_Single_Vertical_Hole
Connections:
- no-connect marks 22 -> 16
Changed lines of the file:
@@
 $EndComp
 $Comp
-L Connector:AudioJack3_Switch J3
+L Connector:AudioJack3_SwitchTR J3
 U 1 1 5F0BD040
 P 3900 2700
 F 0 "J3" H 3882 3125 50  0000 C CNN
 F 1 "IN1" H 3882 3034 50  0000 C CNN
-F 2 "telec:JackHole" H 3900 2700 50  0001 C CNN
+F 2 "telec:Jack_Hole_Square" H 3900 2700 50  0001 C CNN
 F 3 "~" H 3900 2700 50  0001 C CNN
 	1    3900 2700
 	1    0    0    -1
 $EndComp
-NoConn ~ 4100 2600
 NoConn ~ 4100 2700
 NoConn ~ 4100 2800
@@
 L power:GND #PWR030
 U 1 1 5F0D2E83
-P 4200 2550
-F 0 "#PWR030" H 4200 2300 50  0001 C CNN
-F 1 "GND" H 4205 2377 50  0000 C CNN
-F 2 "" H 4200 2550 50  0001 C CNN
-F 3 "" H 4200 2550 50  0001 C CNN
-	1    4200 2550
-	1    0    0    -1
-$EndComp
-Wire Wire Line
-	4100 2500 4200 2500
-Wire Wire Line
-	4200 2500 4200 2550
+P 4200 2650
+F 0 "#PWR030" H 4200 2400 50  0001 C CNN
+F 1 "GND" H 4205 2477 50  0000 C CNN
+F 2 "" H 4200 2650 50  0001 C CNN
+F 3 "" H 4200 2650 50  0001 C CNN
+	1    4200 2650
+	1    0    0    -1
+$EndComp
+Wire Wire Line
+	4100 2600 4200 2600
+Wire Wire Line
+	4200 2600 4200 2650
 $Comp
 L power:GND #PWR034
@@
 F 0 "RV1" V 3800 850 50  0000 C CNN
 F 1 "100k" V 3900 850 50  0000 C CNN
-F 2 "Potentiometer_THT:Potentiometer_Piher_T-16L_Single_Vertical_Hole" H 3900 850 50  0001 C CNN
+F 2 "telec:Potentiometer_Single_Vertical_Hole" H 3900 850 50  0001 C CNN
 F 3 "~" H 3900 850 50  0001 C CNN
 	1    3900 850
@@
 	2150 1250 2150 1350
 $Comp
-L Connector:AudioJack3_Switch J4
+L Connector:AudioJack3_SwitchTR J4
 U 1 1 5F4208DD
 P 9600 2700
 F 0 "J4" H 9582 3125 50  0000 C CNN
 F 1 "OUT1" H 9582 3034 50  0000 C CNN
-F 2 "telec:JackHole" H 9600 2700 50  0001 C CNN
+F 2 "telec:Jack_Hole_Square" H 9600 2700 50  0001 C CNN
 F 3 "~" H 9600 2700 50  0001 C CNN
 	1    9600 2700
@@
 NoConn ~ 9400 2800
 NoConn ~ 9400 2700
-NoConn ~ 9400 2600
 NoConn ~ 9400 3000
 $Comp
 L power:GND #PWR029
 U 1 1 5FBFF003
-P 9400 2500
-F 0 "#PWR029" H 9400 2250 50  0001 C CNN
-F 1 "GND" V 9405 2372 50  0000 R CNN
-F 2 "" H 9400 2500 50  0001 C CNN
-F 3 "" H 9400 2500 50  0001 C CNN
-	1    9400 2500
+P 9400 2600
+F 0 "#PWR029" H 9400 2350 50  0001 C CNN
+F 1 "GND" V 9405 2472 50  0000 R CNN
+F 2 "" H 9400 2600 50  0001 C CNN
+F 3 "" H 9400 2600 50  0001 C CNN
+	1    9400 2600
 	0    1    1    0
 $EndComp
@@
 $EndComp
 $Comp
-L Connector:AudioJack3_Switch J2
+L Connector:AudioJack3_SwitchTR J2
 U 1 1 5F48DF93
 P 3900 1700
 F 0 "J2" H 3882 2125 50  0000 C CNN
 F 1 "CV1" H 3882 2034 50  0000 C CNN
-F 2 "telec:JackHole" H 3900 1700 50  0001 C CNN
+F 2 "telec:Jack_Hole_Square" H 3900 1700 50  0001 C CNN
 F 3 "~" H 3900 1700 50  0001 C CNN
 	1    3900 1700
 	1    0    0    -1
 $EndComp
-NoConn ~ 4100 1600
 NoConn ~ 4100 1700
 NoConn ~ 4100 1800
@@
 L power:GND #PWR015
 U 1 1 5F48DF9C
-P 4200 1550
-F 0 "#PWR015" H 4200 1300 50  0001 C CNN
-F 1 "GND" H 4205 1377 50  0000 C CNN
-F 2 "" H 4200 1550 50  0001 C CNN
-F 3 "" H 4200 1550 50  0001 C CNN
-	1    4200 1550
-	1    0    0    -1
-$EndComp
-Wire Wire Line
-	4100 1500 4200 1500
-Wire Wire Line
-	4200 1500 4200 1550
+P 4200 1650
+F 0 "#PWR015" H 4200 1400 50  0001 C CNN
+F 1 "GND" H 4205 1477 50  0000 C CNN
+F 2 "" H 4200 1650 50  0001 C CNN
+F 3 "" H 4200 1650 50  0001 C CNN
+	1    4200 1650
+	1    0    0    -1
+$EndComp
+Wire Wire Line
+	4100 1600 4200 1600
+Wire Wire Line
+	4200 1600 4200 1650
 $Comp
 L power:GND #PWR022
@@
 F 0 "RV2" V 5050 1450 50  0000 C CNN
 F 1 "100k" V 5150 1450 50  0000 C CNN
-F 2 "Potentiometer_THT:Potentiometer_Piher_T-16L_Single_Vertical_Hole" H 5150 1450 50  0001 C CNN
+F 2 "telec:Potentiometer_Single_Vertical_Hole" H 5150 1450 50  0001 C CNN
 F 3 "~" H 5150 1450 50  0001 C CNN
 	1    5150 1450
@@
 $EndComp
 $Comp
-L Connector:AudioJack3_Switch J6
+L Connector:AudioJack3_SwitchTR J6
 U 1 1 5F8CF6A4
 P 3900 5650
 F 0 "J6" H 3882 6075 50  0000 C CNN
 F 1 "IN2" H 3882 5984 50  0000 C CNN
-F 2 "telec:JackHole" H 3900 5650 50  0001 C CNN
+F 2 "telec:Jack_Hole_Square" H 3900 5650 50  0001 C CNN
 F 3 "~" H 3900 5650 50  0001 C CNN
 	1    3900 5650
 	1    0    0    -1
 $EndComp
-NoConn ~ 4100 5550
 NoConn ~ 4100 5650
 NoConn ~ 4100 5750
@@
 L power:GND #PWR055
 U 1 1 5F8CF6AD
-P 4200 5500
-F 0 "#PWR055" H 4200 5250 50  0001 C CNN
-F 1 "GND" H 4205 5327 50  0000 C CNN
-F 2 "" H 4200 5500 50  0001 C CNN
-F 3 "" H 4200 5500 50  0001 C CNN
-	1    4200 5500
-	1    0    0    -1
-$EndComp
-Wire Wire Line
-	4100 5450 4200 5450
-Wire Wire Line
-	4200 5450 4200 5500
+P 4200 5600
+F 0 "#PWR055" H 4200 5350 50  0001 C CNN
+F 1 "GND" H 4205 5427 50  0000 C CNN
+F 2 "" H 4200 5600 50  0001 C CNN
+F 3 "" H 4200 5600 50  0001 C CNN
+	1    4200 5600
+	1    0    0    -1
+$EndComp
+Wire Wire Line
+	4100 5550 4200 5550
+Wire Wire Line
+	4200 5550 4200 5600
 $Comp
 L power:GND #PWR057
@@
 F 0 "RV4" V 3800 3800 50  0000 C CNN
 F 1 "100k" V 3900 3800 50  0000 C CNN
-F 2 "Potentiometer_THT:Potentiometer_Piher_T-16L_Single_Vertical_Hole" H 3900 3800 50  0001 C CNN
+F 2 "telec:Potentiometer_Single_Vertical_Hole" H 3900 3800 50  0001 C CNN
 F 3 "~" H 3900 3800 50  0001 C CNN
 	1    3900 3800
@@
 $EndComp
 $Comp
-L Connector:AudioJack3_Switch J7
+L Connector:AudioJack3_SwitchTR J7
 U 1 1 5F8CF6C9
 P 9600 5650
 F 0 "J7" H 9582 6075 50  0000 C CNN
 F 1 "OUT2" H 9582 5984 50  0000 C CNN
-F 2 "telec:JackHole" H 9600 5650 50  0001 C CNN
+F 2 "telec:Jack_Hole_Square" H 9600 5650 50  0001 C CNN
 F 3 "~" H 9600 5650 50  0001 C CNN
 	1    9600 5650
@@
 NoConn ~ 9400 5750
 NoConn ~ 9400 5650
-NoConn ~ 9400 5550
 NoConn ~ 9400 5950
 $Comp
 L power:GND #PWR054
 U 1 1 5F8CF6D3
-P 9400 5450
-F 0 "#PWR054" H 9400 5200 50  0001 C CNN
-F 1 "GND" V 9405 5322 50  0000 R CNN
-F 2 "" H 9400 5450 50  0001 C CNN
-F 3 "" H 9400 5450 50  0001 C CNN
-	1    9400 5450
+P 9400 5550
+F 0 "#PWR054" H 9400 5300 50  0001 C CNN
+F 1 "GND" V 9405 5422 50  0000 R CNN
+F 2 "" H 9400 5550 50  0001 C CNN
+F 3 "" H 9400 5550 50  0001 C CNN
+	1    9400 5550
 	0    1    1    0
 $EndComp
 $Comp
-L Connector:AudioJack3_Switch J5
+L Connector:AudioJack3_SwitchTR J5
 U 1 1 5F8CF6D9
 P 3900 4650
 F 0 "J5" H 3882 5075 50  0000 C CNN
 F 1 "CV2" H 3882 4984 50  0000 C CNN
-F 2 "telec:JackHole" H 3900 4650 50  0001 C CNN
+F 2 "telec:Jack_Hole_Square" H 3900 4650 50  0001 C CNN
 F 3 "~" H 3900 4650 50  0001 C CNN
 	1    3900 4650
 	1    0    0    -1
 $EndComp
-NoConn ~ 4100 4550
 NoConn ~ 4100 4650
 NoConn ~ 4100 4750
@@
 L power:GND #PWR038
 U 1 1 5F8CF6E2
-P 4200 4500
-F 0 "#PWR038" H 4200 4250 50  0001 C CNN
-F 1 "GND" H 4205 4327 50  0000 C CNN
-F 2 "" H 4200 4500 50  0001 C CNN
-F 3 "" H 4200 4500 50  0001 C CNN
-	1    4200 4500
-	1    0    0    -1
-$EndComp
-Wire Wire Line
-	4100 4450 4200 4450
-Wire Wire Line
-	4200 4450 4200 4500
+P 4200 4600
+F 0 "#PWR038" H 4200 4350 50  0001 C CNN
+F 1 "GND" H 4205 4427 50  0000 C CNN
+F 2 "" H 4200 4600 50  0001 C CNN
+F 3 "" H 4200 4600 50  0001 C CNN
+	1    4200 4600
+	1    0    0    -1
+$EndComp
+Wire Wire Line
+	4100 4550 4200 4550
+Wire Wire Line
+	4200 4550 4200 4600
 $Comp
 L power:GND #PWR047
@@
 F 0 "RV5" V 5050 4400 50  0000 C CNN
 F 1 "100k" V 5150 4400 50  0000 C CNN
-F 2 "Potentiometer_THT:Potentiometer_Piher_T-16L_Single_Vertical_Hole" H 5150 4400 50  0001 C CNN
+F 2 "telec:Potentiometer_Single_Vertical_Hole" H 5150 4400 50  0001 C CNN
 F 3 "~" H 5150 4400 50  0001 C CNN
 	1    5150 4400

Commit message: VCA ready for prod
Parts:
- R10: value 150k -> 120k
- R11: value 27k -> 220k
- R7: value 10k -> 12k
Changed lines of the file:
@@
 P 6300 2600
 F 0 "R7" V 6400 2600 50  0000 L CNN
-F 1 "10k" V 6300 2550 50  0000 L CNN
+F 1 "12k" V 6300 2550 50  0000 L CNN
 F 2 "Resistor_SMD:R_1206_3216Metric_Pad1.42x1.75mm_HandSolder" V 6230 2600 50  0001 C CNN
 F 3 "~" H 6300 2600 50  0001 C CNN
@@
 P 5700 3000
 F 0 "R10" V 5800 3000 50  0000 L CNN
-F 1 "150k" V 5700 2900 50  0000 L CNN
+F 1 "120k" V 5700 2900 50  0000 L CNN
 F 2 "Resistor_SMD:R_1206_3216Metric_Pad1.42x1.75mm_HandSolder" V 5630 3000 50  0001 C CNN
 F 3 "~" H 5700 3000 50  0001 C CNN
@@
 P 8050 3250
 F 0 "R11" V 8150 3250 50  0000 L CNN
-F 1 "27k" V 8050 3200 50  0000 L CNN
+F 1 "220k" V 8050 3150 50  0000 L CNN
 F 2 "Resistor_SMD:R_1206_3216Metric_Pad1.42x1.75mm_HandSolder" V 7980 3250 50  0001 C CNN
 F 3 "~" H 8050 3250 50  0001 C CNN
