File: VCO/VCO.kicad_pcb (KiCad board)
At the start: 2 copper layers, 51 parts, among them J1 EuroPower, J2 CV, J3 Triangle, J4 Square, J5 CV3, J6 Ramp, Q1 BC547, Q2 BC547, Q3 BC547, Q4 MMDT3904, Q5 BC547, U1 TL082, U2 TL082, U3 TL082

Commit message: VCO PCB
Parts:
- R18: footprint Resistor_THT:R_Axial_DIN0204_L3.6mm_D1.6mm_P7.62mm_Horizontal -> Resistor_THT:R_Axial_DIN0204_L3.6mm_D1.6mm_P2.54mm_Vertical
- R7: moved to F.Cu
- moved R7 93.3 mm to (103.8, 47.2)
- moved TP1 90.3 mm to (104.6, 50.0)
- moved C4 80.6 mm to (100.4, 48.2)
- moved U2 80.6 mm to (93.6, 50.3)
- moved C3 80.5 mm to (97.3, 40.4)
- moved R15 80.3 mm to (91.0, 39.6)
- moved R18 80.2 mm to (97.1, 55.3)
- moved R14 80.1 mm to (100.7, 40.0)
- moved Q4 80.1 mm to (96.5, 46.1)
- moved TP2 80.0 mm to (90.2, 50.0)
- moved RV3 79.8 mm to (94.4, 52.9)
- moved C6 77.9 mm to (93.4, 37.4)
Routing:
- net GND: track 0.00 -> 39.5 mm, vias 0 -> 1
- net -12V: track 0.00 -> 25.5 mm, vias 0 -> 1
- net /Vexp: track 0.00 -> 18.3 mm
- net +12V: track 0.00 -> 15.7 mm, vias 0 -> 1
- net Net-(C6-Pad2): track 0.00 -> 14.2 mm
- net Net-(Q4-Pad1): track 0.00 -> 13.6 mm
- net /CV: track 0.00 -> 12.1 mm
- net Net-(Q4-Pad3): track 0.00 -> 9.74 mm
- net Net-(C6-Pad1): track 0.00 -> 9.73 mm
- net Net-(R7-Pad2): track 0.00 -> 6.96 mm, vias 0 -> 1
- net Net-(R18-Pad1): track 0.00 -> 3.71 mm
Other:
- net class Default: clearance 0.2 -> 0.1524; trace_width 0.25 -> 0.1524; via_dia 0.8 -> 0.6858; via_drill 0.4 -> 0.3302
- rule trace_clearance: 0.2 -> 0.1524
- rule trace_min: 0.2 -> 0.1524
- rule via_min_drill: 0.3 -> 0.254
- rule via_min_size: 0.4 -> 0.508
- board text added: "+12V"
- board text added: "-12V"
- board text added: "Exponentiator"
- board text added: "GND"
- board text added: "IN"

Commit message: VCO - Nice schematic
Parts:
- removed J6: Ramp, Connector_PinHeader_2.54mm:PinHeader_1x01_P2.54mm_Vertical
- added H1: Mounting_Holes, Kosmo_panel:Kosmo_Panel_Dual_Mounting_Holes, F.Cu at (15.0, 209.0)
- added H2: Mounting_Holes, Kosmo_panel:Kosmo_Panel_Dual_Mounting_Holes, F.Cu at (59.0, 209.0)
- added LOGO1: Logo_telec, logo:telec-16, F.Cu at (73.1, 31.9)
- added R23: 130k, Resistor_THT:R_Axial_DIN0204_L3.6mm_D1.6mm_P7.62mm_Horizontal, F.Cu at (24.1, 57.0)
- added TP1: CV3, Connector_PinHeader_2.54mm:PinHeader_1x01_P2.54mm_Vertical, F.Cu at (19.9, 62.2)
- J1: footprint Connector_IDC:IDC-Header_2x05_P2.54mm_Vertical -> telec:EuroPower
- J5: value CV3 -> Ramp; footprint Connector_PinHeader_2.54mm:PinHeader_1x01_P2.54mm_Vertical -> telec:JackHole
- RV1, RV3: footprint Potentiometer_THT:Potentiometer_Runtron_RM-065_Vertical -> Potentiometer_THT:Potentiometer_Bourns_3299W_Vertical
- RV4: footprint Potentiometer_THT:Potentiometer_Runtron_RM-065_Vertical -> telec:Potentiometer_P3.81mmx5.12mm_Vertical
- moved J5 149.4 mm to (21.0, 190.3), turned to 90 degrees
- moved C6 101.2 mm to (-5.90, 56.9)
- moved RV3 101.2 mm to (-4.90, 72.4)
- moved C3 101.2 mm to (-1.98, 59.9)
- moved C4 101.2 mm to (1.07, 67.7)
- moved Q4 101.2 mm to (-2.85, 65.7)
- moved R14 101.2 mm to (1.40, 59.5)
- moved R15 101.2 mm to (-8.30, 59.1)
- moved R18 101.2 mm to (-2.20, 74.8)
- moved R7 101.2 mm to (4.50, 66.7)
- moved TP2 101.2 mm to (5.30, 69.5)
- moved TP3 101.2 mm to (-9.10, 69.5)
- moved U2 101.2 mm to (-5.70, 69.8)
- moved J2 84.5 mm to (22.4, 116.0)
- moved J4 66.6 mm to (21.6, 165.4), turned to 90 degrees
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- renumbered TP1 to TP2, TP2 to TP3, TP3 to TP4
Connections:
- J1 pad 1: -12V -> +12V
- J1 pad 2: -12V -> GND
- J1 pad 3: GND -> -12V
- RV2 pad 1: +12V -> Net-(R23-Pad1)
Other:
- board outline added: 50 x 200 mm

Commit message: VCO layout done!
Parts:
- removed the C6 at (-5.90, 56.9)
- removed the Q4 at (-2.85, 65.7)
- removed the R14 at (1.40, 59.5)
- removed the R15 at (-8.30, 59.1)
- removed the R18 at (-2.20, 74.8)
- removed the R2 at (34.0, 65.3)
- removed the R23 at (24.1, 57.0)
- added C5: 100n, Capacitor_SMD:C_0805_2012Metric_Pad1.15x1.40mm_HandSolder, B.Cu at (18.9, 82.7)
- added D1: LED, LED_SMD:LED_1206_3216Metric_ReverseMount_Hole1.8x2.4mm, B.Cu at (37.1, 181.1)
- added D2: LED, LED_SMD:LED_1206_3216Metric_ReverseMount_Hole1.8x2.4mm, B.Cu at (37.1, 176.3)
- added D3: LED, LED_SMD:LED_1206_3216Metric_Castellated, B.Cu at (41.8, 40.1)
- added D4: LED, LED_SMD:LED_1206_3216Metric_Castellated, B.Cu at (60.6, 33.6)
- added J5: PWM, telec:JackHole, F.Cu at (48.7, 169.4)
- added J6: Triangle, telec:JackHole, F.Cu at (25.3, 192.7)
- added JP2: Buffer ?, Jumper:SolderJumper-2_P1.3mm_Open_Pad1.0x1.5mm, B.Cu at (49.3, 62.5)
- added Q1: MMDT3904, Package_TO_SOT_SMD:SOT-363_SC-70-6, B.Cu at (22.9, 84.8)
- added R1: 130k, Resistor_THT:R_Axial_DIN0204_L3.6mm_D1.6mm_P7.62mm_Horizontal, F.Cu at (20.3, 110.2)
- added R10: 22k, Resistor_THT:R_Axial_DIN0204_L3.6mm_D1.6mm_P7.62mm_Horizontal, F.Cu at (28.5, 77.9)
- added R26: 1k, Resistor_SMD:R_1206_3216Metric_Pad1.42x1.75mm_HandSolder, B.Cu at (17.8, 156.5)
- added R27: 1k, Resistor_SMD:R_1206_3216Metric_Pad1.42x1.75mm_HandSolder, B.Cu at (41.4, 156.6)
- added R28: 1k, Resistor_SMD:R_1206_3216Metric_Pad1.42x1.75mm_HandSolder, B.Cu at (18.0, 179.8)
- added R29: 1k, Resistor_SMD:R_1206_3216Metric_Pad1.42x1.75mm_HandSolder, B.Cu at (41.4, 179.9)
- added R3: 100k, Resistor_THT:R_Axial_DIN0204_L3.6mm_D1.6mm_P7.62mm_Horizontal, F.Cu at (14.6, 109.6)
- added R30: 2k2, Resistor_SMD:R_1206_3216Metric_Pad1.42x1.75mm_HandSolder, B.Cu at (34.3, 181.2)
- added R31: 2k2, Resistor_SMD:R_1206_3216Metric_Pad1.42x1.75mm_HandSolder, B.Cu at (34.3, 176.2)
- added R32: 1k5, Resistor_SMD:R_1206_3216Metric_Pad1.42x1.75mm_HandSolder, B.Cu at (41.8, 33.5)
- added R33: 1k5, Resistor_SMD:R_1206_3216Metric_Pad1.42x1.75mm_HandSolder, B.Cu at (60.6, 40.0)
- added R34: 100k, Resistor_THT:R_Axial_DIN0204_L3.6mm_D1.6mm_P7.62mm_Horizontal, F.Cu at (53.4, 85.0)
- added R35: 100k, Resistor_THT:R_Axial_DIN0204_L3.6mm_D1.6mm_P7.62mm_Horizontal, F.Cu at (38.6, 74.6)
- added R5: 47k, Resistor_THT:R_Axial_DIN0204_L3.6mm_D1.6mm_P7.62mm_Horizontal, F.Cu at (37.0, 135.2)
- added R6: 4k7, Resistor_THT:R_Axial_DIN0204_L3.6mm_D1.6mm_P7.62mm_Horizontal, F.Cu at (33.2, 96.7)
- added R8: 1M, Resistor_THT:R_Axial_DIN0204_L3.6mm_D1.6mm_P7.62mm_Horizontal, F.Cu at (18.6, 90.9)
- added R9: 1k, Resistor_THT:R_Axial_DIN0204_L3.6mm_D1.6mm_P7.62mm_Horizontal, F.Cu at (28.3, 91.3)
- added RV1: 100k, Potentiometer_THT:Potentiometer_Piher_T-16L_Single_Vertical_Hole, F.Cu at (20.3, 112.8)
- added RV5: 10k, Potentiometer_THT:Potentiometer_Bourns_3299W_Vertical, F.Cu at (31.8, 78.0)
- added U4: TL082, Package_DIP:DIP-8_W7.62mm_LongPads, F.Cu at (50.7, 77.3)
- C3: value 100n -> 1n; footprint Capacitor_SMD:C_0805_2012Metric_Pad1.15x1.40mm_HandSolder -> Capacitor_THT:C_Disc_D7.0mm_W2.5mm_P5.00mm; moved to F.Cu
- J3: value Triangle -> CV PWM
- LOGO1: value Logo_telec -> telec
- RV3: value 10k -> 100k; footprint Potentiometer_THT:Potentiometer_Bourns_3299W_Vertical -> Potentiometer_THT:Potentiometer_Piher_T-16L_Single_Vertical_Hole
- moved R18 72.5 mm to (41.3, 47.7), turned to 0 degrees
- moved R17 70.1 mm to (41.4, 49.9), turned to 270 degrees
- moved Q3 67.0 mm to (44.6, 49.9), turned to 270 degrees
- moved R23 64.7 mm to (39.0, 57.5), turned to 90 degrees
- moved RV3 63.2 mm to (43.7, 112.8)
- moved Q4 63.0 mm to (49.4, 49.9), turned to 270 degrees
- moved R2 62.6 mm to (13.5, 127.4), turned to 270 degrees
- moved R16 57.3 mm to (30.0, 47.2), turned to 180 degrees
- moved RV6 57.0 mm to (24.4, 44.1), turned to 270 degrees
- moved Q5 53.9 mm to (45.3, 62.4), turned to 90 degrees
- moved TP1 53.9 mm to (35.8, 113.7), turned to 180 degrees
- moved R25 53.5 mm to (38.7, 64.6), turned to 0 degrees
- moved R24 51.3 mm to (38.7, 67.6), turned to 0 degrees
- moved R21 50.7 mm to (48.7, 57.2), turned to 270 degrees
- moved U1 49.2 mm to (23.1, 106.9), turned to 90 degrees
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- renumbered C7 to C6, C5 to C7, J5 to J7, Q1 to Q3, Q3 to Q4, R3 to R11, R19 to R12, R20 to R13, R21 to R14, R8 to R15, R22 to R16, R5 to R17, R6 to R18, R9 to R19, R1 to R2, R10 to R20, R11 to R21, R12 to R22, R13 to R23, R16 to R24, R17 to R25, RV1 to RV4, RV4 to RV6
Connections:
- net /Ramp renamed /Raw_Ramp
- C3 pad 1: +12V -> Net-(C3-Pad1)
- C3 pad 2: GND -> Net-(C3-Pad2)
- C4 pad 1: -12V -> +12V
- J3 pad T: /Triangle -> /CVP
- J3 pad TN: Net-(J3-PadTN) -> GND
- J4 pad T: /Square -> Net-(J4-PadT)
- J7 pad T: /Triangle -> Net-(J7-PadT)
- R19 pad 2: Net-(R12-Pad1) (its old number) -> Net-(R19-Pad2)
- R20 pad 2: /~Triangle -> /Triangle
- R22 pad 1: Net-(R12-Pad1) (its old number) -> Net-(R19-Pad2)
- R24 pad 2: /Triangle -> /~Triangle
- RV2 pad 1: Net-(R23-Pad1) -> +12V
- RV2 pad 2: /CV2 -> /Offset
- RV2 pad 3: GND -> GNDREF
- RV3 pad 1: Net-(R18-Pad1) -> Net-(R5-Pad2)
- RV3 pad 2: /Vexp -> Net-(R5-Pad2)
- RV3 pad 3: /Vexp -> Net-(R6-Pad1)
- U1 pad 5: GND -> /Offset
- U1 pad 6: Net-(R12-Pad1) (its old number) -> Net-(R5-Pad2)
- U1 pad 7: /~Triangle -> /PWM_level
- U2 pad 6: Net-(C6-Pad2) (its old number) -> Net-(C3-Pad2)
- U2 pad 7: Net-(C6-Pad1) -> Net-(C3-Pad1)
Routing:
- net /Triangle: track 0.00 -> 224.0 mm, vias 0 -> 3
- net +12V: track 15.7 -> 216.4 mm, vias 1 -> 7
- net /Square: track 0.00 -> 186.3 mm, vias 0 -> 6
- net /Ramp: track 0.00 -> 140.8 mm, vias 0 -> 2
- net -12V: track 25.5 -> 135.8 mm, vias 1 -> 4
- net /PWM: track 0.00 -> 88.3 mm, vias 0 -> 1
- net Net-(R5-Pad2): track 0.00 -> 47.6 mm
- net Net-(R2-Pad1): track 0.00 -> 42.8 mm
- net GNDREF: track 0.00 -> 38.5 mm
- net /PWM_level: track 0.00 -> 30.6 mm
- net Net-(R6-Pad1): track 0.00 -> 29.3 mm
- net /Offset: track 0.00 -> 23.4 mm
- net Net-(Q2-Pad1): track 0.00 -> 17.0 mm
- net Net-(R19-Pad2): track 0.00 -> 15.8 mm
- net Net-(C6-Pad2) (its old number): track 14.2 -> 0.00 mm
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- added copper zone on B.Cu, net GND
- added copper zone on B.Cu, net GNDREF
Other:
- board text added: "Mister VCO"
- board text removed: "IN"

Commit message: VCO done !
Parts:
- moved J2 0.30 mm to (25.2, 146.1)
- moved J3 0.10 mm to (48.5, 146.1)
Other:
- outline, holes or cut-outs redrawn
- board text added: "+"
- board text added: "-"
- board text added: "CV"
- board text added: "CV Mix"
- board text added: "CVP"
- board text added: "Hi!"
- board text added: "Integrator + Hysteresis VCO"
- board text added: "PWM"
- board text added: "RMP"
- board text added: "SQU"
- board text added: "TRI"
- board text added: "Triangle to Ramp"
- board text added: "~Triangle~ & PWM generation"

Commit message: Added PCB ref stamp and send to prod!
Other:
- board text added: "Design by telec & the internet"
- board text added: "PCB ref here:"
Changed lines of the file:
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@@
   (general
     (thickness 1.6)
-    (drawings 174)
+    (drawings 180)
     (tracks 395)
     (zones 0)
@@
     )
   )
+  (gr_text "Design by\ntelec & the internet" (at 37.1 209) (layer B.SilkS)
+    (effects (font (size 1.5 1.5) (thickness 0.3)) (justify mirror))
+  )
+  (gr_text "PCB ref here:" (at 48.6 104.7) (layer B.SilkS)
+    (effects (font (size 1 1) (thickness 0.15)) (justify mirror))
+  )
+  (gr_line (start 43 103.8) (end 43 108.1) (layer B.SilkS) (width 0.15))
+  (gr_line (start 54.4 103.8) (end 43 103.8) (layer B.SilkS) (width 0.15))
+  (gr_line (start 54.4 108.1) (end 54.4 103.8) (layer B.SilkS) (width 0.15))
+  (gr_line (start 43 108.1) (end 54.4 108.1) (layer B.SilkS) (width 0.15))
   (gr_text - (at 37.1 182.5) (layer F.SilkS)
     (effects (font (size 1.5 1.5) (thickness 0.3)))

Commit message: New PCB
Parts:
- removed C3, C6: 1n, Capacitor_THT:C_Disc_D7.0mm_W2.5mm_P5.00mm
- removed C4, C5, C7: 100n, Capacitor_SMD:C_0805_2012Metric_Pad1.15x1.40mm_HandSolder
- removed JP1: Reference, Connector_PinHeader_2.54mm:PinHeader_1x03_P2.54mm_Vertical
- removed JP2: Buffer ?, Jumper:SolderJumper-2_P1.3mm_Open_Pad1.0x1.5mm
- removed Q1: MMDT3904, Package_TO_SOT_SMD:SOT-363_SC-70-6
- removed Q2, Q3, Q4, Q5: BC547, Package_TO_SOT_THT:TO-92_Inline_Wide
- removed R1: 130k, Resistor_THT:R_Axial_DIN0204_L3.6mm_D1.6mm_P7.62mm_Horizontal
- removed R10: 22k, Resistor_THT:R_Axial_DIN0204_L3.6mm_D1.6mm_P7.62mm_Horizontal
- removed R11, R15, R16, R17, R18, R19, R2, R22, R23, R3, R34, R35, R4: 100k, Resistor_THT:R_Axial_DIN0204_L3.6mm_D1.6mm_P7.62mm_Horizontal
- removed R12, R13, R14: 56k, Resistor_THT:R_Axial_DIN0204_L3.6mm_D1.6mm_P7.62mm_Horizontal
- removed R20, R21, R24, R25, R5: 47k, Resistor_THT:R_Axial_DIN0204_L3.6mm_D1.6mm_P7.62mm_Horizontal
- removed R6: 4k7, Resistor_THT:R_Axial_DIN0204_L3.6mm_D1.6mm_P7.62mm_Horizontal
- removed R7: 0, Resistor_THT:R_Axial_DIN0204_L3.6mm_D1.6mm_P7.62mm_Horizontal
- removed R8: 1M, Resistor_THT:R_Axial_DIN0204_L3.6mm_D1.6mm_P7.62mm_Horizontal
- removed R9: 1k, Resistor_THT:R_Axial_DIN0204_L3.6mm_D1.6mm_P7.62mm_Horizontal
- removed RV1, RV2, RV3: 100k, Potentiometer_THT:Potentiometer_Piher_T-16L_Single_Vertical_Hole
- removed RV4, RV5: 10k, Potentiometer_THT:Potentiometer_Bourns_3299W_Vertical
- removed RV6: 220k, telec:Potentiometer_P3.81mmx5.12mm_Vertical
- removed TP1: CV3, Connector_PinHeader_2.54mm:PinHeader_1x01_P2.54mm_Vertical
- removed TP4: ~Triangle, Connector_PinHeader_2.54mm:PinHeader_1x01_P2.54mm_Vertical
- removed U1, U2, U3, U4: TL082, Package_DIP:DIP-8_W7.62mm_LongPads
- added C103: 100n, Capacitor_SMD:C_0805_2012Metric_Pad1.15x1.40mm_HandSolder, F.Cu at (74.4, 125.6)
- added C104: 100n, Capacitor_SMD:C_0805_2012Metric_Pad1.15x1.40mm_HandSolder, F.Cu at (69.7, 125.6)
- added C201: 100n, Capacitor_SMD:C_0805_2012Metric_Pad1.15x1.40mm_HandSolder, B.Cu at (22.6, 53.1)
- added C202: 1n, Capacitor_THT:C_Disc_D7.0mm_W2.5mm_P5.00mm, F.Cu at (23.3, 60.8)
- added C401: 100n, Capacitor_SMD:C_0805_2012Metric_Pad1.15x1.40mm_HandSolder, F.Cu at (8.63, 87.7)
- added C402: 100n, Capacitor_SMD:C_0805_2012Metric_Pad1.15x1.40mm_HandSolder, F.Cu at (8.63, 83.0)
- added C403: 220p, Capacitor_THT:C_Disc_D7.0mm_W2.5mm_P5.00mm, F.Cu at (25.7, 73.7)
- added C404: 1n, Capacitor_THT:C_Disc_D7.0mm_W2.5mm_P5.00mm, F.Cu at (25.8, 93.7)
- added D101: Ref, Diode_SMD:D_1206_3216Metric_Pad1.42x1.75mm_HandSolder, F.Cu at (97.3, 117.2)
- added Q201: BC547, Package_TO_SOT_THT:TO-92_Inline_Wide, F.Cu at (13.6, 58.3)
- added Q401: DMMT3904, Package_TO_SOT_SMD:SOT-363_SC-70-6, B.Cu at (22.9, 84.9)
- added Q501: BC547, Package_TO_SOT_THT:TO-92_Inline_Wide, F.Cu at (97.2, 68.1)
- added Q502: BC547, Package_TO_SOT_THT:TO-92_Inline_Wide, F.Cu at (97.2, 73.8)
- added R101: 4k7, Resistor_SMD:R_1206_3216Metric_Pad1.42x1.75mm_HandSolder, F.Cu at (97.3, 123.8)
- added R102: 47k, Resistor_THT:R_Axial_DIN0204_L3.6mm_D1.6mm_P7.62mm_Horizontal, F.Cu at (79.3, 122.8)
- added R103: 47k, Resistor_THT:R_Axial_DIN0204_L3.6mm_D1.6mm_P7.62mm_Horizontal, F.Cu at (95.7, 107.4)
- added R105: 100k, Resistor_SMD:R_1206_3216Metric_Pad1.42x1.75mm_HandSolder, F.Cu at (97.3, 120.5)
- added R106: 100k, Resistor_SMD:R_1206_3216Metric_Pad1.42x1.75mm_HandSolder, F.Cu at (91.4, 122.9)
- added R108: 47k, Resistor_THT:R_Axial_DIN0204_L3.6mm_D1.6mm_P7.62mm_Horizontal, F.Cu at (68.8, 122.5)
- added R201: 100k, Resistor_THT:R_Axial_DIN0204_L3.6mm_D1.6mm_P7.62mm_Horizontal, F.Cu at (24.5, 63.0)
- added R202: 56k, Resistor_THT:R_Axial_DIN0204_L3.6mm_D1.6mm_P7.62mm_Horizontal, F.Cu at (28.5, 63.0)
- added R203: 56k, Resistor_THT:R_Axial_DIN0204_L3.6mm_D1.6mm_P7.62mm_Horizontal, F.Cu at (32.4, 70.5)
- added R204: 56k, Resistor_THT:R_Axial_DIN0204_L3.6mm_D1.6mm_P7.62mm_Horizontal, F.Cu at (20.8, 70.5)
- added R205: 100k, Resistor_THT:R_Axial_DIN0204_L3.6mm_D1.6mm_P7.62mm_Horizontal, F.Cu at (29.9, 47.2)
- added R206: 100k, Resistor_THT:R_Axial_DIN0204_L3.6mm_D1.6mm_P7.62mm_Horizontal, F.Cu at (16.1, 54.7)
- added R301: 1k8, Resistor_THT:R_Axial_DIN0204_L3.6mm_D1.6mm_P7.62mm_Horizontal, F.Cu at (0.59, 98.9)
- added R302: 100k, Resistor_THT:R_Axial_DIN0204_L3.6mm_D1.6mm_P7.62mm_Horizontal, F.Cu at (-11.0, 113.8)
- added R303: 0, Resistor_THT:R_Axial_DIN0204_L3.6mm_D1.6mm_P7.62mm_Horizontal, F.Cu at (14.4, 83.6)
- added R304: 100k, Resistor_THT:R_Axial_DIN0204_L3.6mm_D1.6mm_P7.62mm_Horizontal, F.Cu at (-11.0, 110.6)
- added R305: 100k, Resistor_THT:R_Axial_DIN0204_L3.6mm_D1.6mm_P7.62mm_Horizontal, F.Cu at (-0.44, 110.6)
- added R306: 4k7, Resistor_THT:R_Axial_DIN0204_L3.6mm_D1.6mm_P7.62mm_Horizontal, F.Cu at (0.59, 105.2)
- added R307: 47k, Resistor_THT:R_Axial_DIN0204_L3.6mm_D1.6mm_P7.62mm_Horizontal, F.Cu at (-11.0, 116.9)
- added R401: 22k, Resistor_THT:R_Axial_DIN0204_L3.6mm_D1.6mm_P7.62mm_Horizontal, F.Cu at (28.4, 77.8)
- added R402: 1M, Resistor_THT:R_Axial_DIN0204_L3.6mm_D1.6mm_P7.62mm_Horizontal, F.Cu at (18.6, 91.0)
- added R403: 0, Resistor_THT:R_Axial_DIN0204_L3.6mm_D1.6mm_P7.62mm_Horizontal, F.Cu at (9.80, 70.2)
- added R404: 1k, Resistor_THT:R_Axial_DIN0204_L3.6mm_D1.6mm_P7.62mm_Horizontal, F.Cu at (28.5, 91.3)
- added R501: 100k, Resistor_THT:R_Axial_DIN0204_L3.6mm_D1.6mm_P7.62mm_Horizontal, F.Cu at (86.6, 75.0)
- added R502: 100k, Resistor_THT:R_Axial_DIN0204_L3.6mm_D1.6mm_P7.62mm_Horizontal, F.Cu at (65.4, 68.7)
- added R503: 47k, Resistor_THT:R_Axial_DIN0204_L3.6mm_D1.6mm_P7.62mm_Horizontal, F.Cu at (76.0, 68.7)
- added R504: 47k, Resistor_THT:R_Axial_DIN0204_L3.6mm_D1.6mm_P7.62mm_Horizontal, F.Cu at (65.4, 71.8)
- added R505: 47k, Resistor_THT:R_Axial_DIN0204_L3.6mm_D1.6mm_P7.62mm_Horizontal, F.Cu at (65.4, 75.0)
- added R506: 47k, Resistor_THT:R_Axial_DIN0204_L3.6mm_D1.6mm_P7.62mm_Horizontal, F.Cu at (88.6, 56.9)
- added R507: 100k, Resistor_THT:R_Axial_DIN0204_L3.6mm_D1.6mm_P7.62mm_Horizontal, F.Cu at (76.0, 71.8)
- added R508: 100k, Resistor_THT:R_Axial_DIN0204_L3.6mm_D1.6mm_P7.62mm_Horizontal, F.Cu at (86.6, 68.7)
- added R509: 100k, Resistor_THT:R_Axial_DIN0204_L3.6mm_D1.6mm_P7.62mm_Horizontal, F.Cu at (76.0, 75.0)
- added R510: 100k, Resistor_THT:R_Axial_DIN0204_L3.6mm_D1.6mm_P7.62mm_Horizontal, F.Cu at (88.6, 60.1)
- added R511: 220k, Resistor_THT:R_Axial_DIN0204_L3.6mm_D1.6mm_P7.62mm_Horizontal, F.Cu at (88.6, 63.2)
- added R512: 100k, Resistor_THT:R_Axial_DIN0204_L3.6mm_D1.6mm_P7.62mm_Horizontal, F.Cu at (86.6, 71.8)
- added RV101: 100k, Potentiometer_THT:Potentiometer_Bourns_3296W_Vertical, F.Cu at (91.2, 108.6)
- added RV102: 10k, Potentiometer_THT:Potentiometer_Bourns_3296W_Vertical, F.Cu at (91.2, 116.3)
- added RV103: 100k, telec:Potentiometer_Single_Vertical_Hole, F.Cu at (48.7, 99.5)
- added RV201: 220k, telec:Potentiometer_P3.81mmx5.12mm_Vertical, F.Cu at (24.4, 44.1)
- added RV301: 100k, telec:Potentiometer_Single_Vertical_Hole, F.Cu at (48.7, 123.0)
- added RV401: 10k, Potentiometer_THT:Potentiometer_Bourns_3296W_Vertical, F.Cu at (31.8, 77.9)
- added SW101: Octave, telec:Switch_Hole, F.Cu at (25.5, 122.8)
- added U101: TL082, Package_SO:SOIC-8_3.9x4.9mm_P1.27mm, F.Cu at (98.5, 112.2)
- added U201: TL082, Package_DIP:DIP-8_W7.62mm_LongPads, F.Cu at (22.6, 57.5)
- added U301: TL082, Package_DIP:DIP-8_W7.62mm_LongPads, F.Cu at (23.0, 106.7)
- added U401: TL082, Package_DIP:DIP-8_W7.62mm_LongPads, F.Cu at (25.7, 80.6)
- added U501: TL082, Package_DIP:DIP-8_W7.62mm_LongPads, F.Cu at (77.3, 54.7)
- added U502: TL082, Package_DIP:DIP-8_W7.62mm_LongPads, F.Cu at (64.8, 54.9)
- J102: renamed from J2; footprint telec:JackHole -> telec:Jack_Hole_Square
- J103: renamed from J4; footprint telec:JackHole -> telec:Jack_Hole_Square
- J104: renamed from J5; footprint telec:JackHole -> telec:Jack_Hole_Square
- J105: renamed from J3; footprint telec:JackHole -> telec:Jack_Hole_Square
- J106: renamed from J6; footprint telec:JackHole -> telec:Jack_Hole_Square
- J107: renamed from J7; footprint telec:JackHole -> telec:Jack_Hole_Square
- renumbered C1 to C101, C2 to C102, D4 to D102, D3 to D103, D1 to D104, D2 to D105, H1 to H101, H2 to H102, J1 to J101, LOGO1 to LOGO101, R26 to R104, R27 to R107, R28 to R109, R29 to R110, R32 to R111, R30 to R112, R31 to R113, R33 to R114, TP2 to TP101, TP3 to TP102
Routing:
- net Net-(R307-Pad2): track 0.00 -> 76.8 mm
- net Net-(R5-Pad2): track 47.6 -> 0.00 mm
- net Net-(R301-Pad2): track 0.00 -> 42.8 mm
- net Net-(R2-Pad1): track 42.8 -> 0.00 mm
- net GNDREF: track 38.5 -> 0.00 mm
- net /PWM_level: track 30.6 -> 0.00 mm
- net /PWM_Level: track 0.00 -> 30.6 mm
- net Net-(R6-Pad1): track 29.3 -> 0.00 mm
- net (no net): track 0.00 -> 29.2 mm
- net Net-(R7-Pad2): track 20.5 -> 0.00 mm
- net Net-(R301-Pad1): track 0.00 -> 20.5 mm
- net Net-(Q201-Pad1): track 0.00 -> 17.0 mm
- net Net-(Q2-Pad1): track 17.0 -> 0.00 mm
- net Net-(C404-Pad2): track 0.00 -> 14.2 mm
- net Net-(C3-Pad2): track 14.2 -> 0.00 mm
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- removed copper zone on B.Cu, net GNDREF

Commit message: Layout VCO
Parts:
- C103, C104, C401, C402, D101, R101, R105, R106, RV101, U101: moved to B.Cu
- Q401: footprint Package_TO_SOT_SMD:SOT-363_SC-70-6 -> Package_TO_SOT_SMD:SOT-23-6_Handsoldering
- moved D101 79.9 mm to (18.9, 132.6), turned to 270 degrees
- moved R103 77.7 mm to (18.0, 107.6), turned to 270 degrees
- moved RV101 67.8 mm to (27.8, 132.6)
- moved U101 66.0 mm to (35.9, 133.2), turned to 90 degrees
- moved R101 65.7 mm to (32.0, 131.0), turned to 270 degrees
- moved RV102 64.8 mm to (26.8, 109.6)
- moved R105 59.1 mm to (39.9, 134.2), turned to 270 degrees
- moved R106 55.0 mm to (36.6, 128.2), turned to 180 degrees
- moved R108 53.2 mm to (15.6, 122.8), turned to 270 degrees
- moved R102 50.3 mm to (30.3, 111.7), turned to 90 degrees
- moved C104 49.7 mm to (21.2, 114.3)
- moved C103 46.4 mm to (29.5, 113.8), turned to 180 degrees
- moved R307 41.0 mm to (27.4, 102.7), turned to 90 degrees
- moved U501 35.1 mm to (42.3, 56.2), turned to 90 degrees
- moved U502 29.5 mm to (40.5, 71.6), turned to 90 degrees
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Connections:
- U502 pad 1: /Sheet5FAD0DD2/~Triangle -> /PWM
- U502 pad 2: Net-(R507-Pad1) -> /PWM_Level
- U502 pad 3: GND -> /Triangle
- U502 pad 5: /Triangle -> GND
- U502 pad 6: /PWM_Level -> Net-(R507-Pad1)
- U502 pad 7: /PWM -> /Sheet5FAD0DD2/~Triangle
Routing:
- net +12V: track 207.3 -> 75.7 mm, vias 7 -> 2
- net -12V: track 135.8 -> 46.7 mm, vias 4 -> 0
- net /Triangle: track 224.0 -> 136.0 mm, vias 3 -> 2
- net Net-(R307-Pad2): track 76.8 -> 0.00 mm
- net /+1V: track 0.00 -> 66.6 mm, vias 0 -> 1
- net /Square: track 186.3 -> 136.4 mm, vias 6 -> 5
- net /-1V: track 0.00 -> 37.0 mm, vias 0 -> 1
- net /Offset: track 32.4 -> 0.00 mm
- net Net-(R301-Pad2): track 42.8 -> 11.9 mm
- net /PWM_Level: track 30.6 -> 0.00 mm
- net /CV1: track 0.00 -> 29.8 mm
- net (no net): track 29.2 -> 0.00 mm
- net GND: track 39.7 -> 14.9 mm
- net Net-(R301-Pad1): track 20.5 -> 0.00 mm
- net Net-(R19-Pad2): track 15.8 -> 0.00 mm
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