File: VCO/VCO.sch (KiCad schematic (older format))
At the start: 51 parts, among them J1 EuroPower, J2 CV, J3 Triangle, J4 Square, J5 CV3, J6 Ramp, Q1 BC547, Q2 BC547, Q3 BC547, Q4 MMDT3904, Q5 BC547, U1 TL082, U2 TL082, U3 TL082

Commit message: VCO PCB
Parts:
- R18: footprint Resistor_THT:R_Axial_DIN0204_L3.6mm_D1.6mm_P7.62mm_Horizontal -> Resistor_THT:R_Axial_DIN0204_L3.6mm_D1.6mm_P2.54mm_Vertical
Changed lines of the file:
@@
 F 0 "R18" V 5650 950 50  0000 C CNN
 F 1 "22k" V 5750 950 50  0000 C CNN
-F 2 "Resistor_THT:R_Axial_DIN0204_L3.6mm_D1.6mm_P7.62mm_Horizontal" V 5680 950 50  0001 C CNN
+F 2 "Resistor_THT:R_Axial_DIN0204_L3.6mm_D1.6mm_P2.54mm_Vertical" V 5680 950 50  0001 C CNN
 F 3 "~" H 5750 950 50  0001 C CNN
 	1    5750 950

Commit message: VCO - Nice schematic
Parts:
- removed J1: EuroPower, Connector_IDC:IDC-Header_2x05_P2.54mm_Vertical, symbol Connector_Generic:Conn_02x05_Odd_Even
- removed J5: CV3, Connector_PinHeader_2.54mm:PinHeader_1x01_P2.54mm_Vertical, symbol Connector:Conn_01x01_Female
- removed J6: Ramp, Connector_PinHeader_2.54mm:PinHeader_1x01_P2.54mm_Vertical, symbol Connector:Conn_01x01_Female
- added D1, D2: LED, LED_SMD:LED_1206_3216Metric_ReverseMount_Hole1.8x2.4mm, symbol Device:LED
- added D3, D4: LED, LED_SMD:LED_1206_3216Metric_Castellated, symbol Device:LED
- added H1, H2: Mounting_Holes, Kosmo_panel:Kosmo_Panel_Dual_Mounting_Holes, symbol Kosmo:Mounting_Holes
- added J1: EuroPower, telec:EuroPower, symbol Connector:Screw_Terminal_01x03
- added J3: CV PWM, telec:JackHole, symbol Connector:AudioJack3_Switch
- added J5: PWM, telec:JackHole, symbol Connector:AudioJack3_Switch
- added J7: Ramp, telec:JackHole, symbol Connector:AudioJack3_Switch
- added LOGO1: telec, logo:telec-16, symbol logo:Logo_telec
- added R1: 130k, Resistor_THT:R_Axial_DIN0204_L3.6mm_D1.6mm_P7.62mm_Horizontal, symbol Device:R
- added R26, R27, R28, R29: 1k, Resistor_SMD:R_1206_3216Metric_Pad1.42x1.75mm_HandSolder, symbol Device:R
- added R30, R31: 2k2, Resistor_SMD:R_1206_3216Metric_Pad1.42x1.75mm_HandSolder, symbol Device:R
- added R32, R33: 1k5, Resistor_SMD:R_1206_3216Metric_Pad1.42x1.75mm_HandSolder, symbol Device:R
- added R5: 47k, Resistor_SMD:R_1206_3216Metric_Pad1.42x1.75mm_HandSolder, symbol Device:R
- added R6: 4k7, Resistor_SMD:R_1206_3216Metric_Pad1.42x1.75mm_HandSolder, symbol Device:R
- added RV1, RV3: 100k, Potentiometer_THT:Potentiometer_Piher_T-16L_Single_Vertical_Hole, symbol Device:R_POT
- added TP1: CV3, Connector_PinHeader_2.54mm:PinHeader_1x01_P2.54mm_Vertical, symbol Connector:TestPoint
- added unit 2 of U1
- added unit 3 of U1
- added unit 2 of U4
- RV4: renamed from RV1; footprint Potentiometer_THT:Potentiometer_Runtron_RM-065_Vertical -> Potentiometer_THT:Potentiometer_Bourns_3299W_Vertical
- RV5: renamed from RV3; footprint Potentiometer_THT:Potentiometer_Runtron_RM-065_Vertical -> Potentiometer_THT:Potentiometer_Bourns_3299W_Vertical
- RV6: renamed from RV4; footprint Potentiometer_THT:Potentiometer_Runtron_RM-065_Vertical -> telec:Potentiometer_P3.81mmx5.12mm_Vertical
- renumbered C6 to C3, C3 to C4, C4 to C5, C7 to C6, C5 to C7, J3 to J6, Q4 to Q1, Q1 to Q3, Q3 to Q4, R18 to R10, R3 to R11, R19 to R12, R20 to R13, R21 to R14, R8 to R15, R22 to R16, R5 to R17, R6 to R18, R9 to R19, R1 to R2, R10 to R20, R11 to R21, R12 to R22, R13 to R23, R16 to R24, R17 to R25, R2 to R3, R14 to R8, R15 to R9, TP1 to TP2, TP2 to TP3, TP3 to TP4, U1 to U4
Connections:
- net labels added: CVP, Offset, PWM, PWM_level
- wire segments 158 -> 184
- no-connect marks 11 -> 22
Other:
- note added: "5V"
- note added: "CV mix"
- note added: "Exponentiator"
- note added: "Front Panel"
- note added: "Input"
- note added: "Output"
- note added: "PWM"
- note added: "Ramp"
- note added: "VCO"
- moved on the sheet: C1, C2, C3, C4, C5, C6, C7, J4, J6, JP1, Q1A, Q1B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

Commit message: VCO layout done!
Parts:
- added JP2: Buffer ?, Jumper:SolderJumper-2_P1.3mm_Open_Pad1.0x1.5mm, symbol Jumper:SolderJumper_2_Open
- added R34, R35: 100k, Resistor_THT:R_Axial_DIN0204_L3.6mm_D1.6mm_P7.62mm_Horizontal, symbol Device:R
- R10: footprint Resistor_THT:R_Axial_DIN0204_L3.6mm_D1.6mm_P2.54mm_Vertical -> Resistor_THT:R_Axial_DIN0204_L3.6mm_D1.6mm_P7.62mm_Horizontal
- R5, R6: footprint Resistor_SMD:R_1206_3216Metric_Pad1.42x1.75mm_HandSolder -> Resistor_THT:R_Axial_DIN0204_L3.6mm_D1.6mm_P7.62mm_Horizontal
- U1: footprint Package_SO:SOIC-8_3.9x4.9mm_P1.27mm -> Package_DIP:DIP-8_W7.62mm_LongPads
Connections:
- net +12V: now also R34.1
- net GND: no longer U4.3 (+)
- net GNDREF: now also R35.1
- net Ramp: now also JP2.2 (B); no longer R21.2, R25.2
- net Triangle: now also R20.2; no longer R24.2
- net ~Triangle: now also R24.2; no longer R20.2
- new net: R34.2, R35.2, U4.3 (+)
- new net Raw_Ramp: JP2.1 (A), R21.2, R25.2
Other:
- note added: "Triangle"
- moved on the sheet: Q3, Q4, Q5, R17, R18, R19, R20, R21, R22, R23, R24, R25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

Commit message: Analog modules finished
Parts:
- removed JP1: Reference, Connector_PinHeader_2.54mm:PinHeader_1x03_P2.54mm_Vertical, symbol Jumper:Jumper_3_Bridged12
- removed JP2: Buffer ?, Jumper:SolderJumper-2_P1.3mm_Open_Pad1.0x1.5mm, symbol Jumper:SolderJumper_2_Open
- removed Q3: BC547, Package_TO_SOT_THT:TO-92_Inline_Wide, symbol Transistor_BJT:BC547
- removed R18, R34, R35: 100k, Resistor_THT:R_Axial_DIN0204_L3.6mm_D1.6mm_P7.62mm_Horizontal, symbol Device:R
- added R? (x3): 100k, Resistor_THT:R_Axial_DIN0204_L3.6mm_D1.6mm_P7.62mm_Horizontal, symbol Device:R
- added R?: 220k, Resistor_THT:R_Axial_DIN0204_L3.6mm_D1.6mm_P7.62mm_Horizontal, symbol Device:R
- added U5: TL082, Package_DIP:DIP-8_W7.62mm_LongPads, symbol Amplifier_Operational:TL082
Connections:
- net +12V: now also U5.8 (V+)
- net -12V: now also C7.2, RV2.3, RV6.3, U3.4 (V-), U5.4 (V-)
- net GND: now also Q2.3 (E), Q4.3 (E), Q5.3 (E), R13.1, U4.3 (+), R?.1, U5.3 (+)
- net Ramp: now also R?.2, U5.7
- net Raw_Ramp: now also U5.5 (+)
- net Square: now also R?.1; no longer R17.2
- net at Q4.2 (B): now also R17.1
- removed net GNDREF: C7.2, Q2.3 (E), Q4.3 (E), Q5.3 (E), R13.1, RV2.3, RV6.3, U3.4 (V-)
- new net: R?.1, R?.2, U5.2 (-)
- new net: R?.1, R?.2, U5.6 (-)
- new net ~Square: R17.2, R?.2, U5.1
Other:
- moved on the sheet: R17

Commit message: fix stuffs
Parts:
- removed R1: 130k, Resistor_THT:R_Axial_DIN0204_L3.6mm_D1.6mm_P7.62mm_Horizontal, symbol Device:R
- removed RV1: 100k, Potentiometer_THT:Potentiometer_Piher_T-16L_Single_Vertical_Hole, symbol Device:R_POT
- removed TP1: CV3, Connector_PinHeader_2.54mm:PinHeader_1x01_P2.54mm_Vertical, symbol Connector:TestPoint
- added C?: 220p, Capacitor_THT:C_Disc_D7.0mm_W2.5mm_P5.00mm, symbol Device:C
- added R?: 1k8, Resistor_THT:R_Axial_DIN0204_L3.6mm_D1.6mm_P7.62mm_Horizontal, symbol Device:R
- added R?: 0, Resistor_THT:R_Axial_DIN0204_L3.6mm_D1.6mm_P7.62mm_Horizontal, symbol Device:R
- added R? (x2): 560k, Resistor_THT:R_Axial_DIN0204_L3.6mm_D1.6mm_P7.62mm_Horizontal, symbol Device:R
- added R? (x2): 300k, Resistor_THT:R_Axial_DIN0204_L3.6mm_D1.6mm_P7.62mm_Horizontal, symbol Device:R
- added R? (x2): 27k, Resistor_THT:R_Axial_DIN0204_L3.6mm_D1.6mm_P7.62mm_Horizontal, symbol Device:R
Connections:
- net +12V: now also R?.1, R?.1
- net -12V: now also R?.2, R?.2
- net CV3: now also RV4.2
- net Vexp: now also R?.1; no longer RV5.2, RV5.3, U2.1
- net at Q1.3 (C2), R10.2, U2.2 (-): now also C?.2
- net at R2.1, R3.1, R4.1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: now also R?.2; no longer RV4.1
- net at R7.2, U1.1: now also R?.1; no longer RV4.2, RV4.3
- new net: C?.1, R?.2, RV5.2, RV5.3, U2.1
- new net: R?.2, RV4.1
- new net: R?.1, RV4.3
- new net: R?.1, R?.2 (x3)
Other:
- note added: "+100mV"
- note added: "+1V"
- note added: "-100mV"
- note added: "-1V"
- note added: "0V"
- note removed: "5V"
- moved on the sheet: R2, R3, R4, R5, R6, R7, RV3, RV4, U1A, U1B, U1C

Commit message: Refactor VCO
Parts:
- removed C3, C6: 1n, Capacitor_THT:C_Disc_D7.0mm_W2.5mm_P5.00mm, symbol Device:C
- removed C4, C5, C7: 100n, Capacitor_SMD:C_0805_2012Metric_Pad1.15x1.40mm_HandSolder, symbol Device:C
- removed C?: 220p, Capacitor_THT:C_Disc_D7.0mm_W2.5mm_P5.00mm, symbol Device:C
- removed Q1: MMDT3904, Package_TO_SOT_SMD:SOT-363_SC-70-6, symbol Transistor_BJT:MMDT3904
- removed Q2, Q4, Q5: BC547, Package_TO_SOT_THT:TO-92_Inline_Wide, symbol Transistor_BJT:BC547
- removed R10: 22k, Resistor_THT:R_Axial_DIN0204_L3.6mm_D1.6mm_P7.62mm_Horizontal, symbol Device:R
- removed R11, R15, R16, R17, R19, R2, R22, R23, R3, R4, R? (x3): 100k, Resistor_THT:R_Axial_DIN0204_L3.6mm_D1.6mm_P7.62mm_Horizontal, symbol Device:R
- removed R12, R13, R14: 56k, Resistor_THT:R_Axial_DIN0204_L3.6mm_D1.6mm_P7.62mm_Horizontal, symbol Device:R
- removed R20, R21, R24, R25, R5: 47k, Resistor_THT:R_Axial_DIN0204_L3.6mm_D1.6mm_P7.62mm_Horizontal, symbol Device:R
- removed R6: 4k7, Resistor_THT:R_Axial_DIN0204_L3.6mm_D1.6mm_P7.62mm_Horizontal, symbol Device:R
- removed R7, R?: 0, Resistor_THT:R_Axial_DIN0204_L3.6mm_D1.6mm_P7.62mm_Horizontal, symbol Device:R
- removed R8: 1M, Resistor_THT:R_Axial_DIN0204_L3.6mm_D1.6mm_P7.62mm_Horizontal, symbol Device:R
- removed R9: 1k, Resistor_THT:R_Axial_DIN0204_L3.6mm_D1.6mm_P7.62mm_Horizontal, symbol Device:R
- removed R?: 220k, Resistor_THT:R_Axial_DIN0204_L3.6mm_D1.6mm_P7.62mm_Horizontal, symbol Device:R
- removed R?: 1k8, Resistor_THT:R_Axial_DIN0204_L3.6mm_D1.6mm_P7.62mm_Horizontal, symbol Device:R
- removed R? (x2): 560k, Resistor_THT:R_Axial_DIN0204_L3.6mm_D1.6mm_P7.62mm_Horizontal, symbol Device:R
- removed R? (x2): 27k, Resistor_THT:R_Axial_DIN0204_L3.6mm_D1.6mm_P7.62mm_Horizontal, symbol Device:R
- removed RV3: 100k, Potentiometer_THT:Potentiometer_Piher_T-16L_Single_Vertical_Hole, symbol Device:R_POT
- removed RV4, RV5: 10k, Potentiometer_THT:Potentiometer_Bourns_3299W_Vertical, symbol Device:R_POT_TRIM
- removed RV6: 220k, telec:Potentiometer_P3.81mmx5.12mm_Vertical, symbol Device:R_POT_TRIM
- removed U1, U2, U3, U4, U5: TL082, Package_DIP:DIP-8_W7.62mm_LongPads, symbol Amplifier_Operational:TL082
- added C?: 100n, Capacitor_SMD:C_0805_2012Metric_Pad1.15x1.40mm_HandSolder, symbol Device:C
- added R? (x2): 560k, Resistor_THT:R_Axial_DIN0204_L3.6mm_D1.6mm_P7.62mm_Horizontal, symbol Device:R
- added R?: 100k, Resistor_THT:R_Axial_DIN0204_L3.6mm_D1.6mm_P7.62mm_Horizontal, symbol Device:R
- added RV?: 100k, Potentiometer_THT:Potentiometer_Bourns_3299W_Vertical, symbol Device:R_POT_TRIM
- added SW?: Octave, symbol Switch:SW_SPDT_MSM
- R? (x2): value 300k -> 100k
Connections:
- net GND: now also C?.2
- net +1V: now reaches R?.2
- net +1V: now also R?.1, R?.1, SW?.1
- net -1V: now reaches R?.1
- net -1V: now also R?.2, R?.2, SW?.3
- new net: R?.1, RV?.3
- new net: R?.2, RV?.1
- new net CVoct: C?.1, SW?.2
- new net CVtrim: RV?.2
Other:
- note removed: "+1V"
- note removed: "-1V"
- note removed: "0V"
- note removed: "CV mix"
- note removed: "Exponentiator"
- note removed: "PWM"
- note removed: "Ramp"
- note removed: "Triangle"
- note removed: "VCO"
- moved on the sheet: J4, J5, J6, J7, R26, R27, R28, R29, R?

Commit message: New PCB
Parts:
- removed R? (x3): 100k, Resistor_THT:R_Axial_DIN0204_L3.6mm_D1.6mm_P7.62mm_Horizontal, symbol Device:R
- removed TP4: ~Triangle, Connector_PinHeader_2.54mm:PinHeader_1x01_P2.54mm_Vertical, symbol Connector:TestPoint
- added C103: 100n, Capacitor_SMD:C_0805_2012Metric_Pad1.15x1.40mm_HandSolder, symbol Device:C
- added D101: Ref, Diode_SMD:D_1206_3216Metric_Pad1.42x1.75mm_HandSolder, symbol Device:D_Zener
- added R101: 4k7, Resistor_SMD:R_1206_3216Metric_Pad1.42x1.75mm_HandSolder, symbol Device:R_Small
- added R105, R106: 100k, Resistor_SMD:R_1206_3216Metric_Pad1.42x1.75mm_HandSolder, symbol Device:R_Small
- added R108: 47k, Resistor_THT:R_Axial_DIN0204_L3.6mm_D1.6mm_P7.62mm_Horizontal, symbol Device:R
- added RV101: 100k, Potentiometer_THT:Potentiometer_Bourns_3296W_Vertical, symbol Device:R_POT_TRIM
- added U101: TL082, Package_SO:SOIC-8_3.9x4.9mm_P1.27mm, symbol Amplifier_Operational:TL082
- J102: renamed from J2; footprint telec:JackHole -> telec:Jack_Hole_Square; symbol Connector:AudioJack3_Switch -> Connector:AudioJack3_SwitchTR
- J103: renamed from J4; footprint telec:JackHole -> telec:Jack_Hole_Square; symbol Connector:AudioJack3_Switch -> Connector:AudioJack3_SwitchTR
- J104: renamed from J5; footprint telec:JackHole -> telec:Jack_Hole_Square; symbol Connector:AudioJack3_Switch -> Connector:AudioJack3_SwitchTR
- J105: renamed from J3; footprint telec:JackHole -> telec:Jack_Hole_Square; symbol Connector:AudioJack3_Switch -> Connector:AudioJack3_SwitchTR
- J106: renamed from J6; footprint telec:JackHole -> telec:Jack_Hole_Square; symbol Connector:AudioJack3_Switch -> Connector:AudioJack3_SwitchTR
- J107: renamed from J7; footprint telec:JackHole -> telec:Jack_Hole_Square; symbol Connector:AudioJack3_Switch -> Connector:AudioJack3_SwitchTR
- R102, R103: renamed from R?; value 560k -> 47k
- RV102: renamed from RV?; value 100k -> 10k; footprint Potentiometer_THT:Potentiometer_Bourns_3299W_Vertical -> Potentiometer_THT:Potentiometer_Bourns_3296W_Vertical
- RV103: renamed from RV2; footprint Potentiometer_THT:Potentiometer_Piher_T-16L_Single_Vertical_Hole -> telec:Potentiometer_Single_Vertical_Hole
- SW101: renamed from SW?; footprint (none) -> telec:Switch_Hole
- gave numbers to parts that had none: 1
- renumbered C1 to C101, C2 to C102, D4 to D102, D3 to D103, D1 to D104, D2 to D105, H1 to H101, H2 to H102, J1 to J101, LOGO1 to LOGO101, R26 to R104, R27 to R107, R28 to R109, R29 to R110, R32 to R111, R30 to R112, R31 to R113, R33 to R114, TP2 to TP101, TP3 to TP102
Connections:
- net +12V: now also R101.1, U101.8 (V+)
- net +1V: now also C103.1, R105.2, U101.1, U101.2 (-)
- net -12V: now also U101.4 (V-)
- net -1V: now also C104.1, R106.1, U101.7
- net CVoct: now also R108.1; no longer C104.1
- net GND: now also C103.2, D101.2 (A), R108.2, RV101.3, U101.5 (+)
- new net: RV101.2, U101.3 (+)
- new net: R105.1, R106.2, U101.6 (-)
- new net: D101.1 (K), R101.2, RV101.1
- no-connect marks 22 -> 16
Other:
- moved on the sheet: C104, R102, R103, RV102, SW101, TP102
