File: VCO/SecondariesWaveforms.sch (KiCad schematic (older format))
At the start: 20 parts

Commit message: New PCB
Parts:
- gave numbers to parts that had none: 16

Commit message: Layout VCO
Connections:
- net GND: now also U502.5 (+); no longer U502.3 (+)
- net PWM: now also U502.1; no longer U502.7
- net PWNlevel: now also U502.2 (-); no longer U502.6 (-)
- net Triangle: now also U502.3 (+); no longer U502.5 (+)
- net ~Triangle: now also U502.7; no longer U502.1
- net at R507.1, R510.2: now also U502.6 (-); no longer U502.2 (-)
Changed lines of the file:
@@
 $Comp
 L Amplifier_Operational:TL082 U?
-U 1 1 5FCBFBA4
+U 2 1 5FCBFBA4
 P 2550 3150
 AR Path="/5FCBFBA4" Ref="U?"  Part="1"
-AR Path="/5FAD0DD3/5FCBFBA4" Ref="U502"  Part="1"
+AR Path="/5FAD0DD3/5FCBFBA4" Ref="U502"  Part="2"
 F 0 "U502" H 2750 2950 50  0000 C CNN
 F 1 "TL082" H 2750 3050 50  0000 C CNN
 F 2 "Package_DIP:DIP-8_W7.62mm_LongPads" H 2550 3150 50  0001 C CNN
 F 3 "http://www.ti.com/lit/ds/symlink/tl081.pdf" H 2550 3150 50  0001 C CNN
-	1    2550 3150
+	2    2550 3150
 	1    0    0    1
 $EndComp
@@
 $Comp
 L Amplifier_Operational:TL082 U?
-U 2 1 5FCC95BB
+U 1 1 5FCC95BB
 P 2550 5000
 AR Path="/5FCC95BB" Ref="U?"  Part="2"
-AR Path="/5FAD0DD3/5FCC95BB" Ref="U502"  Part="2"
+AR Path="/5FAD0DD3/5FCC95BB" Ref="U502"  Part="1"
 F 0 "U502" H 2750 4800 50  0000 C CNN
 F 1 "TL082" H 2750 4900 50  0000 C CNN
 F 2 "Package_DIP:DIP-8_W7.62mm_LongPads" H 2550 5000 50  0001 C CNN
 F 3 "http://www.ti.com/lit/ds/symlink/tl081.pdf" H 2550 5000 50  0001 C CNN
-	2    2550 5000
-	1    0    0    1
-$EndComp
+	1    2550 5000
+	1    0    0    1
+$EndComp

Commit message: Layout VCO done
Parts:
- R501: footprint Resistor_THT:R_Axial_DIN0204_L3.6mm_D1.6mm_P7.62mm_Horizontal -> Resistor_THT:R_Axial_DIN0204_L3.6mm_D1.6mm_P2.54mm_Vertical
Changed lines of the file:
@@
 F 0 "R501" V 2450 1750 50  0000 C CNN
 F 1 "100k" V 2550 1750 50  0000 C CNN
-F 2 "Resistor_THT:R_Axial_DIN0204_L3.6mm_D1.6mm_P7.62mm_Horizontal" V 2480 1750 50  0001 C CNN
+F 2 "Resistor_THT:R_Axial_DIN0204_L3.6mm_D1.6mm_P2.54mm_Vertical" V 2480 1750 50  0001 C CNN
 F 3 "~" H 2550 1750 50  0001 C CNN
 	1    2550 1750
