File: VCO/CVmixer.sch (KiCad schematic (older format))
At the start: 11 parts

Commit message: New PCB
Parts:
- RV301: renamed from RV?; footprint Potentiometer_THT:Potentiometer_Piher_T-16L_Single_Vertical_Hole -> telec:Potentiometer_Single_Vertical_Hole
- gave numbers to parts that had none: 8
Changed lines of the file:
@@
 P 1900 2200
 AR Path="/5FBA3739" Ref="U?"  Part="1"
-AR Path="/5FADAEA0/5FBA3739" Ref="U?"  Part="1"
-F 0 "U?" H 2100 2000 50  0000 C CNN
+AR Path="/5FADAEA0/5FBA3739" Ref="U301"  Part="1"
+F 0 "U301" H 2100 2000 50  0000 C CNN
 F 1 "TL082" H 2100 2100 50  0000 C CNN
 F 2 "Package_DIP:DIP-8_W7.62mm_LongPads" H 1900 2200 50  0001 C CNN
@@
 P 1550 2400
 AR Path="/5FBA3744" Ref="#PWR?"  Part="1"
-AR Path="/5FADAEA0/5FBA3744" Ref="#PWR?"  Part="1"
-F 0 "#PWR?" H 1550 2150 50  0001 C CNN
+AR Path="/5FADAEA0/5FBA3744" Ref="#PWR0303"  Part="1"
+F 0 "#PWR0303" H 1550 2150 50  0001 C CNN
 F 1 "GND" H 1555 2227 50  0000 C CNN
 F 2 "" H 1550 2400 50  0001 C CNN
@@
 P 1200 2100
 AR Path="/5FBA3750" Ref="R?"  Part="1"
-AR Path="/5FADAEA0/5FBA3750" Ref="R?"  Part="1"
-F 0 "R?" V 1300 2100 50  0000 C CNN
+AR Path="/5FADAEA0/5FBA3750" Ref="R302"  Part="1"
+F 0 "R302" V 1300 2100 50  0000 C CNN
 F 1 "100k" V 1200 2100 50  0000 C CNN
 F 2 "Resistor_THT:R_Axial_DIN0204_L3.6mm_D1.6mm_P7.62mm_Horizontal" V 1130 2100 50  0001 C CNN
@@
 P 1200 2300
 AR Path="/5FBA3758" Ref="R?"  Part="1"
-AR Path="/5FADAEA0/5FBA3758" Ref="R?"  Part="1"
-F 0 "R?" V 1300 2300 50  0000 C CNN
+AR Path="/5FADAEA0/5FBA3758" Ref="R304"  Part="1"
+F 0 "R304" V 1300 2300 50  0000 C CNN
 F 1 "100k" V 1200 2300 50  0000 C CNN
 F 2 "Resistor_THT:R_Axial_DIN0204_L3.6mm_D1.6mm_P7.62mm_Horizontal" V 1130 2300 50  0001 C CNN
@@
 P 1200 2500
 AR Path="/5FBA375F" Ref="R?"  Part="1"
-AR Path="/5FADAEA0/5FBA375F" Ref="R?"  Part="1"
-F 0 "R?" V 1300 2500 50  0000 C CNN
+AR Path="/5FADAEA0/5FBA375F" Ref="R305"  Part="1"
+F 0 "R305" V 1300 2500 50  0000 C CNN
 F 1 "100k" V 1200 2500 50  0000 C CNN
 F 2 "Resistor_THT:R_Axial_DIN0204_L3.6mm_D1.6mm_P7.62mm_Horizontal" V 1130 2500 50  0001 C CNN
@@
 P 2700 2200
 AR Path="/5FBA376F" Ref="R?"  Part="1"
-AR Path="/5FADAEA0/5FBA376F" Ref="R?"  Part="1"
-F 0 "R?" V 2800 2200 50  0000 C CNN
+AR Path="/5FADAEA0/5FBA376F" Ref="R303"  Part="1"
+F 0 "R303" V 2800 2200 50  0000 C CNN
 F 1 "0" V 2700 2200 50  0000 C CNN
 F 2 "Resistor_THT:R_Axial_DIN0204_L3.6mm_D1.6mm_P7.62mm_Horizontal" V 2630 2200 50  0001 C CNN
@@
 P 1350 3250
 AR Path="/5FBA3778" Ref="R?"  Part="1"
-AR Path="/5FADAEA0/5FBA3778" Ref="R?"  Part="1"
-F 0 "R?" V 1450 3250 50  0000 L CNN
+AR Path="/5FADAEA0/5FBA3778" Ref="R307"  Part="1"
+F 0 "R307" V 1450 3150 50  0000 L CNN
 F 1 "47k" V 1350 3200 50  0000 L CNN
 F 2 "Resistor_THT:R_Axial_DIN0204_L3.6mm_D1.6mm_P7.62mm_Horizontal" V 1280 3250 50  0001 C CNN
@@
 P 1900 3350
 AR Path="/5FBA377F" Ref="U?"  Part="2"
-AR Path="/5FADAEA0/5FBA377F" Ref="U?"  Part="2"
-F 0 "U?" H 1900 3050 50  0000 C CNN
+AR Path="/5FADAEA0/5FBA377F" Ref="U301"  Part="2"
+F 0 "U301" H 1900 3050 50  0000 C CNN
 F 1 "TL082" H 1900 3150 50  0000 C CNN
 F 2 "Package_DIP:DIP-8_W7.62mm_LongPads" H 1900 3350 50  0001 C CNN
@@
 P 1800 2800
 AR Path="/5FBA3786" Ref="RV?"  Part="1"
-AR Path="/5FADAEA0/5FBA3786" Ref="RV?"  Part="1"
-F 0 "RV?" V 1700 2800 50  0000 C CNN
+AR Path="/5FADAEA0/5FBA3786" Ref="RV301"  Part="1"
+F 0 "RV301" V 1700 2800 50  0000 C CNN
 F 1 "100k" V 1800 2800 50  0000 C CNN
-F 2 "Potentiometer_THT:Potentiometer_Piher_T-16L_Single_Vertical_Hole" H 1800 2800 50  0001 C CNN
+F 2 "telec:Potentiometer_Single_Vertical_Hole" H 1800 2800 50  0001 C CNN
 F 3 "~" H 1800 2800 50  0001 C CNN
 	1    1800 2800
@@
 P 2200 2800
 AR Path="/5FBA3793" Ref="R?"  Part="1"
-AR Path="/5FADAEA0/5FBA3793" Ref="R?"  Part="1"
-F 0 "R?" V 2300 2800 50  0000 L CNN
+AR Path="/5FADAEA0/5FBA3793" Ref="R306"  Part="1"
+F 0 "R306" V 2300 2700 50  0000 L CNN
 F 1 "4k7" V 2200 2750 50  0000 L CNN
 F 2 "Resistor_THT:R_Axial_DIN0204_L3.6mm_D1.6mm_P7.62mm_Horizontal" V 2130 2800 50  0001 C CNN
@@
 P 1050 1150
 AR Path="/5FBA37A3" Ref="U?"  Part="3"
-AR Path="/5FADAEA0/5FBA37A3" Ref="U?"  Part="3"
-F 0 "U?" H 1150 1100 50  0000 C CNN
+AR Path="/5FADAEA0/5FBA37A3" Ref="U301"  Part="3"
+F 0 "U301" H 1150 1100 50  0000 C CNN
 F 1 "TL082" H 1150 1200 50  0000 C CNN
 F 2 "Package_DIP:DIP-8_W7.62mm_LongPads" H 1050 1150 50  0001 C CNN
@@
 P 1150 850
 AR Path="/5FBA37A9" Ref="#PWR?"  Part="1"
-AR Path="/5FADAEA0/5FBA37A9" Ref="#PWR?"  Part="1"
-F 0 "#PWR?" H 1150 700 50  0001 C CNN
+AR Path="/5FADAEA0/5FBA37A9" Ref="#PWR0301"  Part="1"
+F 0 "#PWR0301" H 1150 700 50  0001 C CNN
 F 1 "+12V" H 1165 1023 50  0000 C CNN
 F 2 "" H 1150 850 50  0001 C CNN
@@
 P 1150 1450
 AR Path="/5FBA37AF" Ref="#PWR?"  Part="1"
-AR Path="/5FADAEA0/5FBA37AF" Ref="#PWR?"  Part="1"
-F 0 "#PWR?" H 1150 1550 50  0001 C CNN
+AR Path="/5FADAEA0/5FBA37AF" Ref="#PWR0302"  Part="1"
+F 0 "#PWR0302" H 1150 1550 50  0001 C CNN
 F 1 "-12V" H 1165 1623 50  0000 C CNN
 F 2 "" H 1150 1450 50  0001 C CNN
@@
 P 1850 1800
 AR Path="/5FBA37B5" Ref="R?"  Part="1"
-AR Path="/5FADAEA0/5FBA37B5" Ref="R?"  Part="1"
-F 0 "R?" V 1950 1800 50  0000 C CNN
+AR Path="/5FADAEA0/5FBA37B5" Ref="R301"  Part="1"
+F 0 "R301" V 1950 1800 50  0000 C CNN
 F 1 "1k8" V 1850 1800 50  0000 C CNN
 F 2 "Resistor_THT:R_Axial_DIN0204_L3.6mm_D1.6mm_P7.62mm_Horizontal" V 1780 1800 50  0001 C CNN

Commit message: VCO done
Parts:
- removed R303: 0, Resistor_THT:R_Axial_DIN0204_L3.6mm_D1.6mm_P7.62mm_Horizontal, symbol Device:R
Connections:
- net CV: now also R301.1, U301.1
Other:
- note added: "Multiply by 0.018 for the next stage:\n5V -> 90mV"
- note added: "Offset is also affected by the gain,\nnot really great"
Changed lines of the file:
@@
 	1450 2100 1350 2100
 Connection ~ 1450 2100
-Wire Wire Line
-	2850 2200 2950 2200
 $Comp
 L Device:R R?
@@
 Wire Wire Line
 	1050 2100 900  2100
-$Comp
-L Device:R R?
-U 1 1 5FBA376F
-P 2700 2200
-AR Path="/5FBA376F" Ref="R?"  Part="1"
-AR Path="/5FADAEA0/5FBA376F" Ref="R303"  Part="1"
-F 0 "R303" V 2800 2200 50  0000 C CNN
-F 1 "0" V 2700 2200 50  0000 C CNN
-F 2 "Resistor_THT:R_Axial_DIN0204_L3.6mm_D1.6mm_P7.62mm_Horizontal" V 2630 2200 50  0001 C CNN
-F 3 "~" H 2700 2200 50  0001 C CNN
-	1    2700 2200
-	0    1    -1   0
-$EndComp
-Wire Wire Line
-	2550 2200 2450 2200
 Connection ~ 2450 2200
 $Comp
@@
 Text HLabel 900  2500 0    50   Input ~ 0
 CV3
+Wire Wire Line
+	2450 2200 2950 2200
+Text Notes 1350 3750 0    50   ~ 0
+Offset is also affected by the gain,\nnot really great
+Text Notes 2650 1900 0    50   ~ 0
+Multiply by 0.018 for the next stage:\n5V -> 90mV
 $EndSCHEMATC
