File: Glider/Glider.sch (KiCad schematic (older format))
At the start: 38 parts, among them J1 EuroPower, J2 OUT, J3 IN, J4 OUT, J5 IN, SW1 LIN/LOG, SW2 UP/DOWN, SW3 LIN/LOG, SW4 UP/DOWN, U1 TL082, U2 TL082

Commit message: Glider done !
Parts:
- removed D5, D6, D7, D8: LED, LED_SMD:LED_1206_3216Metric_Castellated, symbol Device:LED
- removed R5, R6, R7, R8: 1k, Resistor_SMD:R_1206_3216Metric_Pad1.42x1.75mm_HandSolder, symbol Device:R
- added D4: LED, LED_SMD:LED_1206_3216Metric_ReverseMount_Hole1.8x2.4mm, symbol Device:LED
- added R4: 2k2, Resistor_SMD:R_1206_3216Metric_Pad1.42x1.75mm_HandSolder, symbol Device:R
- J2: value OUT -> OUT1
- J3: value IN -> IN1
- J4: value OUT -> OUT2
- J5: value IN -> IN2
- LOGO1: footprint logo:telec-32 -> logo:telec-8
- R1: renamed from R9; value 1k -> 2k2
- RV1, RV2: footprint Potentiometer_THT:Potentiometer_Piher_T-16L_Single_Vertical_Hole -> Potentiometer_THT:Potentiometer_Alps_RK09K_Single_Vertical
- SW1, SW2, SW3, SW4: footprint (none) -> telec:SW_L13.2mm_W7.9mm_P4.7mm
- renumbered D9 to D1, D1 to D2, D2 to D3, D3 to D5, D4 to D6, R1 to R2, R2 to R3, R3 to R5, R4 to R6
Connections:
- net Clk is gone; now on net OUT1: R1.1
- net GND: now also D4.1 (K)
- net IN1: now reaches J3.T, U1.3 (+)
- net at C3.2, RV1.1, SW1.1 (A)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: now also D2.1 (K), D3.2 (A); no longer D2.2 (A), D3.1 (K)
- net at SW2.1: now also D2.2 (A); no longer D2.1 (K)
- net at SW2.3: now also D3.1 (K); no longer D3.2 (A)
- net IN2: now reaches J5.T, U2.3 (+)
- net OUT2: now reaches R5.2, U2.7
- net OUT2: now also R4.1
- net at C4.2, RV2.1, SW3.1 (A)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: now also D5.1 (K), D6.2 (A); no longer D5.2 (A), D6.1 (K)
- net at SW4.1: now also D5.2 (A); no longer D5.1 (K)
- net at SW4.3: now also D6.1 (K); no longer D6.2 (A)
- net OUT1: now reaches R2.2, U1.7
- new net: D4.2 (A), R4.2
Other:
- note added: "From Harald Antes schematic,\nfrom Ives Uson"
- moved on the sheet: C3, C4, D1, D2, D3, D5, D6, J2, J3, J4, J5, R1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

Commit message: Changed pot direction
Connections:
- net at C3.2, D2.1 (K), D3.2 (A)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: now also RV1.2
- net at R3.2, RV1.3, SW2.2: no longer RV1.2
- net at C4.2, D5.1 (K), D6.2 (A)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: now also RV2.2
- net at R6.2, RV2.3, SW4.2: no longer RV2.2
Changed lines of the file:
@@
 Front Panel
-$Comp
-L Device:R_POT RV1
-U 1 1 5F360F90
-P 4350 2900
-F 0 "RV1" V 4250 2950 50  0000 R CNN
-F 1 "1M" V 4350 2950 50  0000 R CNN
-F 2 "Potentiometer_THT:Potentiometer_Alps_RK09K_Single_Vertical" H 4350 2900 50  0001 C CNN
-F 3 "~" H 4350 2900 50  0001 C CNN
-	1    4350 2900
-	0    1    1    0
-$EndComp
 $Comp
 L Diode:1N4148 D2
@@
 	3350 2900 3400 2900
 Wire Wire Line
-	4350 3050 4150 3050
-Wire Wire Line
-	4150 3050 4150 2900
-Connection ~ 4150 2900
-Wire Wire Line
-	4150 2900 4200 2900
+	4350 3050 4550 3050
+Wire Wire Line
+	4550 3050 4550 2900
 Wire Wire Line
 	2750 2800 2650 2800
@@
 	4750 2400 4750 2750
 Wire Wire Line
-	4500 2900 4750 2900
+	4500 2900 4550 2900
 Connection ~ 4750 2900
 Wire Wire Line
@@
 	3750 2900 3850 2900
 Connection ~ 3850 2900
-Wire Wire Line
-	3850 2900 4150 2900
 $Comp
 L Device:C C3
@@
 $EndComp
 $Comp
-L Device:R_POT RV2
-U 1 1 5FE8ECA1
-P 4350 4850
-F 0 "RV2" V 4250 4900 50  0000 R CNN
-F 1 "1M" V 4350 4900 50  0000 R CNN
-F 2 "Potentiometer_THT:Potentiometer_Alps_RK09K_Single_Vertical" H 4350 4850 50  0001 C CNN
-F 3 "~" H 4350 4850 50  0001 C CNN
-	1    4350 4850
-	0    1    1    0
-$EndComp
-$Comp
 L Diode:1N4148 D5
 U 1 1 5FE8ECA7
@@
 	3350 4850 3400 4850
 Wire Wire Line
-	4350 5000 4150 5000
-Wire Wire Line
-	4150 5000 4150 4850
-Connection ~ 4150 4850
-Wire Wire Line
-	4150 4850 4200 4850
+	4350 5000 4550 5000
+Wire Wire Line
+	4550 5000 4550 4850
 Wire Wire Line
 	2750 4750 2650 4750
@@
 	4750 4350 4750 4700
 Wire Wire Line
-	4500 4850 4750 4850
+	4500 4850 4550 4850
 Connection ~ 4750 4850
 Wire Wire Line
@@
 	3750 4850 3850 4850
 Connection ~ 3850 4850
-Wire Wire Line
-	3850 4850 4150 4850
 $Comp
 L Device:C C4
@@
 Text Notes 7050 6950 0    50   ~ 0
 From Harald Antes schematic,\nfrom Ives Uson
+$Comp
+L Device:R_POT RV2
+U 1 1 5FE8ECA1
+P 4350 4850
+F 0 "RV2" V 4250 4900 50  0000 R CNN
+F 1 "1M" V 4350 4900 50  0000 R CNN
+F 2 "Potentiometer_THT:Potentiometer_Alps_RK09K_Single_Vertical" H 4350 4850 50  0001 C CNN
+F 3 "~" H 4350 4850 50  0001 C CNN
+	1    4350 4850
+	0    1    1    0
+$EndComp
+$Comp
+L Device:R_POT RV1
+U 1 1 5F360F90
+P 4350 2900
+F 0 "RV1" V 4250 2950 50  0000 R CNN
+F 1 "1M" V 4350 2950 50  0000 R CNN
+F 2 "Potentiometer_THT:Potentiometer_Alps_RK09K_Single_Vertical" H 4350 2900 50  0001 C CNN
+F 3 "~" H 4350 2900 50  0001 C CNN
+	1    4350 2900
+	0    1    1    0
+$EndComp
+Connection ~ 4550 2900
+Wire Wire Line
+	4550 2900 4750 2900
+Wire Wire Line
+	3850 2900 4200 2900
+Connection ~ 4550 4850
+Wire Wire Line
+	4550 4850 4750 4850
+Wire Wire Line
+	3850 4850 4200 4850
 $EndSCHEMATC

Commit message: Analog modules finished
Connections:
- net at C3.2, RV1.1, RV1.2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: now also D2.2 (A), D3.1 (K); no longer D2.1 (K), D3.2 (A)
- net at SW2.1: now also D2.1 (K); no longer D2.2 (A)
- net at SW2.3: now also D3.2 (A); no longer D3.1 (K)
- net at C4.2, RV2.1, RV2.2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: now also D5.2 (A), D6.1 (K); no longer D5.1 (K), D6.2 (A)
- net at SW4.1: now also D5.1 (K); no longer D5.2 (A)
- net at SW4.3: now also D6.2 (A); no longer D6.1 (K)
Changed lines of the file:
@@
 F 3 "https://assets.nexperia.com/documents/data-sheet/1N4148_1N4448.pdf" H 4550 2200 50  0001 C CNN
 	1    4550 2200
-	-1   0    0    -1
+	1    0    0    -1
 $EndComp
 $Comp
@@
 F 3 "https://assets.nexperia.com/documents/data-sheet/1N4148_1N4448.pdf" H 4550 2400 50  0001 C CNN
 	1    4550 2400
-	1    0    0    1
+	-1   0    0    1
 $EndComp
 $Comp
@@
 F 3 "https://assets.nexperia.com/documents/data-sheet/1N4148_1N4448.pdf" H 4550 4150 50  0001 C CNN
 	1    4550 4150
-	-1   0    0    -1
+	1    0    0    -1
 $EndComp
 $Comp
@@
 F 3 "https://assets.nexperia.com/documents/data-sheet/1N4148_1N4448.pdf" H 4550 4350 50  0001 C CNN
 	1    4550 4350
-	1    0    0    1
-$EndComp
-$Comp
+	-1   0    0    1
+$EndComp
+$Comp

Commit message: updated footprints on Glider
Parts:
- J2, J3, J4, J5: footprint telec:JackHole -> telec:Jack_Hole_Square; symbol Connector:AudioJack3_Switch -> Connector:AudioJack3_SwitchTR
Connections:
- no-connect marks 14 -> 10
Changed lines of the file:
@@
 $EndComp
 $Comp
-L Connector:AudioJack3_Switch J3
+L Connector:AudioJack3_SwitchTR J3
 U 1 1 5F0BD040
 P 1850 2800
 F 0 "J3" H 1832 3225 50  0000 C CNN
 F 1 "IN1" H 1832 3134 50  0000 C CNN
-F 2 "telec:JackHole" H 1850 2800 50  0001 C CNN
+F 2 "telec:Jack_Hole_Square" H 1850 2800 50  0001 C CNN
 F 3 "~" H 1850 2800 50  0001 C CNN
 	1    1850 2800
@@
 	2200 1350 2200 1450
 $Comp
-L Connector:AudioJack3_Switch J2
+L Connector:AudioJack3_SwitchTR J2
 U 1 1 5F4208DD
 P 7150 2650
 F 0 "J2" H 7132 3075 50  0000 C CNN
 F 1 "OUT1" H 7132 2984 50  0000 C CNN
-F 2 "telec:JackHole" H 7150 2650 50  0001 C CNN
+F 2 "telec:Jack_Hole_Square" H 7150 2650 50  0001 C CNN
 F 3 "~" H 7150 2650 50  0001 C CNN
 	1    7150 2650
@@
 NoConn ~ 6950 2750
 NoConn ~ 6950 2650
-NoConn ~ 6950 2550
 NoConn ~ 6950 2950
 $Comp
 L power:GND #PWR012
 U 1 1 5F62EF49
-P 6950 2450
-F 0 "#PWR012" H 6950 2200 50  0001 C CNN
-F 1 "GND" V 6955 2322 50  0000 R CNN
-F 2 "" H 6950 2450 50  0001 C CNN
-F 3 "" H 6950 2450 50  0001 C CNN
-	1    6950 2450
+P 6950 2550
+F 0 "#PWR012" H 6950 2300 50  0001 C CNN
+F 1 "GND" V 6955 2422 50  0000 R CNN
+F 2 "" H 6950 2550 50  0001 C CNN
+F 3 "" H 6950 2550 50  0001 C CNN
+	1    6950 2550
 	0    1    1    0
 $EndComp
 NoConn ~ 2050 2900
-NoConn ~ 2050 2800
-NoConn ~ 2050 2700
 $Comp
 L power:GND #PWR014
 U 1 1 5F63005B
-P 2050 2600
-F 0 "#PWR014" H 2050 2350 50  0001 C CNN
-F 1 "GND" V 2055 2472 50  0000 R CNN
-F 2 "" H 2050 2600 50  0001 C CNN
-F 3 "" H 2050 2600 50  0001 C CNN
-	1    2050 2600
+P 2050 2700
+F 0 "#PWR014" H 2050 2450 50  0001 C CNN
+F 1 "GND" V 2055 2572 50  0000 R CNN
+F 2 "" H 2050 2700 50  0001 C CNN
+F 3 "" H 2050 2700 50  0001 C CNN
+	1    2050 2700
 	0    -1   1    0
 $EndComp
@@
 	2650 2250 2650 2800
 $Comp
-L Connector:AudioJack3_Switch J5
-U 1 1 5FE8EC60
-P 1850 4750
-F 0 "J5" H 1832 5175 50  0000 C CNN
-F 1 "IN2" H 1832 5084 50  0000 C CNN
-F 2 "telec:JackHole" H 1850 4750 50  0001 C CNN
-F 3 "~" H 1850 4750 50  0001 C CNN
-	1    1850 4750
-	1    0    0    -1
-$EndComp
-$Comp
-L Connector:AudioJack3_Switch J4
+L Connector:AudioJack3_SwitchTR J4
 U 1 1 5FE8EC66
 P 7150 4600
 F 0 "J4" H 7132 5025 50  0000 C CNN
 F 1 "OUT2" H 7132 4934 50  0000 C CNN
-F 2 "telec:JackHole" H 7150 4600 50  0001 C CNN
+F 2 "telec:Jack_Hole_Square" H 7150 4600 50  0001 C CNN
 F 3 "~" H 7150 4600 50  0001 C CNN
 	1    7150 4600
@@
 NoConn ~ 6950 4700
 NoConn ~ 6950 4600
-NoConn ~ 6950 4500
 NoConn ~ 6950 4900
 $Comp
 L power:GND #PWR020
 U 1 1 5FE8EC70
-P 6950 4400
-F 0 "#PWR020" H 6950 4150 50  0001 C CNN
-F 1 "GND" V 6955 4272 50  0000 R CNN
-F 2 "" H 6950 4400 50  0001 C CNN
-F 3 "" H 6950 4400 50  0001 C CNN
-	1    6950 4400
+P 6950 4500
+F 0 "#PWR020" H 6950 4250 50  0001 C CNN
+F 1 "GND" V 6955 4372 50  0000 R CNN
+F 2 "" H 6950 4500 50  0001 C CNN
+F 3 "" H 6950 4500 50  0001 C CNN
+	1    6950 4500
 	0    1    1    0
 $EndComp
 NoConn ~ 2050 4850
-NoConn ~ 2050 4750
-NoConn ~ 2050 4650
 $Comp
 L power:GND #PWR021
 U 1 1 5FE8EC79
-P 2050 4550
-F 0 "#PWR021" H 2050 4300 50  0001 C CNN
-F 1 "GND" V 2055 4422 50  0000 R CNN
-F 2 "" H 2050 4550 50  0001 C CNN
-F 3 "" H 2050 4550 50  0001 C CNN
-	1    2050 4550
+P 2050 4650
+F 0 "#PWR021" H 2050 4400 50  0001 C CNN
+F 1 "GND" V 2055 4522 50  0000 R CNN
+F 2 "" H 2050 4650 50  0001 C CNN
+F 3 "" H 2050 4650 50  0001 C CNN
+	1    2050 4650
 	0    -1   1    0
 $EndComp
@@
 Wire Wire Line
 	3850 4850 4200 4850
+$Comp
+L Connector:AudioJack3_SwitchTR J5
+U 1 1 5FE8EC60
+P 1850 4750
+F 0 "J5" H 1832 5175 50  0000 C CNN
+F 1 "IN2" H 1832 5084 50  0000 C CNN
+F 2 "telec:Jack_Hole_Square" H 1850 4750 50  0001 C CNN
+F 3 "~" H 1850 4750 50  0001 C CNN
+	1    1850 4750
+	1    0    0    -1
+$EndComp
+NoConn ~ 2050 4750
+NoConn ~ 2050 2800
 $EndSCHEMATC
