File: Quantizer/Quantizer.sch (KiCad schematic (older format))
At the start: 42 parts, among them J1 EuroPower, J2 CV, J3 Gate, J4 Clock, Q1 BC557, Q2 BC547, SW1 Reset, U1 L7805, U2 TL082

Commit message: Quantizer...
Parts:
- removed Q1: BC557, Package_TO_SOT_THT:TO-92_Inline_Wide, symbol Transistor_BJT:BC557
- removed Q2: BC547, Package_TO_SOT_THT:TO-92_Inline_Wide, symbol Transistor_BJT:BC547
- removed R3, R4, R6: 10k, Resistor_THT:R_Axial_DIN0204_L3.6mm_D1.6mm_P7.62mm_Horizontal, symbol Device:R
- removed RV1: R_POT_Small, Potentiometer_THT:Potentiometer_Bourns_3339P_Vertical, symbol Device:R_POT_Small
- removed RV3: R_POT_TRIM, Potentiometer_THT:Potentiometer_Bourns_3299W_Vertical, symbol Device:R_POT_TRIM
- added D? (x3): 1N4148, Diode_THT:D_DO-35_SOD27_P7.62mm_Horizontal, symbol Diode:1N4148
- added J?: Prog, symbol Connector:Conn_01x03_Female
- added J?: IN2, telec:JackHole, symbol Connector:AudioJack3_Switch
- added R?: 100k, Resistor_THT:R_Axial_DIN0204_L3.6mm_D1.6mm_P7.62mm_Horizontal, symbol Device:R
- added RV?: 100k, Potentiometer_THT:Potentiometer_Piher_T-16L_Single_Vertical_Hole, symbol Device:R_POT
- added U?: MCP4801, symbol Analog_DAC:MCP4801
- J4: value Clock -> IN1
- RV2: value R_POT -> 100k
Connections:
- net labels added: IN1, IN2, Mode1, Mode2, UPDI
- wire segments 51 -> 57
- no-connect marks 11 -> 14
Other:
- moved on the sheet: C4, C5, D1, J4, R5, RV2, U2C

Commit message: Quantizer layout done!
Parts:
- removed C6: 10n, Capacitor_THT:C_Disc_D7.0mm_W2.5mm_P5.00mm, symbol Device:C
- removed D2, D3, D4, D5: LED, LED_SMD:LED_1206_3216Metric_Castellated, symbol Device:LED
- removed D6: LED, LED_SMD:LED_1206_3216Metric_ReverseMount_Hole1.8x2.4mm, symbol Device:LED
- removed H3, H4: Mounting_Holes, Kosmo_panel:Kosmo_Panel_Dual_Mounting_Holes, symbol Kosmo:Mounting_Holes
- removed J?: Prog, symbol Connector:Conn_01x03_Female
- removed R10, R11, R7, R8, R9: 1k, Resistor_SMD:R_1206_3216Metric_Pad1.42x1.75mm_HandSolder, symbol Device:R
- removed R12: 10k, Resistor_THT:R_Axial_DIN0204_L3.6mm_D1.6mm_P7.62mm_Horizontal, symbol Device:R
- removed SW1: Reset, Button_Switch_THT:SW_PUSH_6mm, symbol Switch:SW_SPST
- added C4, C5: 100n, Capacitor_SMD:C_1206_3216Metric_Pad1.42x1.75mm_HandSolder, symbol Device:C
- added D5, D6: 1N4148, Diode_SMD:D_1206_3216Metric_Pad1.42x1.75mm_HandSolder, symbol Diode:1N4148
- added J2: Prog, TestPoint:TestPoint_Pad_D2.5mm, symbol Connector:Conn_01x01_Female
- added J5: IN3, telec:JackHole, symbol Connector:AudioJack3_Switch
- added J8: OUT3, telec:JackHole, symbol Connector:AudioJack3_Switch
- added R3: 100k, Resistor_SMD:R_1206_3216Metric_Pad1.42x1.75mm_HandSolder, symbol Device:R
- added R6: 1k, Resistor_SMD:R_1206_3216Metric_Pad1.42x1.75mm_HandSolder, symbol Device:R
- added unit 1 of U2
- added unit 3 of U2
- added unit 1 of U3
- added unit 3 of U3
- added unit 2 of U4
- added unit 1 of U4
- added U7: MCP4801, Package_DIP:DIP-8_W7.62mm, symbol Analog_DAC:MCP4801
- C1, C2: footprint Capacitor_THT:CP_Radial_D8.0mm_P3.80mm -> Capacitor_THT:CP_Radial_D4.0mm_P1.50mm
- C3: footprint Capacitor_THT:C_Disc_D7.0mm_W2.5mm_P5.00mm -> Capacitor_SMD:C_1206_3216Metric_Pad1.42x1.75mm_HandSolder
- C6: renamed from C4; footprint Capacitor_THT:C_Disc_D7.0mm_W2.5mm_P5.00mm -> Capacitor_SMD:C_1206_3216Metric_Pad1.42x1.75mm_HandSolder
- C7: renamed from C5; footprint Capacitor_THT:C_Disc_D7.0mm_W2.5mm_P5.00mm -> Capacitor_SMD:C_1206_3216Metric_Pad1.42x1.75mm_HandSolder
- D1: footprint Diode_THT:D_DO-35_SOD27_P7.62mm_Horizontal -> Diode_SMD:D_1206_3216Metric_Pad1.42x1.75mm_HandSolder
- D2, D3, D4: renamed from D?; footprint Diode_THT:D_DO-35_SOD27_P7.62mm_Horizontal -> Diode_SMD:D_1206_3216Metric_Pad1.42x1.75mm_HandSolder
- J6: renamed from J2; value CV -> OUT1
- J7: renamed from J3; value Gate -> OUT2
- LOGO1: footprint logo:telec-32 -> logo:telec-8
- R1: renamed from R5; footprint Resistor_THT:R_Axial_DIN0204_L3.6mm_D1.6mm_P7.62mm_Horizontal -> Resistor_SMD:R_1206_3216Metric_Pad1.42x1.75mm_HandSolder
- R2: renamed from R?; footprint Resistor_THT:R_Axial_DIN0204_L3.6mm_D1.6mm_P7.62mm_Horizontal -> Resistor_SMD:R_1206_3216Metric_Pad1.42x1.75mm_HandSolder
- R4: renamed from R1; footprint Resistor_THT:R_Axial_DIN0204_L3.6mm_D1.6mm_P7.62mm_Horizontal -> Resistor_SMD:R_1206_3216Metric_Pad1.42x1.75mm_HandSolder
- R5: renamed from R2; footprint Resistor_THT:R_Axial_DIN0204_L3.6mm_D1.6mm_P7.62mm_Horizontal -> Resistor_SMD:R_1206_3216Metric_Pad1.42x1.75mm_HandSolder
- RV1: renamed from RV2; footprint Potentiometer_THT:Potentiometer_Piher_T-16L_Single_Vertical_Hole -> Potentiometer_THT:Potentiometer_Alps_RK09K_Single_Vertical
- RV2: renamed from RV?; footprint Potentiometer_THT:Potentiometer_Piher_T-16L_Single_Vertical_Hole -> Potentiometer_THT:Potentiometer_Alps_RK09K_Single_Vertical
- U1: footprint Package_TO_SOT_THT:TO-220-3_Horizontal_TabDown -> Package_TO_SOT_THT:TO-220-3_Vertical
- U2: footprint Package_DIP:DIP-8_W7.62mm_LongPads -> Package_SO:SOIC-8_3.9x4.9mm_P1.27mm
- U3, U4: renamed from U2; footprint Package_DIP:DIP-8_W7.62mm_LongPads -> Package_SO:SOIC-8_3.9x4.9mm_P1.27mm
- U6: renamed from U?; footprint (none) -> Package_DIP:DIP-8_W7.62mm
- gave numbers to parts that had none: 2
- renumbered J4 to J3
Connections:
- net labels added: DAC0, IN3, MOSI, SCK, ~CS1, ~CS2, ~LDAC
- net labels removed: Clk, Rst
- wire segments 57 -> 97
- no-connect marks 14 -> 27
Other:
- moved on the sheet: C1, C2, C6, C7, D1, D2, D3, D4, J1, J3, J4, J7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

Commit message: Quantizer done!
Parts:
- added C8, C9: 100n, Capacitor_SMD:C_1206_3216Metric_Pad1.42x1.75mm_HandSolder, symbol Device:C
- added SW1: Bank, Connector_PinHeader_2.54mm:PinHeader_1x03_P2.54mm_Vertical, symbol Switch:SW_SPDT
Connections:
- net GND: now also C8.1, C9.1, SW1.3 (C)
- net at U3.5 (+), U7.8 (Vout): now also C9.2
- net at U2.5 (+), U6.8 (Vout): now also C8.2
- net at U5.9 (PB2): now also SW1.2 (B)
Changed lines of the file:
@@
 	1850 5250 1850 5150
 Wire Wire Line
-	8750 2350 9150 2350
+	8750 2350 8900 2350
 $Comp
 L power:+5V #PWR037
@@
 $EndComp
 Wire Wire Line
-	8750 3650 9150 3650
+	8750 3650 8900 3650
 Wire Wire Line
 	4850 4000 4500 4000
@@
 	6050 4400 6400 4400
 NoConn ~ 6050 4200
-NoConn ~ 6050 4100
 NoConn ~ 6050 3500
 NoConn ~ 6050 3400
@@
 $EndComp
 $Comp
-L power:+5V #PWR?
+L power:+5V #PWR0106
 U 1 1 642BACD9
 P 5450 900
-F 0 "#PWR?" H 5450 750 50  0001 C CNN
+F 0 "#PWR0106" H 5450 750 50  0001 C CNN
 F 1 "+5V" H 5465 1073 50  0000 C CNN
 F 2 "" H 5450 900 50  0001 C CNN
@@
 $EndComp
 $Comp
-L power:GND #PWR?
+L power:GND #PWR0107
 U 1 1 642BACE6
 P 5450 1200
-AR Path="/642BACE6" Ref="#PWR?"  Part="1"
+AR Path="/642BACE6" Ref="#PWR0107"  Part="1"
 AR Path="/5F345A0C/642BACE6" Ref="#PWR?"  Part="1"
-F 0 "#PWR?" H 5450 950 50  0001 C CNN
+F 0 "#PWR0107" H 5450 950 50  0001 C CNN
 F 1 "GND" H 5455 1027 50  0000 C CNN
 F 2 "" H 5450 1200 50  0001 C CNN
@@
 $EndComp
 $Comp
-L power:+5V #PWR?
+L power:+5V #PWR0108
 U 1 1 64306F8B
 P 7600 850
-F 0 "#PWR?" H 7600 700 50  0001 C CNN
+F 0 "#PWR0108" H 7600 700 50  0001 C CNN
 F 1 "+5V" H 7615 1023 50  0000 C CNN
 F 2 "" H 7600 850 50  0001 C CNN
@@
 $EndComp
 $Comp
-L power:GND #PWR?
+L power:GND #PWR0109
 U 1 1 64306F97
 P 7600 1150
-AR Path="/64306F97" Ref="#PWR?"  Part="1"
+AR Path="/64306F97" Ref="#PWR0109"  Part="1"
 AR Path="/5F345A0C/64306F97" Ref="#PWR?"  Part="1"
-F 0 "#PWR?" H 7600 900 50  0001 C CNN
+F 0 "#PWR0109" H 7600 900 50  0001 C CNN
 F 1 "GND" H 7605 977 50  0000 C CNN
 F 2 "" H 7600 1150 50  0001 C CNN
@@
 $EndComp
 $Comp
-L power:+5V #PWR?
+L power:+5V #PWR0110
 U 1 1 64341828
 P 8100 850
-F 0 "#PWR?" H 8100 700 50  0001 C CNN
+F 0 "#PWR0110" H 8100 700 50  0001 C CNN
 F 1 "+5V" H 8115 1023 50  0000 C CNN
 F 2 "" H 8100 850 50  0001 C CNN
@@
 $EndComp
 $Comp
-L power:GND #PWR?
+L power:GND #PWR0111
 U 1 1 64341834
 P 8100 1150
-AR Path="/64341834" Ref="#PWR?"  Part="1"
+AR Path="/64341834" Ref="#PWR0111"  Part="1"
 AR Path="/5F345A0C/64341834" Ref="#PWR?"  Part="1"
-F 0 "#PWR?" H 8100 900 50  0001 C CNN
+F 0 "#PWR0111" H 8100 900 50  0001 C CNN
 F 1 "GND" H 8105 977 50  0000 C CNN
 F 2 "" H 8100 1150 50  0001 C CNN
@@
 	-1   0    0    -1
 $EndComp
+$Comp
+L Device:C C8
+U 1 1 64388CF5
+P 8900 2600
+AR Path="/64388CF5" Ref="C8"  Part="1"
+AR Path="/5F345A0C/64388CF5" Ref="C?"  Part="1"
+F 0 "C8" V 9050 2600 50  0000 C CNN
+F 1 "100n" V 9150 2600 50  0000 C CNN
+F 2 "Capacitor_SMD:C_1206_3216Metric_Pad1.42x1.75mm_HandSolder" H 8938 2450 50  0001 C CNN
+F 3 "~" H 8900 2600 50  0001 C CNN
+	1    8900 2600
+	-1   0    0    1
+$EndComp
+$Comp
+L power:GND #PWR011
+U 1 1 64388CFB
+P 8900 2750
+AR Path="/64388CFB" Ref="#PWR011"  Part="1"
+AR Path="/5F345A0C/64388CFB" Ref="#PWR?"  Part="1"
+F 0 "#PWR011" H 8900 2500 50  0001 C CNN
+F 1 "GND" H 8905 2577 50  0000 C CNN
+F 2 "" H 8900 2750 50  0001 C CNN
+F 3 "" H 8900 2750 50  0001 C CNN
+	1    8900 2750
+	1    0    0    -1
+$EndComp
+Wire Wire Line
+	8900 2450 8900 2350
+Connection ~ 8900 2350
+Wire Wire Line
+	8900 2350 9150 2350
+$Comp
+L Device:C C9
+U 1 1 6439B7A5
+P 8900 3900
+AR Path="/6439B7A5" Ref="C9"  Part="1"
+AR Path="/5F345A0C/6439B7A5" Ref="C?"  Part="1"
+F 0 "C9" V 9050 3900 50  0000 C CNN
+F 1 "100n" V 9150 3900 50  0000 C CNN
+F 2 "Capacitor_SMD:C_1206_3216Metric_Pad1.42x1.75mm_HandSolder" H 8938 3750 50  0001 C CNN
+F 3 "~" H 8900 3900 50  0001 C CNN
+	1    8900 3900
+	-1   0    0    1
+$EndComp
+$Comp
+L power:GND #PWR013
+U 1 1 6439B7AB
+P 8900 4050
+AR Path="/6439B7AB" Ref="#PWR013"  Part="1"
+AR Path="/5F345A0C/6439B7AB" Ref="#PWR?"  Part="1"
+F 0 "#PWR013" H 8900 3800 50  0001 C CNN
+F 1 "GND" H 8905 3877 50  0000 C CNN
+F 2 "" H 8900 4050 50  0001 C CNN
+F 3 "" H 8900 4050 50  0001 C CNN
+	1    8900 4050
+	1    0    0    -1
+$EndComp
+Wire Wire Line
+	8900 3750 8900 3650
+Connection ~ 8900 3650
+Wire Wire Line
+	8900 3650 9150 3650
+$Comp
+L Switch:SW_SPDT SW1
+U 1 1 643B6879
+P 6700 4100
+F 0 "SW1" H 6700 4385 50  0000 C CNN
+F 1 "Bank" H 6700 4294 50  0000 C CNN
+F 2 "Connector_PinHeader_2.54mm:PinHeader_1x03_P2.54mm_Vertical" H 6700 4100 50  0001 C CNN
+F 3 "~" H 6700 4100 50  0001 C CNN
+	1    6700 4100
+	1    0    0    -1
+$EndComp
+Wire Wire Line
+	6050 4100 6500 4100
+$Comp
+L power:GND #PWR?
+U 1 1 643C660C
+P 6950 4250
+F 0 "#PWR?" H 6950 4000 50  0001 C CNN
+F 1 "GND" H 6955 4077 50  0000 C CNN
+F 2 "" H 6950 4250 50  0001 C CNN
+F 3 "" H 6950 4250 50  0001 C CNN
+	1    6950 4250
+	1    0    0    -1
+$EndComp
+Wire Wire Line
+	6900 4200 6950 4200
+Wire Wire Line
+	6950 4200 6950 4250
+NoConn ~ 6900 4000
 $EndSCHEMATC

Commit message: updated footprints on Quantizer
Parts:
- J3, J4, J5, J6, J7, J8: footprint telec:JackHole -> telec:Jack_Hole_Square; symbol Connector:AudioJack3_Switch -> Connector:AudioJack3_SwitchTR
Connections:
- no-connect marks 27 -> 21
Changed lines of the file:
@@
 $EndComp
 $Comp
-L Connector:AudioJack3_Switch J3
+L Connector:AudioJack3_SwitchTR J3
 U 1 1 5F0BD040
 P 950 2250
 F 0 "J3" H 932 2675 50  0000 C CNN
 F 1 "IN1" H 932 2584 50  0000 C CNN
-F 2 "telec:JackHole" H 950 2250 50  0001 C CNN
+F 2 "telec:Jack_Hole_Square" H 950 2250 50  0001 C CNN
 F 3 "~" H 950 2250 50  0001 C CNN
 	1    950  2250
@@
 	2250 1350 2250 1450
 $Comp
-L Connector:AudioJack3_Switch J7
+L Connector:AudioJack3_SwitchTR J7
 U 1 1 5F41F070
 P 10650 3550
 F 0 "J7" H 10632 3975 50  0000 C CNN
 F 1 "OUT2" H 10632 3884 50  0000 C CNN
-F 2 "telec:JackHole" H 10650 3550 50  0001 C CNN
+F 2 "telec:Jack_Hole_Square" H 10650 3550 50  0001 C CNN
 F 3 "~" H 10650 3550 50  0001 C CNN
 	1    10650 3550
@@
 $EndComp
 $Comp
-L Connector:AudioJack3_Switch J6
+L Connector:AudioJack3_SwitchTR J6
 U 1 1 5F4208DD
 P 10650 2250
 F 0 "J6" H 10632 2675 50  0000 C CNN
 F 1 "OUT1" H 10632 2584 50  0000 C CNN
-F 2 "telec:JackHole" H 10650 2250 50  0001 C CNN
+F 2 "telec:Jack_Hole_Square" H 10650 2250 50  0001 C CNN
 F 3 "~" H 10650 2250 50  0001 C CNN
 	1    10650 2250
@@
 NoConn ~ 10450 3650
 NoConn ~ 10450 3550
-NoConn ~ 10450 3450
 NoConn ~ 10450 3850
 $Comp
 L power:GND #PWR048
 U 1 1 5F62E5EC
-P 10450 3350
-F 0 "#PWR048" H 10450 3100 50  0001 C CNN
-F 1 "GND" V 10455 3222 50  0000 R CNN
-F 2 "" H 10450 3350 50  0001 C CNN
-F 3 "" H 10450 3350 50  0001 C CNN
-	1    10450 3350
+P 10450 3450
+F 0 "#PWR048" H 10450 3200 50  0001 C CNN
+F 1 "GND" V 10455 3322 50  0000 R CNN
+F 2 "" H 10450 3450 50  0001 C CNN
+F 3 "" H 10450 3450 50  0001 C CNN
+	1    10450 3450
 	0    1    1    0
 $EndComp
 NoConn ~ 10450 2350
 NoConn ~ 10450 2250
-NoConn ~ 10450 2150
 NoConn ~ 10450 2550
 $Comp
 L power:GND #PWR047
 U 1 1 5F62EF49
-P 10450 2050
-F 0 "#PWR047" H 10450 1800 50  0001 C CNN
-F 1 "GND" V 10455 1922 50  0000 R CNN
-F 2 "" H 10450 2050 50  0001 C CNN
-F 3 "" H 10450 2050 50  0001 C CNN
-	1    10450 2050
+P 10450 2150
+F 0 "#PWR047" H 10450 1900 50  0001 C CNN
+F 1 "GND" V 10455 2022 50  0000 R CNN
+F 2 "" H 10450 2150 50  0001 C CNN
+F 3 "" H 10450 2150 50  0001 C CNN
+	1    10450 2150
 	0    1    1    0
 $EndComp
 NoConn ~ 1150 2350
 NoConn ~ 1150 2250
-NoConn ~ 1150 2150
 $Comp
 L power:GND #PWR016
 U 1 1 5F63005B
-P 1150 2050
-F 0 "#PWR016" H 1150 1800 50  0001 C CNN
-F 1 "GND" V 1155 1922 50  0000 R CNN
-F 2 "" H 1150 2050 50  0001 C CNN
-F 3 "" H 1150 2050 50  0001 C CNN
-	1    1150 2050
+P 1150 2150
+F 0 "#PWR016" H 1150 1900 50  0001 C CNN
+F 1 "GND" V 1155 2022 50  0000 R CNN
+F 2 "" H 1150 2150 50  0001 C CNN
+F 3 "" H 1150 2150 50  0001 C CNN
+	1    1150 2150
 	0    -1   1    0
 $EndComp
@@
 Mode1
 $Comp
-L Connector:AudioJack3_Switch J4
+L Connector:AudioJack3_SwitchTR J4
 U 1 1 63B8B221
 P 950 3650
 F 0 "J4" H 932 4075 50  0000 C CNN
 F 1 "IN2" H 932 3984 50  0000 C CNN
-F 2 "telec:JackHole" H 950 3650 50  0001 C CNN
+F 2 "telec:Jack_Hole_Square" H 950 3650 50  0001 C CNN
 F 3 "~" H 950 3650 50  0001 C CNN
 	1    950  3650
@@
 NoConn ~ 1150 3750
 NoConn ~ 1150 3650
-NoConn ~ 1150 3550
 $Comp
 L power:GND #PWR018
 U 1 1 63B8B22A
-P 1150 3450
-F 0 "#PWR018" H 1150 3200 50  0001 C CNN
-F 1 "GND" V 1155 3322 50  0000 R CNN
-F 2 "" H 1150 3450 50  0001 C CNN
-F 3 "" H 1150 3450 50  0001 C CNN
-	1    1150 3450
+P 1150 3550
+F 0 "#PWR018" H 1150 3300 50  0001 C CNN
+F 1 "GND" V 1155 3422 50  0000 R CNN
+F 2 "" H 1150 3550 50  0001 C CNN
+F 3 "" H 1150 3550 50  0001 C CNN
+	1    1150 3550
 	0    -1   1    0
 $EndComp
@@
 $EndComp
 $Comp
-L Connector:AudioJack3_Switch J5
+L Connector:AudioJack3_SwitchTR J5
 U 1 1 63BBC976
 P 950 5050
 F 0 "J5" H 932 5475 50  0000 C CNN
 F 1 "IN3" H 932 5384 50  0000 C CNN
-F 2 "telec:JackHole" H 950 5050 50  0001 C CNN
+F 2 "telec:Jack_Hole_Square" H 950 5050 50  0001 C CNN
 F 3 "~" H 950 5050 50  0001 C CNN
 	1    950  5050
@@
 NoConn ~ 1150 5150
 NoConn ~ 1150 5050
-NoConn ~ 1150 4950
 $Comp
 L power:GND #PWR020
 U 1 1 63BBC97F
-P 1150 4850
-F 0 "#PWR020" H 1150 4600 50  0001 C CNN
-F 1 "GND" V 1155 4722 50  0000 R CNN
-F 2 "" H 1150 4850 50  0001 C CNN
-F 3 "" H 1150 4850 50  0001 C CNN
-	1    1150 4850
+P 1150 4950
+F 0 "#PWR020" H 1150 4700 50  0001 C CNN
+F 1 "GND" V 1155 4822 50  0000 R CNN
+F 2 "" H 1150 4950 50  0001 C CNN
+F 3 "" H 1150 4950 50  0001 C CNN
+	1    1150 4950
 	0    -1   1    0
 $EndComp
@@
 NoConn ~ 4850 3900
 $Comp
-L Connector:AudioJack3_Switch J8
+L Connector:AudioJack3_SwitchTR J8
 U 1 1 63FD48AA
 P 10650 4800
 F 0 "J8" H 10632 5225 50  0000 C CNN
 F 1 "OUT3" H 10632 5134 50  0000 C CNN
-F 2 "telec:JackHole" H 10650 4800 50  0001 C CNN
+F 2 "telec:Jack_Hole_Square" H 10650 4800 50  0001 C CNN
 F 3 "~" H 10650 4800 50  0001 C CNN
 	1    10650 4800
@@
 NoConn ~ 10450 4900
 NoConn ~ 10450 4800
-NoConn ~ 10450 4700
 NoConn ~ 10450 5100
 $Comp
 L power:GND #PWR0101
 U 1 1 63FD48B4
-P 10450 4600
-F 0 "#PWR0101" H 10450 4350 50  0001 C CNN
-F 1 "GND" V 10455 4472 50  0000 R CNN
-F 2 "" H 10450 4600 50  0001 C CNN
-F 3 "" H 10450 4600 50  0001 C CNN
-	1    10450 4600
+P 10450 4700
+F 0 "#PWR0101" H 10450 4450 50  0001 C CNN
+F 1 "GND" V 10455 4572 50  0000 R CNN
+F 2 "" H 10450 4700 50  0001 C CNN
+F 3 "" H 10450 4700 50  0001 C CNN
+	1    10450 4700
 	0    1    1    0
 $EndComp
