File: Scope/Scope.kicad_pcb (KiCad board)
At the start: 2 copper layers, 100 x 200 mm, 43 parts, among them J1 Clock, J2 EuroPower, J3 SSD1306, J4 CV, J5 Gate, Q1 BC547, Q2 BC557, SW1 Reset, U1 TL082, U2 L7805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

Commit message: Scope schematic done, how I will fit that?
Parts:
- removed C6: 10n, Capacitor_THT:C_Disc_D7.0mm_W2.5mm_P5.00mm
- removed H3, H4: Mounting_Holes, Kosmo_panel:Kosmo_Panel_Dual_Mounting_Holes
- removed the J5 at (217.6, 25.5)
- removed Q1: BC547, Package_TO_SOT_THT:TO-92_Inline_Wide
- removed Q2: BC557, Package_TO_SOT_THT:TO-92_Inline_Wide
- removed the RV1 at (222.7, 47.9)
- added D2: 1N4148, Diode_THT:D_DO-35_SOD27_P7.62mm_Horizontal, F.Cu at (63.0, 121.3)
- added D3: 1N4148, Diode_THT:D_DO-35_SOD27_P7.62mm_Horizontal, F.Cu at (1.42, 92.2)
- added D4: 1N4148, Diode_THT:D_DO-35_SOD27_P7.62mm_Horizontal, F.Cu at (4.97, 92.2)
- added J2: IN2, telec:JackHole, F.Cu at (32.0, 175.9)
- added J4: Conn_Pickit_5, Connector_PinHeader_2.54mm:PinHeader_1x05_P2.54mm_Vertical, F.Cu at (15.4, 80.9)
- added R10: 1k, Resistor_THT:R_Axial_DIN0204_L3.6mm_D1.6mm_P7.62mm_Horizontal, F.Cu at (68.3, 104.4)
- added R11: 33k, Resistor_THT:R_Axial_DIN0204_L3.6mm_D1.6mm_P7.62mm_Horizontal, F.Cu at (62.0, 103.6)
- added R13: 20k, Resistor_THT:R_Axial_DIN0204_L3.6mm_D1.6mm_P7.62mm_Horizontal, F.Cu at (74.2, 109.1)
- added R14: 33k, Resistor_THT:R_Axial_DIN0204_L3.6mm_D1.6mm_P7.62mm_Horizontal, F.Cu at (85.0, 124.3)
- added R4: 33k, Resistor_THT:R_Axial_DIN0204_L3.6mm_D1.6mm_P7.62mm_Horizontal, F.Cu at (58.9, 103.6)
- added R5: 120k, Resistor_THT:R_Axial_DIN0204_L3.6mm_D1.6mm_P7.62mm_Horizontal, F.Cu at (75.0, 135.2)
- added R7: 33k, Resistor_THT:R_Axial_DIN0204_L3.6mm_D1.6mm_P7.62mm_Horizontal, F.Cu at (80.5, 119.7)
- added R8: 68k, Resistor_THT:R_Axial_DIN0204_L3.6mm_D1.6mm_P7.62mm_Horizontal, F.Cu at (71.0, 115.2)
- added RV2: 100k, Potentiometer_THT:Potentiometer_Piher_T-16L_Single_Vertical_Hole, F.Cu at (30.5, 134.2)
- added RV4: 100k, Potentiometer_THT:Potentiometer_Piher_T-16L_Single_Vertical_Hole, F.Cu at (23.7, 127.2)
- added RV5: 100k, Potentiometer_THT:Potentiometer_Piher_T-16L_Single_Vertical_Hole, F.Cu at (30.4, 100.7)
- added RV6: 100k, Potentiometer_THT:Potentiometer_Piher_T-16L_Single_Vertical_Hole, F.Cu at (23.8, 94.1)
- added SW2: SW, Button_Switch_THT:SW_PUSH_6mm, F.Cu at (21.1, 65.2)
- added SW3: SW, Button_Switch_THT:SW_PUSH_6mm, F.Cu at (28.6, 65.2)
- added SW4: SW, Button_Switch_THT:SW_PUSH_6mm, F.Cu at (36.1, 65.2)
- added U2: TL082, Package_DIP:DIP-8_W7.62mm_LongPads, F.Cu at (57.5, 114.9)
- added U4: TL082, Package_DIP:DIP-8_W7.62mm_LongPads, F.Cu at (-17.9, 206.0)
- C3, C4: moved to B.Cu
- D5: renamed from D1; moved to B.Cu
- D6: renamed from D2; moved to B.Cu
- D7: renamed from D4; moved to B.Cu
- D8: renamed from D5; moved to B.Cu
- D9: renamed from D6; moved to B.Cu
- J1: value Clock -> IN1
- J6: renamed from J4; value CV -> OUT
- R1: value 100k -> 68k
- R12: value 1k -> 120k
- R16: renamed from R4; moved to B.Cu
- R17: renamed from R5; moved to B.Cu
- R18: renamed from R7; moved to B.Cu
- R19: renamed from R8; moved to B.Cu
- R2, R9: value 10k -> 68k
- R20: renamed from R10; moved to B.Cu
- R3: value 10k -> 1k
- R6: value 10k -> 20k
- RV1: renamed from RV2; value R_POT -> 100k
- RV3: value R_POT_TRIM -> 100k; footprint Potentiometer_THT:Potentiometer_Bourns_3299W_Vertical -> telec:Potentiometer_P3.81mmx5.12mm_Vertical
- SW1: value Reset -> SW
- U3: renamed from U2; moved to B.Cu
- moved C2 305.5 mm to (0.30, 114.9)
- moved J6 301.0 mm to (-18.4, 182.2)
- moved J1 292.7 mm to (21.9, 196.2), turned to 90 degrees
- moved RV1 291.2 mm to (24.0, 160.6)
- moved U1 282.9 mm to (13.5, 118.5)
- moved R15 256.5 mm to (-19.7, 195.1)
- moved SW1 250.9 mm to (13.6, 65.2), turned to 90 degrees
- moved U3 244.5 mm to (29.6, 54.5), turned to 180 degrees
- moved C3 239.1 mm to (35.7, 45.2)
- moved R16 221.7 mm to (-7.46, -23.8), turned to 90 degrees
- moved R18 217.5 mm to (-4.17, -23.8), turned to 90 degrees
- moved R17 214.1 mm to (-7.46, -17.9), turned to 90 degrees
- moved R19 210.0 mm to (-4.17, -17.9), turned to 90 degrees
- moved D5 203.3 mm to (-4.86, -11.9), turned to 90 degrees
- moved D6 195.7 mm to (-4.86, -5.82), turned to 90 degrees
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- renumbered D3 to D1, J2 to J3, J3 to J5, R11 to R15, U3 to U5
Connections:
- D1 pad 1: Net-(D3-Pad1) -> +5V
- D1 pad 2: Net-(D3-Pad2) -> /ANA0
- J6 pad T: Net-(J4-PadT) -> Net-(J6-PadT)
- R1 pad 1: Net-(Q1-Pad2) -> +12V
- R1 pad 2: Net-(J1-PadT) -> Net-(R1-Pad2)
- R12 pad 1: Net-(J5-PadT) -> Net-(R12-Pad1)
- R15 pad 1: Net-(J4-PadT) -> Net-(J6-PadT)
- R15 pad 2: Net-(R11-Pad2) -> Net-(R15-Pad2)
- R2 pad 1: Net-(Q1-Pad1) -> -12V
- R2 pad 2: +5V -> Net-(R2-Pad2)
- R3 pad 1: Net-(Q2-Pad2) -> Net-(R3-Pad1)
- R3 pad 2: Net-(Q1-Pad1) -> /ANA0
- R6 pad 1: GND -> Net-(R5-Pad2)
- R6 pad 2: /Clk -> Net-(R3-Pad1)
- R9 pad 1: /Rst -> -12V
- R9 pad 2: GND -> Net-(R9-Pad2)
- RV1 pad 1: Net-(RV2-Pad1) -> Net-(R2-Pad2)
- RV1 pad 2: Net-(RV2-Pad2) -> Net-(RV1-Pad2)
- RV1 pad 3: Net-(RV2-Pad3) -> Net-(R1-Pad2)
- RV3 pad 1: Net-(RV3-Pad1) -> +5V
- RV3 pad 2: Net-(RV3-Pad2) -> /REF
- RV3 pad 3: Net-(RV3-Pad3) -> GND
- SW1 pad 1: +5V -> /SW1
- SW1 pad 2: /Rst -> GND
- U1 pad 1: Net-(R12-Pad2) -> Net-(R5-Pad1)
- U1 pad 2: Net-(J5-PadT) -> Net-(R4-Pad2)
- U1 pad 3: Net-(U1-Pad3) -> Net-(RV1-Pad2)
- U1 pad 5: Net-(U1-Pad5) -> /REF
- U1 pad 6: Net-(J4-PadT) -> Net-(R5-Pad2)
- U1 pad 7: Net-(R11-Pad2) -> Net-(R3-Pad1)
- U5 pad 1: Net-(U3-Pad1) -> /~MCLR
- U5 pad 14: Net-(U3-Pad14) -> /SCL
- U5 pad 15: Net-(U3-Pad15) -> /SDA
- U5 pad 19: Net-(U3-Pad19) -> GND
- U5 pad 2: Net-(U3-Pad2) -> /ANA0
- U5 pad 20: Net-(U3-Pad20) -> +5V
- U5 pad 23: Net-(U3-Pad23) -> /SW4
- U5 pad 24: Net-(U3-Pad24) -> /SW3
- U5 pad 25: Net-(U3-Pad25) -> /SW2
- U5 pad 26: Net-(U3-Pad26) -> /SW1
- U5 pad 27: Net-(U3-Pad27) -> /PGC
- U5 pad 28: Net-(U3-Pad28) -> /PGD
- U5 pad 3: Net-(U3-Pad3) -> /ANA1
- U5 pad 4: Net-(U3-Pad4) -> /DAC1OUT1
- U5 pad 5: Net-(U3-Pad5) -> /ANA3
- U5 pad 8: Net-(U3-Pad19) -> GND
Other:
- outline, holes or cut-outs redrawn

Commit message: Scope layout
Parts:
- removed D5, D6, D7, D8: LED, LED_SMD:LED_1206_3216Metric_Castellated
- removed D9: LED, LED_SMD:LED_1206_3216Metric_ReverseMount_Hole1.8x2.4mm
- removed R15: 1k, Resistor_THT:R_Axial_DIN0204_L3.6mm_D1.6mm_P7.62mm_Horizontal
- removed R16, R17, R18, R19, R20: 1k, Resistor_SMD:R_1206_3216Metric_Pad1.42x1.75mm_HandSolder
- removed U4: TL082, Package_DIP:DIP-8_W7.62mm_LongPads
- added C6: 100n, Capacitor_SMD:C_1206_3216Metric_Pad1.42x1.75mm_HandSolder, B.Cu at (39.5, 134.1)
- added C7: 100n, Capacitor_SMD:C_1206_3216Metric_Pad1.42x1.75mm_HandSolder, B.Cu at (39.8, 103.0)
- added C8: 100n, Capacitor_SMD:C_1206_3216Metric_Pad1.42x1.75mm_HandSolder, B.Cu at (39.8, 113.8)
- C1, C2, C5: footprint Capacitor_THT:C_Disc_D7.0mm_W2.5mm_P5.00mm -> Capacitor_SMD:C_1206_3216Metric_Pad1.42x1.75mm_HandSolder; moved to B.Cu
- D1, D3: footprint Diode_THT:D_DO-35_SOD27_P7.62mm_Horizontal -> Diode_SMD:D_1206_3216Metric_Pad1.42x1.75mm_HandSolder
- D2, D4: footprint Diode_THT:D_DO-35_SOD27_P7.62mm_Horizontal -> Diode_SMD:D_1206_3216Metric_Pad1.42x1.75mm_HandSolder; moved to B.Cu
- J6: value OUT -> DAC; footprint telec:JackHole -> Connector_PinHeader_2.54mm:PinHeader_1x01_P2.54mm_Vertical; moved to B.Cu
- LOGO1: footprint logo:telec-32 -> logo:telec-8
- R1, R10, R11, R12, R13, R14, R2, R3, R4, R5, R6, R7, R8, R9: footprint Resistor_THT:R_Axial_DIN0204_L3.6mm_D1.6mm_P7.62mm_Horizontal -> Resistor_SMD:R_1206_3216Metric_Pad1.42x1.75mm_HandSolder; moved to B.Cu
- U1, U2: footprint Package_DIP:DIP-8_W7.62mm_LongPads -> Package_SO:SOIC-8_3.9x4.9mm_P1.27mm; moved to B.Cu
- U5: moved to B.Cu
- moved J6 94.7 mm to (18.6, 95.0)
- moved R2 87.1 mm to (19.6, 182.8), turned to 0 degrees
- moved R4 83.9 mm to (19.6, 177.7)
- moved R1 82.9 mm to (19.6, 172.8), turned to 0 degrees
- moved C2 65.3 mm to (39.8, 166.9), turned to 90 degrees
- moved R7 64.9 mm to (35.2, 166.1), turned to 0 degrees
- moved R9 58.6 mm to (19.6, 129.5), turned to 0 degrees
- moved LOGO1 56.9 mm to (27.0, 16.4)
- moved C1 52.5 mm to (39.8, 156.2), turned to 270 degrees
- moved R3 51.6 mm to (35.4, 153.8), turned to 180 degrees
- moved R8 51.6 mm to (19.6, 119.5), turned to 0 degrees
- moved R14 51.2 mm to (35.1, 113.0), turned to 0 degrees
- moved R12 51.0 mm to (39.8, 108.2)
- moved R6 49.9 mm to (35.4, 156.2), turned to 0 degrees
- moved D1 49.0 mm to (36.9, 79.7), turned to 270 degrees
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Connections:
- U5 pad 16: Net-(U5-Pad16) -> /SW1
- U5 pad 17: Net-(U5-Pad17) -> /SW2
- U5 pad 23: /SW4 -> Net-(U5-Pad23)
- U5 pad 24: /SW3 -> Net-(U5-Pad24)
- U5 pad 25: /SW2 -> /SW3
- U5 pad 26: /SW1 -> /SW4
Routing:
- net -12V: track 0.00 -> 250.9 mm, vias 0 -> 10
- net +12V: track 0.00 -> 247.3 mm, vias 0 -> 6
- net +5V: track 0.00 -> 119.8 mm, vias 0 -> 2
- net /REF: track 0.00 -> 107.4 mm
- net /ANA0: track 0.00 -> 81.4 mm, vias 0 -> 3
- net /SCL: track 0.00 -> 66.2 mm
- net /SDA: track 0.00 -> 53.4 mm
- net Net-(R11-Pad2): track 0.00 -> 33.1 mm
- net Net-(R4-Pad2): track 0.00 -> 33.0 mm
- net /ANA1: track 0.00 -> 29.7 mm, vias 0 -> 3
- net /DAC1OUT1: track 0.00 -> 24.3 mm
- net Net-(RV1-Pad2): track 0.00 -> 19.8 mm
- net Net-(RV4-Pad2): track 0.00 -> 19.8 mm
- net Net-(J2-PadT): track 0.00 -> 19.3 mm
- net Net-(J1-PadT): track 0.00 -> 19.3 mm
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- added copper zone on F.Cu, net GND
Other:
- board size 100 x 200 mm -> 30 x 200 mm
- board text added: "PCB ref here:"

Commit message: Scope done !
Other:
- board text added: "Design by telec"
- board text added: "Dual Scope"
- board text added: "Gain"
- board text added: "IN1"
- board text added: "IN2"
- board text added: "Off"
- board text added: "Offset"
- board text added: "TB"

Commit message: updated footprints on Scope, not done...
Parts:
- J1, J2: footprint telec:JackHole -> telec:Jack_Hole_Square
- RV1, RV2, RV4, RV5, RV6: footprint Potentiometer_THT:Potentiometer_Piher_T-16L_Single_Vertical_Hole -> telec:Potentiometer_Single_Vertical_Hole
- moved RV1 13.2 mm to (35.9, 177.5), turned to 270 degrees
- moved RV6 13.0 mm to (35.5, 90.1), turned to 270 degrees
- moved RV2 12.8 mm to (18.5, 161.0), turned to 90 degrees
- moved RV4 12.5 mm to (35.3, 124.7), turned to 270 degrees
- moved RV5 10.3 mm to (20.1, 103.3), turned to 90 degrees
- moved J2 1.20 mm to (23.3, 142.8)
