File: Scope/Scope.sch (KiCad schematic (older format))
At the start: 43 parts, among them J1 Clock, J2 EuroPower, J3 SSD1306, J4 CV, J5 Gate, Q1 BC547, Q2 BC557, SW1 Reset, U1 TL082, U2 L7805, U3 PIC18F26Q43

Commit message: Scope schematic done, how I will fit that?
Parts:
- removed C6: 10n, Capacitor_THT:C_Disc_D7.0mm_W2.5mm_P5.00mm, symbol Device:C
- removed H3, H4: Mounting_Holes, Kosmo_panel:Kosmo_Panel_Dual_Mounting_Holes, symbol Kosmo:Mounting_Holes
- removed J5: Gate, telec:JackHole, symbol Connector:AudioJack3_Switch
- removed Q1: BC547, Package_TO_SOT_THT:TO-92_Inline_Wide, symbol Transistor_BJT:BC547
- removed Q2: BC557, Package_TO_SOT_THT:TO-92_Inline_Wide, symbol Transistor_BJT:BC557
- removed RV1: R_POT_Small, Potentiometer_THT:Potentiometer_Bourns_3339P_Vertical, symbol Device:R_POT_Small
- added D2, D3, D4: 1N4148, Diode_THT:D_DO-35_SOD27_P7.62mm_Horizontal, symbol Diode:1N4148
- added J2: IN2, telec:JackHole, symbol Connector:AudioJack3_Switch
- added J4: Conn_Pickit_5, Connector_PinHeader_2.54mm:PinHeader_1x05_P2.54mm_Vertical, symbol telec:Conn_Pickit_5
- added R10: 1k, Resistor_THT:R_Axial_DIN0204_L3.6mm_D1.6mm_P7.62mm_Horizontal, symbol Device:R
- added R11, R14, R4, R7: 33k, Resistor_THT:R_Axial_DIN0204_L3.6mm_D1.6mm_P7.62mm_Horizontal, symbol Device:R
- added R13: 20k, Resistor_THT:R_Axial_DIN0204_L3.6mm_D1.6mm_P7.62mm_Horizontal, symbol Device:R
- added R5: 120k, Resistor_THT:R_Axial_DIN0204_L3.6mm_D1.6mm_P7.62mm_Horizontal, symbol Device:R
- added R8: 68k, Resistor_THT:R_Axial_DIN0204_L3.6mm_D1.6mm_P7.62mm_Horizontal, symbol Device:R
- added RV2, RV4, RV5, RV6: 100k, Potentiometer_THT:Potentiometer_Piher_T-16L_Single_Vertical_Hole, symbol Device:R_POT
- added SW2, SW3, SW4: SW, Button_Switch_THT:SW_PUSH_6mm, symbol Switch:SW_Push
- added unit 1 of U1
- added U2: TL082, Package_DIP:DIP-8_W7.62mm_LongPads, symbol Amplifier_Operational:TL082
- J1: value Clock -> IN1
- J6: renamed from J4; value CV -> OUT
- R1: value 100k -> 68k
- R12: value 1k -> 120k
- R2, R9: value 10k -> 68k
- R3: value 10k -> 1k
- R6: value 10k -> 20k
- RV1: renamed from RV2; value R_POT -> 100k
- RV3: value R_POT_TRIM -> 100k; footprint Potentiometer_THT:Potentiometer_Bourns_3299W_Vertical -> telec:Potentiometer_P3.81mmx5.12mm_Vertical
- SW1: value Reset -> SW; symbol Switch:SW_SPST -> Switch:SW_Push
- renumbered D3 to D1, D1 to D5, D2 to D6, D4 to D7, D5 to D8, D6 to D9, J2 to J3, J3 to J5, R11 to R15, R4 to R16, R5 to R17, R7 to R18, R8 to R19, R10 to R20, U2 to U3, U1 to U4, U3 to U5
Connections:
- net labels added: ANA0, ANA1, ANA3, DAC1OUT1, PGC, PGD, REF, SW1, SW2, SW3, SW4, ~MCLR
- net labels removed: Rst
- wire segments 59 -> 130
- no-connect marks 11 -> 22
Other:
- note added: "+/-15V => 0-5V"
- note added: "2.14V"
- note added: "Gain (1-4) + offset"
- note added: "Input stage"
- note added: "Timebase"
- moved on the sheet: C1, C2, C3, C4, C5, D1, J1, J3, J5, J6, R15, RV1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

Commit message: Scope layout
Parts:
- removed D5, D6, D7, D8: LED, LED_SMD:LED_1206_3216Metric_Castellated, symbol Device:LED
- removed D9: LED, LED_SMD:LED_1206_3216Metric_ReverseMount_Hole1.8x2.4mm, symbol Device:LED
- removed J6: OUT, telec:JackHole, symbol Connector:AudioJack3_Switch
- removed R15: 1k, Resistor_THT:R_Axial_DIN0204_L3.6mm_D1.6mm_P7.62mm_Horizontal, symbol Device:R
- removed R16, R17, R18, R19, R20: 1k, Resistor_SMD:R_1206_3216Metric_Pad1.42x1.75mm_HandSolder, symbol Device:R
- removed U4: TL082, Package_DIP:DIP-8_W7.62mm_LongPads, symbol Amplifier_Operational:TL082
- added C6, C7, C8: 100n, Capacitor_SMD:C_1206_3216Metric_Pad1.42x1.75mm_HandSolder, symbol Device:C
- added J6: DAC, Connector_PinHeader_2.54mm:PinHeader_1x01_P2.54mm_Vertical, symbol Connector:Conn_01x01_Female
- C1, C2, C5: footprint Capacitor_THT:C_Disc_D7.0mm_W2.5mm_P5.00mm -> Capacitor_SMD:C_1206_3216Metric_Pad1.42x1.75mm_HandSolder
- D1, D2, D3, D4: footprint Diode_THT:D_DO-35_SOD27_P7.62mm_Horizontal -> Diode_SMD:D_1206_3216Metric_Pad1.42x1.75mm_HandSolder
- LOGO1: footprint logo:telec-32 -> logo:telec-8
- R1, R10, R11, R12, R13, R14, R2, R3, R4, R5, R6, R7, R8, R9: footprint Resistor_THT:R_Axial_DIN0204_L3.6mm_D1.6mm_P7.62mm_Horizontal -> Resistor_SMD:R_1206_3216Metric_Pad1.42x1.75mm_HandSolder
- U1, U2: footprint Package_DIP:DIP-8_W7.62mm_LongPads -> Package_SO:SOIC-8_3.9x4.9mm_P1.27mm
Connections:
- net +12V: now also C7.2
- net -12V: now also C8.2
- net DAC1OUT1: now also J6.1 (Pin_1)
- net GND: now also C6.1, C7.1, C8.1
- net REF: now also C6.2
- net SW1: now also U5.16 (RC5); no longer U5.26 (RB5)
- net SW2: now also U5.17 (RC6); no longer U5.25 (RB4)
- net SW3: now also U5.25 (RB4); no longer U5.24 (RB3)
- net SW4: now also U5.26 (RB5); no longer U5.23 (RB2)
- no-connect marks 22 -> 18
Other:
- note removed: "Output buffer"
- moved on the sheet: C1, C2, U1C, U2C

Commit message: updated footprints on Scope, not done...
Parts:
- J1, J2: footprint telec:JackHole -> telec:Jack_Hole_Square; symbol Connector:AudioJack3_Switch -> Connector:AudioJack3_SwitchTR
- RV1, RV2, RV4, RV5, RV6: footprint Potentiometer_THT:Potentiometer_Piher_T-16L_Single_Vertical_Hole -> telec:Potentiometer_Single_Vertical_Hole
Connections:
- no-connect marks 18 -> 16
Changed lines of the file:
@@
 $EndComp
 $Comp
-L Connector:AudioJack3_Switch J1
+L Connector:AudioJack3_SwitchTR J1
 U 1 1 5F0BD040
 P 850 3400
 F 0 "J1" H 832 3825 50  0000 C CNN
 F 1 "IN1" H 832 3734 50  0000 C CNN
-F 2 "telec:JackHole" H 850 3400 50  0001 C CNN
+F 2 "telec:Jack_Hole_Square" H 850 3400 50  0001 C CNN
 F 3 "~" H 850 3400 50  0001 C CNN
 	1    850  3400
@@
 NoConn ~ 1050 3500
 NoConn ~ 1050 3400
-NoConn ~ 1050 3300
 $Comp
 L power:GND #PWR012
 U 1 1 5F63005B
-P 1050 3200
-F 0 "#PWR012" H 1050 2950 50  0001 C CNN
-F 1 "GND" V 1055 3072 50  0000 R CNN
-F 2 "" H 1050 3200 50  0001 C CNN
-F 3 "" H 1050 3200 50  0001 C CNN
-	1    1050 3200
+P 1050 3300
+F 0 "#PWR012" H 1050 3050 50  0001 C CNN
+F 1 "GND" V 1055 3172 50  0000 R CNN
+F 2 "" H 1050 3300 50  0001 C CNN
+F 3 "" H 1050 3300 50  0001 C CNN
+	1    1050 3300
 	0    -1   1    0
 $EndComp
@@
 F 0 "RV1" V 1800 3150 50  0000 R CNN
 F 1 "100k" V 1900 3200 50  0000 R CNN
-F 2 "Potentiometer_THT:Potentiometer_Piher_T-16L_Single_Vertical_Hole" H 1900 3100 50  0001 C CNN
+F 2 "telec:Potentiometer_Single_Vertical_Hole" H 1900 3100 50  0001 C CNN
 F 3 "~" H 1900 3100 50  0001 C CNN
 	1    1900 3100
@@
 F 0 "RV6" H 5781 4846 50  0000 R CNN
 F 1 "100k" H 5781 4755 50  0000 R CNN
-F 2 "Potentiometer_THT:Potentiometer_Piher_T-16L_Single_Vertical_Hole" H 5850 4800 50  0001 C CNN
+F 2 "telec:Potentiometer_Single_Vertical_Hole" H 5850 4800 50  0001 C CNN
 F 3 "~" H 5850 4800 50  0001 C CNN
 	1    5850 4800
@@
 	2150 3100 2050 3100
 $Comp
-L Connector:AudioJack3_Switch J2
+L Connector:AudioJack3_SwitchTR J2
 U 1 1 6305FFDF
 P 850 5200
 F 0 "J2" H 832 5625 50  0000 C CNN
 F 1 "IN2" H 832 5534 50  0000 C CNN
-F 2 "telec:JackHole" H 850 5200 50  0001 C CNN
+F 2 "telec:Jack_Hole_Square" H 850 5200 50  0001 C CNN
 F 3 "~" H 850 5200 50  0001 C CNN
 	1    850  5200
@@
 NoConn ~ 1050 5300
 NoConn ~ 1050 5200
-NoConn ~ 1050 5100
 $Comp
 L power:GND #PWR020
 U 1 1 6305FFE8
-P 1050 5000
-F 0 "#PWR020" H 1050 4750 50  0001 C CNN
-F 1 "GND" V 1055 4872 50  0000 R CNN
-F 2 "" H 1050 5000 50  0001 C CNN
-F 3 "" H 1050 5000 50  0001 C CNN
-	1    1050 5000
+P 1050 5100
+F 0 "#PWR020" H 1050 4850 50  0001 C CNN
+F 1 "GND" V 1055 4972 50  0000 R CNN
+F 2 "" H 1050 5100 50  0001 C CNN
+F 3 "" H 1050 5100 50  0001 C CNN
+	1    1050 5100
 	0    -1   1    0
 $EndComp
@@
 F 0 "RV4" V 1800 4950 50  0000 R CNN
 F 1 "100k" V 1900 5000 50  0000 R CNN
-F 2 "Potentiometer_THT:Potentiometer_Piher_T-16L_Single_Vertical_Hole" H 1900 4900 50  0001 C CNN
+F 2 "telec:Potentiometer_Single_Vertical_Hole" H 1900 4900 50  0001 C CNN
 F 3 "~" H 1900 4900 50  0001 C CNN
 	1    1900 4900
@@
 F 0 "RV5" V 2000 5850 50  0000 R CNN
 F 1 "100k" V 2100 5850 50  0000 R CNN
-F 2 "Potentiometer_THT:Potentiometer_Piher_T-16L_Single_Vertical_Hole" H 2100 5750 50  0001 C CNN
+F 2 "telec:Potentiometer_Single_Vertical_Hole" H 2100 5750 50  0001 C CNN
 F 3 "~" H 2100 5750 50  0001 C CNN
 	1    2100 5750
@@
 F 0 "RV2" V 2000 4050 50  0000 R CNN
 F 1 "100k" V 2100 4050 50  0000 R CNN
-F 2 "Potentiometer_THT:Potentiometer_Piher_T-16L_Single_Vertical_Hole" H 2100 3950 50  0001 C CNN
+F 2 "telec:Potentiometer_Single_Vertical_Hole" H 2100 3950 50  0001 C CNN
 F 3 "~" H 2100 3950 50  0001 C CNN
 	1    2100 3950
