File: ADSR/ADSR.kicad_pcb (KiCad board)
At the start: 2 copper layers, 47 parts, among them J1 EuroPower, J2 GATE, J3 Hard Envelope, J4 Envelope, Q1 BC557, Q2 BC547, Q3 BC547, Q4 BC547, U1 LM741, U2 LM741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

Commit message: Will it fits ?
Parts:
- added H1: Mounting_Holes, Kosmo_panel:Kosmo_Panel_Dual_Mounting_Holes, F.Cu at (15.0, 209.0)
- added H2: Mounting_Holes, Kosmo_panel:Kosmo_Panel_Dual_Mounting_Holes, F.Cu at (34.0, 209.0)
- D10, D11, D12, D9: footprint LED_THT:LED_D3.0mm -> LED_SMD:LED_1206_3216Metric_ReverseMount_Hole1.8x2.4mm
- J1: footprint Connector_IDC:IDC-Header_2x05_P2.54mm_Vertical -> telec:EuroPower
- moved R8 105.6 mm to (14.4, 156.5), turned to 0 degrees
- moved J3 99.7 mm to (27.1, 196.0)
- moved C1 99.2 mm to (18.9, 148.8), turned to 270 degrees
- moved D10 96.7 mm to (-3.30, 95.8)
- moved D11 96.7 mm to (-3.30, 101.0)
- moved D12 96.7 mm to (-3.30, 106.3)
- moved D9 96.7 mm to (-3.30, 90.5)
- moved R13 96.7 mm to (1.20, 90.5)
- moved R14 96.7 mm to (1.20, 95.8)
- moved R15 96.7 mm to (1.20, 101.0)
- moved R16 96.7 mm to (1.20, 106.3)
- moved Q2 96.1 mm to (14.6, 148.8), turned to 270 degrees
- moved D1 95.3 mm to (21.8, 143.5), turned to 270 degrees
- moved Q1 91.2 mm to (14.3, 145.0), turned to 0 degrees
- moved R4 89.2 mm to (21.7, 138.1), turned to 180 degrees
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Connections:
- J1 pad 2: -12V -> GND
- J1 pad 3: GND -> +12V
Other:
- board outline added: 25 x 200 mm
- net class Default: clearance 0.2 -> 0.1524; trace_width 0.25 -> 0.1524; via_dia 0.8 -> 0.6858; via_drill 0.4 -> 0.3302
- rule trace_clearance: 0.2 -> 0.1524
- rule trace_min: 0.2 -> 0.1524
- rule via_min_drill: 0.3 -> 0.254
- rule via_min_size: 0.4 -> 0.508

Commit message: It fits !
Parts:
- removed H2: Mounting_Holes, Kosmo_panel:Kosmo_Panel_Dual_Mounting_Holes
- R11: moved to B.Cu
- RV1, RV2, RV3, RV4: footprint Potentiometer_THT:Potentiometer_Piher_T-16L_Single_Vertical_Hole -> Potentiometer_THT:Potentiometer_Alps_RK09K_Single_Vertical
- moved R14 138.8 mm to (31.2, 231.3)
- moved R15 134.6 mm to (35.4, 231.3)
- moved R16 131.3 mm to (39.2, 232.0)
- moved D10 130.3 mm to (23.8, 223.3)
- moved D11 130.3 mm to (23.8, 228.6)
- moved D12 130.3 mm to (23.8, 233.8)
- moved D9 130.3 mm to (23.8, 218.1)
- moved R13 130.3 mm to (28.3, 218.1)
- moved D7 87.3 mm to (13.3, 75.7)
- moved C2 86.9 mm to (18.6, 81.1), turned to 180 degrees
- moved Q3 75.9 mm to (35.9, 73.6), turned to 180 degrees
- moved R11 70.4 mm to (26.5, 72.2)
- moved R12 68.1 mm to (28.2, 96.5), turned to 0 degrees
- moved D8 67.9 mm to (35.7, 92.1), turned to 180 degrees
- moved R8 63.6 mm to (28.2, 94.4)
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Routing:
- net /Cap: track 0.00 -> 66.1 mm
- net /~IN: track 0.00 -> 50.0 mm
- net +12V: track 0.00 -> 36.6 mm
- net /Hard: track 0.00 -> 32.4 mm
- net /GATE: track 0.00 -> 29.8 mm
- net Net-(Q2-Pad2): track 0.00 -> 24.9 mm
- net Net-(R1-Pad2): track 0.00 -> 20.8 mm
- net Net-(D8-Pad1): track 0.00 -> 18.9 mm
- net Net-(D2-Pad2): track 0.00 -> 18.8 mm
- net Net-(D4-Pad1): track 0.00 -> 18.0 mm
- net Net-(Q4-Pad1): track 0.00 -> 15.8 mm
- net Net-(Q4-Pad2): track 0.00 -> 10.5 mm
- net Net-(D3-Pad2): track 0.00 -> 7.35 mm
- net Net-(D7-Pad1): track 0.00 -> 5.54 mm
- net Net-(R7-Pad1): track 0.00 -> 5.10 mm
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- added copper zone on B.Cu, net GND

Commit message: Now the power lines...
Parts:
- added H2: Mounting_Holes, Kosmo_panel:Kosmo_Panel_Dual_Mounting_Holes, F.Cu at (34.0, 209.0)
- R13, R14: footprint Resistor_THT:R_Axial_DIN0204_L3.6mm_D1.6mm_P7.62mm_Horizontal -> Resistor_SMD:R_1206_3216Metric
- R15, R16: value 1k5 -> 2k2; footprint Resistor_THT:R_Axial_DIN0204_L3.6mm_D1.6mm_P7.62mm_Horizontal -> Resistor_SMD:R_1206_3216Metric
- moved R14 79.8 mm to (5.50, 155.8)
- moved D9 76.4 mm to (48.3, 145.7)
- moved R13 75.8 mm to (40.5, 143.2)
- moved D10 66.4 mm to (-0.60, 161.5)
- moved R16 62.8 mm to (42.9, 169.3)
- moved D12 61.9 mm to (39.8, 174.1)
- moved D11 43.0 mm to (6.70, 189.1)
- moved D5 41.5 mm to (21.2, 125.5), turned to 270 degrees
- moved R15 39.8 mm to (9.20, 201.3), turned to 90 degrees
- moved D6 30.4 mm to (24.0, 133.1), turned to 90 degrees
- moved R10 30.3 mm to (18.8, 125.5)
- moved U4 20.7 mm to (26.9, 133.0), turned to 90 degrees
- moved U3 17.8 mm to (22.1, 143.7), turned to 270 degrees
- moved D1 15.3 mm to (35.0, 135.8), turned to 180 degrees
- moved C1 14.9 mm to (29.8, 138.6), turned to 0 degrees
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Connections:
- D9 pad 1: GND -> Net-(D9-Pad1)
- D9 pad 2: Net-(D9-Pad2) -> GND
- R13 pad 1: /IN -> /~IN
- R13 pad 2: Net-(D9-Pad2) -> Net-(D9-Pad1)
Routing:
- net /Hard: track 32.4 -> 78.1 mm
- net +12V: track 36.6 -> 78.7 mm
- net /~IN: track 50.0 -> 91.6 mm
- net /Triggered: track 0.00 -> 37.8 mm
- net /Cap: track 66.1 -> 103.4 mm
- net Net-(Q2-Pad1): track 3.20 -> 32.1 mm
- net Net-(Q1-Pad1): track 0.00 -> 20.8 mm
- net Net-(D5-Pad2): track 0.00 -> 14.9 mm
- net /Envelope: track 0.00 -> 13.2 mm
- net Net-(C1-Pad1): track 0.00 -> 11.4 mm

Commit message: Layout done! Art to do
Parts:
- added R17: 1k, Resistor_THT:R_Axial_DIN0204_L3.6mm_D1.6mm_P7.62mm_Horizontal, F.Cu at (35.1, 166.3)
- added R18: 1k, Resistor_THT:R_Axial_DIN0204_L3.6mm_D1.6mm_P7.62mm_Horizontal, F.Cu at (13.8, 197.1)
- D10, D11, D12, D9, R13, R14, R15, R16: moved to B.Cu
- R11: moved to F.Cu
- moved R13 72.8 mm to (25.9, 71.9)
- moved D9 72.1 mm to (27.5, 76.7), turned to 90 degrees
- moved U3 20.9 mm to (15.3, 163.5), turned to 90 degrees
- moved D10 20.5 mm to (17.6, 152.1), turned to 90 degrees
- moved R14 15.3 mm to (20.3, 152.1), turned to 90 degrees
- moved R16 12.8 mm to (35.1, 179.5)
- moved D12 12.2 mm to (34.1, 184.8), turned to 90 degrees
- moved R3 11.4 mm to (16.5, 144.5)
- moved R4 11.4 mm to (14.4, 136.9)
- moved C1 11.4 mm to (29.8, 150.0)
- moved D5 11.4 mm to (21.2, 136.9)
- moved D6 11.4 mm to (24.0, 144.5)
- moved Q1 11.4 mm to (23.5, 147.0)
- moved Q4 11.4 mm to (29.9, 119.3)
- moved R10 11.4 mm to (18.8, 136.9)
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Connections:
- D9 pad 1: Net-(D9-Pad1) -> GND
- D9 pad 2: GND -> Net-(D9-Pad2)
- J3 pad T: /Hard -> Net-(J3-PadT)
- R13 pad 1: /~IN -> /IN
- R13 pad 2: Net-(D9-Pad1) -> Net-(D9-Pad2)
- R16 pad 1: /Envelope -> /PEnvelope
- U5 pad 6: /Envelope -> /PEnvelope
Routing:
- net -12V: track 0.00 -> 192.5 mm, vias 0 -> 2
- net +12V: track 78.7 -> 213.1 mm, vias 0 -> 1
- net /Hard: track 78.1 -> 158.2 mm
- net GND: track 0.00 -> 72.5 mm, vias 0 -> 9
- net /PEnvelope: track 0.00 -> 24.3 mm
- net /Cap: track 103.4 -> 126.8 mm, vias 0 -> 1
- net /~IN: track 91.6 -> 102.9 mm
- net Net-(Q4-Pad2): track 10.5 -> 18.1 mm
- net Net-(Q1-Pad1): track 20.8 -> 28.3 mm
- net /Triggered: track 37.8 -> 30.4 mm
- net Net-(Q2-Pad2): track 24.9 -> 30.5 mm
- net Net-(Q3-Pad2): track 1.71 -> 5.82 mm
- net Net-(Q2-Pad1): track 32.1 -> 35.5 mm
- net Net-(D12-Pad2): track 0.00 -> 2.81 mm
- net Net-(D11-Pad2): track 0.00 -> 2.80 mm
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
Commit message: ADSR done !
Parts:
- added LOGO1: Logo_telec, logo:telec-8, F.Cu at (24.4, 16.5)
- moved C2 14.4 mm to (15.7, 95.2), turned to 270 degrees
- moved R16 2.10 mm to (35.1, 177.4)
- moved D12 1.27 mm to (33.9, 183.6), turned to 0 degrees
- moved D11 1.05 mm to (15.4, 189.1), turned to 180 degrees
Routing:
- net +12V: track 213.1 -> 235.9 mm
- net /Cap: track 126.8 -> 139.4 mm
- net GND: track 72.5 -> 76.8 mm
- net Net-(D12-Pad2): track 2.81 -> 4.92 mm
- net /PEnvelope: track 24.3 -> 22.7 mm
- net /Hard: track 158.2 -> 159.5 mm
- net /~IN: track 102.9 -> 104.0 mm
- net Net-(Q4-Pad2): track 18.1 -> 18.6 mm
Other:
- rule trace_min: 0.1524 -> 0
- board text added: "+12V"
- board text added: "-12V"
- board text added: "741 ADSR"
- board text added: "D"
- board text added: "Design by telec"
- board text added: "ENV"
- board text added: "GND"
- board text added: "Gate"
- board text added: "HRD"
- board text added: "R"
- board text added: "S"
- board text added: "Triggered"

Commit message: Added PCB ref stamp and send to prod!
Other:
- board text added: "PCB ref here:"
Changed lines of the file:
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@@
   (general
     (thickness 1.6)
-    (drawings 42)
+    (drawings 47)
     (tracks 366)
     (zones 0)
@@
   )
   (setup
-    (last_trace_width 0.508)
+    (last_trace_width 0.1524)
     (user_trace_width 0.1524)
     (user_trace_width 0.254)
@@
     )
   )
-  (gr_text -12V (at 30 12.7 90) (layer B.SilkS)
+  (gr_text "PCB ref here:" (at 24.6 12.9) (layer B.SilkS)
+    (effects (font (size 1 1) (thickness 0.15)) (justify mirror))
+  )
+  (gr_line (start 19 12) (end 19 16.3) (layer B.SilkS) (width 0.15))
+  (gr_line (start 30.4 12) (end 19 12) (layer B.SilkS) (width 0.15))
+  (gr_line (start 30.4 16.3) (end 30.4 12) (layer B.SilkS) (width 0.15))
+  (gr_line (start 19 16.3) (end 30.4 16.3) (layer B.SilkS) (width 0.15))
+  (gr_text -12V (at 30.2 28.1 135) (layer B.SilkS)
     (effects (font (size 2 2) (thickness 0.5)) (justify left mirror))
   )
-  (gr_text +12V (at 19.8 12.9 90) (layer B.SilkS)
+  (gr_text +12V (at 20.5 27.7 45) (layer B.SilkS)
     (effects (font (size 2 2) (thickness 0.5)) (justify left mirror))
   )
-  (gr_text GND (at 24.9 12.7 90) (layer B.SilkS)
+  (gr_text GND (at 20.8 29.6 180) (layer B.SilkS)
     (effects (font (size 2 2.8) (thickness 0.5)) (justify left mirror))
   )

Commit message: updated footprints on ADSR
Parts:
- J2, J3, J4: footprint telec:JackHole -> telec:Jack_Hole_Square
Routing:
- net /GATE: track 29.8 -> 34.8 mm
- net /Envelope: track 13.4 -> 17.3 mm
- net Net-(J3-PadT): track 2.51 -> 6.38 mm
- net GND: track 76.8 -> 73.9 mm
- net +12V: track 235.9 -> 233.4 mm

Commit message: ADSR ready for prod
Parts:
- R1: value 10k -> 47k
- R2: value 5k -> 15k
Changed lines of the file:
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@@
   )
   (setup
-    (last_trace_width 0.762)
+    (last_trace_width 0.1524)
     (user_trace_width 0.1524)
     (user_trace_width 0.254)
@@
       (effects (font (size 1 1) (thickness 0.15)) (justify mirror))
     )
-    (fp_text value 5k (at 1.8 0) (layer B.SilkS)
+    (fp_text value 15k (at 1.8 0) (layer B.SilkS)
       (effects (font (size 1 1) (thickness 0.15)) (justify mirror))
     )
@@
       (effects (font (size 1 1) (thickness 0.15)) (justify mirror))
     )
-    (fp_text value 10k (at 5.32 0) (layer B.SilkS)
-      (effects (font (size 1 1) (thickness 0.15)) (justify mirror))
-    )
+    (fp_text value 47k (at 5.32 0) (layer B.SilkS)
+      (effects (font (size 1 1) (thickness 0.15)) (justify mirror))
+    )
