File: ADSR/ADSR.sch (KiCad schematic (older format))
At the start: 47 parts, among them J1 EuroPower, J2 GATE, J3 Hard Envelope, J4 Envelope, Q1 BC557, Q2 BC547, Q3 BC547, Q4 BC547, U1 LM741, U2 LM741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

Commit message: Will it fits ?
Parts:
- removed J1: EuroPower, Connector_IDC:IDC-Header_2x05_P2.54mm_Vertical, symbol Connector_Generic:Conn_02x05_Odd_Even
- added H1, H2: Mounting_Holes, Kosmo_panel:Kosmo_Panel_Dual_Mounting_Holes, symbol Kosmo:Mounting_Holes
- added J1: EuroPower, telec:EuroPower, symbol Connector:Screw_Terminal_01x03
- D10, D11, D12, D9: footprint LED_THT:LED_D3.0mm -> LED_SMD:LED_1206_3216Metric_ReverseMount_Hole1.8x2.4mm
Connections:
- wire segments 118 -> 108
Other:
- note added: "Attack"
- note added: "Decay"
- note added: "Release"
- note added: "Sustain"
Changed lines of the file:
@@
-$EndComp
-$Comp
-L Connector_Generic:Conn_02x05_Odd_Even J1
-U 1 1 5F0BA5B1
-P 1150 2850
-F 0 "J1" H 1200 2425 50  0000 C CNN
-F 1 "EuroPower" H 1200 2516 50  0000 C CNN
-F 2 "Connector_IDC:IDC-Header_2x05_P2.54mm_Vertical" H 1150 2850 50  0001 C CNN
-F 3 "~" H 1150 2850 50  0001 C CNN
-	1    1150 2850
-	1    0    0    1
 $EndComp
 $Comp
 L power:-12V #PWR05
 U 1 1 5F0BB51F
-P 1550 3150
-F 0 "#PWR05" H 1550 3250 50  0001 C CNN
-F 1 "-12V" H 1565 3323 50  0000 C CNN
-F 2 "" H 1550 3150 50  0001 C CNN
-F 3 "" H 1550 3150 50  0001 C CNN
-	1    1550 3150
+P 1650 1150
+F 0 "#PWR05" H 1650 1250 50  0001 C CNN
+F 1 "-12V" H 1665 1323 50  0000 C CNN
+F 2 "" H 1650 1150 50  0001 C CNN
+F 3 "" H 1650 1150 50  0001 C CNN
+	1    1650 1150
 	-1   0    0    1
 $EndComp
@@
 L power:+12V #PWR04
 U 1 1 5F0BB646
-P 1550 2600
-F 0 "#PWR04" H 1550 2450 50  0001 C CNN
-F 1 "+12V" H 1565 2773 50  0000 C CNN
-F 2 "" H 1550 2600 50  0001 C CNN
-F 3 "" H 1550 2600 50  0001 C CNN
-	1    1550 2600
+P 1650 800
+F 0 "#PWR04" H 1650 650 50  0001 C CNN
+F 1 "+12V" H 1665 973 50  0000 C CNN
+F 2 "" H 1650 800 50  0001 C CNN
+F 3 "" H 1650 800 50  0001 C CNN
+	1    1650 800
 	1    0    0    -1
 $EndComp
@@
 L power:GND #PWR06
 U 1 1 5F0BC459
-P 1650 2900
-F 0 "#PWR06" H 1650 2650 50  0001 C CNN
-F 1 "GND" H 1655 2727 50  0000 C CNN
-F 2 "" H 1650 2900 50  0001 C CNN
-F 3 "" H 1650 2900 50  0001 C CNN
-	1    1650 2900
+P 1750 1000
+F 0 "#PWR06" H 1750 750 50  0001 C CNN
+F 1 "GND" H 1755 827 50  0000 C CNN
+F 2 "" H 1750 1000 50  0001 C CNN
+F 3 "" H 1750 1000 50  0001 C CNN
+	1    1750 1000
 	1    0    0    -1
 $EndComp
@@
 $EndComp
 Wire Wire Line
-	1450 2650 1550 2650
-Wire Wire Line
-	1550 2650 1550 2600
-Wire Wire Line
-	1450 2750 1450 2850
-Connection ~ 1450 2850
-Wire Wire Line
-	1450 2850 1450 2950
-Wire Wire Line
-	1450 2850 1650 2850
-Wire Wire Line
-	1650 2850 1650 2900
-Wire Wire Line
-	1450 3050 1550 3050
-Wire Wire Line
-	1550 3050 1550 3150
-$Comp
-L power:-12V #PWR03
-U 1 1 5F0D1780
-P 850 3150
-F 0 "#PWR03" H 850 3250 50  0001 C CNN
-F 1 "-12V" H 865 3323 50  0000 C CNN
-F 2 "" H 850 3150 50  0001 C CNN
-F 3 "" H 850 3150 50  0001 C CNN
-	1    850  3150
-	1    0    0    1
-$EndComp
-$Comp
-L power:+12V #PWR02
-U 1 1 5F0D1786
-P 850 2600
-F 0 "#PWR02" H 850 2450 50  0001 C CNN
-F 1 "+12V" H 865 2773 50  0000 C CNN
-F 2 "" H 850 2600 50  0001 C CNN
-F 3 "" H 850 2600 50  0001 C CNN
-	1    850  2600
-	-1   0    0    -1
-$EndComp
-$Comp
-L power:GND #PWR01
-U 1 1 5F0D178C
-P 750 2900
-F 0 "#PWR01" H 750 2650 50  0001 C CNN
-F 1 "GND" H 755 2727 50  0000 C CNN
-F 2 "" H 750 2900 50  0001 C CNN
-F 3 "" H 750 2900 50  0001 C CNN
-	1    750  2900
-	-1   0    0    -1
-$EndComp
-Wire Wire Line
-	950  2650 850  2650
-Wire Wire Line
-	850  2650 850  2600
-Wire Wire Line
-	950  2850 750  2850
-Wire Wire Line
-	750  2850 750  2900
-Wire Wire Line
-	950  3050 850  3050
-Wire Wire Line
-	850  3050 850  3150
-Wire Wire Line
-	950  2950 950  2850
-Connection ~ 950  2850
-Wire Wire Line
-	950  2850 950  2750
+	1550 850  1650 850
+Wire Wire Line
+	1650 850  1650 800
+Wire Wire Line
+	1550 950  1750 950
+Wire Wire Line
+	1750 950  1750 1000
+Wire Wire Line
+	1550 1050 1650 1050
+Wire Wire Line
+	1650 1050 1650 1150
 NoConn ~ 2400 4750
 NoConn ~ 2400 4850
@@
 F 0 "D10" V 10039 1483 50  0000 R CNN
 F 1 "LED" V 9948 1483 50  0000 R CNN
-F 2 "LED_THT:LED_D3.0mm" H 10000 1600 50  0001 C CNN
+F 2 "LED_SMD:LED_1206_3216Metric_ReverseMount_Hole1.8x2.4mm" H 10000 1600 50  0001 C CNN
 F 3 "~" H 10000 1600 50  0001 C CNN
 	1    10000 1600
@@
 F 0 "D11" V 10389 1483 50  0000 R CNN
 F 1 "LED" V 10298 1483 50  0000 R CNN
-F 2 "LED_THT:LED_D3.0mm" H 10350 1600 50  0001 C CNN
+F 2 "LED_SMD:LED_1206_3216Metric_ReverseMount_Hole1.8x2.4mm" H 10350 1600 50  0001 C CNN
 F 3 "~" H 10350 1600 50  0001 C CNN
 	1    10350 1600
@@
 F 0 "D12" V 10739 1483 50  0000 R CNN
 F 1 "LED" V 10648 1483 50  0000 R CNN
-F 2 "LED_THT:LED_D3.0mm" H 10700 1600 50  0001 C CNN
+F 2 "LED_SMD:LED_1206_3216Metric_ReverseMount_Hole1.8x2.4mm" H 10700 1600 50  0001 C CNN
 F 3 "~" H 10700 1600 50  0001 C CNN
 	1    10700 1600
@@
 F 0 "D9" V 9689 1483 50  0000 R CNN
 F 1 "LED" V 9598 1483 50  0000 R CNN
-F 2 "LED_THT:LED_D3.0mm" H 9650 1600 50  0001 C CNN
+F 2 "LED_SMD:LED_1206_3216Metric_ReverseMount_Hole1.8x2.4mm" H 9650 1600 50  0001 C CNN
 F 3 "~" H 9650 1600 50  0001 C CNN
 	1    9650 1600
@@
 Text Label 9650 750  3    50   ~ 0
 IN
+$Comp
+L Connector:Screw_Terminal_01x03 J1
+U 1 1 5FC53096
+P 1350 950
+F 0 "J1" H 1268 625 50  0000 C CNN
+F 1 "EuroPower" H 1268 716 50  0000 C CNN
+F 2 "telec:EuroPower" H 1350 950 50  0001 C CNN
+F 3 "~" H 1350 950 50  0001 C CNN
+	1    1350 950
+	-1   0    0    1
+$EndComp
+$Comp
+L power:+12V #PWR0101
+U 1 1 5FC8D2DC
+P 600 900
+F 0 "#PWR0101" H 600 750 50  0001 C CNN
+F 1 "+12V" H 615 1073 50  0000 C CNN
+F 2 "" H 600 900 50  0001 C CNN
+F 3 "" H 600 900 50  0001 C CNN
+	1    600  900
+	1    0    0    -1
+$EndComp
+$Comp
+L power:GND #PWR0102
+U 1 1 5FC8D87A
+P 800 900
+F 0 "#PWR0102" H 800 650 50  0001 C CNN
+F 1 "GND" H 805 727 50  0000 C CNN
+F 2 "" H 800 900 50  0001 C CNN
+F 3 "" H 800 900 50  0001 C CNN
+	1    800  900
+	1    0    0    -1
+$EndComp
+$Comp
+L power:-12V #PWR0103
+U 1 1 5FC8DD79
+P 1000 900
+F 0 "#PWR0103" H 1000 1000 50  0001 C CNN
+F 1 "-12V" H 1015 1073 50  0000 C CNN
+F 2 "" H 1000 900 50  0001 C CNN
+F 3 "" H 1000 900 50  0001 C CNN
+	1    1000 900
+	-1   0    0    1
+$EndComp
+$Comp
+L power:PWR_FLAG #FLG0101
+U 1 1 5FC92121
+P 800 900
+F 0 "#FLG0101" H 800 975 50  0001 C CNN
+F 1 "PWR_FLAG" H 800 1073 50  0000 C CNN
+F 2 "" H 800 900 50  0001 C CNN
+F 3 "~" H 800 900 50  0001 C CNN
+	1    800  900
+	1    0    0    -1
+$EndComp
+$Comp
+L power:PWR_FLAG #FLG0102
+U 1 1 5FC92A56
+P 1000 900
+F 0 "#FLG0102" H 1000 975 50  0001 C CNN
+F 1 "PWR_FLAG" H 1000 1073 50  0000 C CNN
+F 2 "" H 1000 900 50  0001 C CNN
+F 3 "~" H 1000 900 50  0001 C CNN
+	1    1000 900
+	1    0    0    -1
+$EndComp
+$Comp
+L power:PWR_FLAG #FLG0103
+U 1 1 5FC92DDD
+P 600 900
+F 0 "#FLG0103" H 600 975 50  0001 C CNN
+F 1 "PWR_FLAG" H 600 1073 50  0000 C CNN
+F 2 "" H 600 900 50  0001 C CNN
+F 3 "~" H 600 900 50  0001 C CNN
+	1    600  900
+	-1   0    0    1
+$EndComp
+$Comp
+L Kosmo:Mounting_Holes H1
+U 1 1 5FCA465F
+P 1050 6900
+F 0 "H1" H 1000 6950 50  0000 L CNN
+F 1 "Mounting_Holes" V 900 6600 50  0000 L CNN
+F 2 "Kosmo_panel:Kosmo_Panel_Dual_Mounting_Holes" H 1050 6900 50  0001 C CNN
+F 3 "" H 1050 6900 50  0001 C CNN
+	1    1050 6900
+	1    0    0    -1
+$EndComp
+$Comp
+L power:GND #PWR0104
+U 1 1 5FCA5AE3
+P 1050 7250
+F 0 "#PWR0104" H 1050 7000 50  0001 C CNN
+F 1 "GND" H 1055 7077 50  0000 C CNN
+F 2 "" H 1050 7250 50  0001 C CNN
+F 3 "" H 1050 7250 50  0001 C CNN
+	1    1050 7250
+	1    0    0    -1
+$EndComp
+$Comp
+L Kosmo:Mounting_Holes H2
+U 1 1 5FCA86D9
+P 1400 6900
+F 0 "H2" H 1350 6950 50  0000 L CNN
+F 1 "Mounting_Holes" V 1250 6600 50  0000 L CNN
+F 2 "Kosmo_panel:Kosmo_Panel_Dual_Mounting_Holes" H 1400 6900 50  0001 C CNN
+F 3 "" H 1400 6900 50  0001 C CNN
+	1    1400 6900
+	1    0    0    -1
+$EndComp
+$Comp
+L power:GND #PWR0105
+U 1 1 5FCA86DF
+P 1400 7250
+F 0 "#PWR0105" H 1400 7000 50  0001 C CNN
+F 1 "GND" H 1405 7077 50  0000 C CNN
+F 2 "" H 1400 7250 50  0001 C CNN
+F 3 "" H 1400 7250 50  0001 C CNN
+	1    1400 7250
+	1    0    0    -1
+$EndComp
+Text Notes 7550 2250 0    50   ~ 0
+Attack
+Text Notes 4650 2200 0    50   ~ 0
+Sustain
+Text Notes 7550 2750 0    50   ~ 0
+Decay
+Text Notes 8200 2600 0    50   ~ 0
+Release
 $EndSCHEMATC

Commit message: It fits !
Parts:
- RV1, RV2, RV3, RV4: footprint Potentiometer_THT:Potentiometer_Piher_T-16L_Single_Vertical_Hole -> Potentiometer_THT:Potentiometer_Alps_RK09K_Single_Vertical
Changed lines of the file:
@@
 F 0 "RV2" V 7550 2450 50  0000 C CNN
 F 1 "100k" V 7650 2450 50  0000 C CNN
-F 2 "Potentiometer_THT:Potentiometer_Piher_T-16L_Single_Vertical_Hole" H 7650 2450 50  0001 C CNN
+F 2 "Potentiometer_THT:Potentiometer_Alps_RK09K_Single_Vertical" H 7650 2450 50  0001 C CNN
 F 3 "~" H 7650 2450 50  0001 C CNN
 	1    7650 2450
@@
 F 0 "RV3" V 7550 2900 50  0000 C CNN
 F 1 "100k" V 7650 2900 50  0000 C CNN
-F 2 "Potentiometer_THT:Potentiometer_Piher_T-16L_Single_Vertical_Hole" H 7650 2900 50  0001 C CNN
+F 2 "Potentiometer_THT:Potentiometer_Alps_RK09K_Single_Vertical" H 7650 2900 50  0001 C CNN
 F 3 "~" H 7650 2900 50  0001 C CNN
 	1    7650 2900
@@
 F 0 "RV1" H 4950 2700 50  0000 R CNN
 F 1 "100k" V 4750 2700 50  0000 R CNN
-F 2 "Potentiometer_THT:Potentiometer_Piher_T-16L_Single_Vertical_Hole" H 4750 2600 50  0001 C CNN
+F 2 "Potentiometer_THT:Potentiometer_Alps_RK09K_Single_Vertical" H 4750 2600 50  0001 C CNN
 F 3 "~" H 4750 2600 50  0001 C CNN
 	1    4750 2600
@@
 F 0 "RV4" H 8230 3046 50  0000 R CNN
 F 1 "100k" V 8300 3100 50  0000 R CNN
-F 2 "Potentiometer_THT:Potentiometer_Piher_T-16L_Single_Vertical_Hole" H 8300 3000 50  0001 C CNN
+F 2 "Potentiometer_THT:Potentiometer_Alps_RK09K_Single_Vertical" H 8300 3000 50  0001 C CNN
 F 3 "~" H 8300 3000 50  0001 C CNN
 	1    8300 3000

Commit message: Now the power lines...
Parts:
- R13, R14: footprint Resistor_THT:R_Axial_DIN0204_L3.6mm_D1.6mm_P7.62mm_Horizontal -> Resistor_SMD:R_1206_3216Metric
- R15, R16: value 1k5 -> 2k2; footprint Resistor_THT:R_Axial_DIN0204_L3.6mm_D1.6mm_P7.62mm_Horizontal -> Resistor_SMD:R_1206_3216Metric
Connections:
- net GND: now also D9.2 (A); no longer D9.1 (K)
- net IN: no longer R13.1
- net ~IN: now also R13.1
- net at R13.2: now also D9.1 (K); no longer D9.2 (A)
Other:
- moved on the sheet: D9
Changed lines of the file:
@@
 F 0 "R14" H 10070 1346 50  0000 L CNN
 F 1 "1k5" V 10000 1250 50  0000 L CNN
-F 2 "Resistor_THT:R_Axial_DIN0204_L3.6mm_D1.6mm_P7.62mm_Horizontal" V 9930 1300 50  0001 C CNN
+F 2 "Resistor_SMD:R_1206_3216Metric" V 9930 1300 50  0001 C CNN
 F 3 "~" H 10000 1300 50  0001 C CNN
 	1    10000 1300
@@
 P 10350 1300
 F 0 "R15" H 10420 1346 50  0000 L CNN
-F 1 "1k5" V 10350 1250 50  0000 L CNN
-F 2 "Resistor_THT:R_Axial_DIN0204_L3.6mm_D1.6mm_P7.62mm_Horizontal" V 10280 1300 50  0001 C CNN
+F 1 "2k2" V 10350 1250 50  0000 L CNN
+F 2 "Resistor_SMD:R_1206_3216Metric" V 10280 1300 50  0001 C CNN
 F 3 "~" H 10350 1300 50  0001 C CNN
 	1    10350 1300
@@
 P 10700 1300
 F 0 "R16" H 10770 1346 50  0000 L CNN
-F 1 "1k5" V 10700 1250 50  0000 L CNN
-F 2 "Resistor_THT:R_Axial_DIN0204_L3.6mm_D1.6mm_P7.62mm_Horizontal" V 10630 1300 50  0001 C CNN
+F 1 "2k2" V 10700 1250 50  0000 L CNN
+F 2 "Resistor_SMD:R_1206_3216Metric" V 10630 1300 50  0001 C CNN
 F 3 "~" H 10700 1300 50  0001 C CNN
 	1    10700 1300
@@
 F 3 "~" H 9650 1600 50  0001 C CNN
 	1    9650 1600
-	0    -1   -1   0
+	0    1    1    0
 $EndComp
 $Comp
@@
 F 0 "R13" H 9720 1346 50  0000 L CNN
 F 1 "1k5" V 9650 1250 50  0000 L CNN
-F 2 "Resistor_THT:R_Axial_DIN0204_L3.6mm_D1.6mm_P7.62mm_Horizontal" V 9580 1300 50  0001 C CNN
+F 2 "Resistor_SMD:R_1206_3216Metric" V 9580 1300 50  0001 C CNN
 F 3 "~" H 9650 1300 50  0001 C CNN
 	1    9650 1300
@@
 	9650 1150 9650 750
 Text Label 9650 750  3    50   ~ 0
-IN
+~IN
 $Comp
 L Connector:Screw_Terminal_01x03 J1

Commit message: Layout done! Art to do
Parts:
- added R17, R18: 1k, Resistor_THT:R_Axial_DIN0204_L3.6mm_D1.6mm_P7.62mm_Horizontal, symbol Device:R
Connections:
- net Envelope: now also R17.2; no longer R16.1, U5.6
- net GND: now also D9.1 (K); no longer D9.2 (A)
- net Hard: now also R18.1; no longer J3.T
- net IN: now also R13.1
- net ~IN: no longer R13.1
- net at R13.2: now also D9.2 (A); no longer D9.1 (K)
- new net: J3.T, R18.2
- new net PEnvelope: R16.1, R17.1, U5.6
Other:
- moved on the sheet: D9
Changed lines of the file:
@@
 $EndComp
 Wire Wire Line
-	9600 2800 9700 2800
-Wire Wire Line
-	9700 3350 8900 3350
+	10250 3350 8900 3350
 Wire Wire Line
 	8900 3350 8900 2900
@@
 	8900 2900 9000 2900
 Wire Wire Line
-	9700 3350 9700 2800
+	10250 3350 10250 2800
 $Comp
 L power:+12V #PWR013
@@
 Text Label 6350 2700 0    50   ~ 0
 Hard
-Text Label 10050 2800 2    50   ~ 0
+Text Label 10600 2800 2    50   ~ 0
 Envelope
 Text Label 8400 2700 0    50   ~ 0
@@
 Connection ~ 8650 2700
 Wire Wire Line
-	9700 2800 10050 2800
-Connection ~ 9700 2800
-Text Label 9050 5800 0    50   ~ 0
+	10250 2800 10600 2800
+Connection ~ 10250 2800
+Text Label 8700 5800 0    50   ~ 0
 Envelope
 Wire Wire Line
-	9400 5800 9050 5800
+	9400 5800 8700 5800
 NoConn ~ 9400 5900
 NoConn ~ 9400 5700
@@
 Wire Wire Line
 	9300 5400 9300 5450
-Text Label 9050 4850 0    50   ~ 0
+Text Label 8700 4850 0    50   ~ 0
 Hard
-Wire Wire Line
-	9400 4850 9050 4850
 NoConn ~ 9400 4950
 NoConn ~ 9400 4750
@@
 Wire Wire Line
 	10700 1150 10700 750
-Text Label 10700 750  3    50   ~ 0
-Envelope
 $Comp
 L Device:LED D9
@@
 F 3 "~" H 9650 1600 50  0001 C CNN
 	1    9650 1600
-	0    1    1    0
+	0    -1   -1   0
 $EndComp
 $Comp
@@
 	9650 1150 9650 750
 Text Label 9650 750  3    50   ~ 0
-~IN
+IN
 $Comp
 L Connector:Screw_Terminal_01x03 J1
@@
 Text Notes 8200 2600 0    50   ~ 0
 Release
+$Comp
+L Device:R R17
+U 1 1 6055851E
+P 9950 2800
+F 0 "R17" V 10050 2800 50  0000 C CNN
+F 1 "1k" V 9950 2800 50  0000 C CNN
+F 2 "Resistor_THT:R_Axial_DIN0204_L3.6mm_D1.6mm_P7.62mm_Horizontal" V 9880 2800 50  0001 C CNN
+F 3 "~" H 9950 2800 50  0001 C CNN
+	1    9950 2800
+	0    -1   1    0
+$EndComp
+Wire Wire Line
+	10100 2800 10250 2800
+$Comp
+L Device:R R18
+U 1 1 6055A415
+P 9100 4850
+F 0 "R18" V 9200 4850 50  0000 C CNN
+F 1 "1k" V 9100 4850 50  0000 C CNN
+F 2 "Resistor_THT:R_Axial_DIN0204_L3.6mm_D1.6mm_P7.62mm_Horizontal" V 9030 4850 50  0001 C CNN
+F 3 "~" H 9100 4850 50  0001 C CNN
+	1    9100 4850
+	0    -1   1    0
+$EndComp
+Wire Wire Line
+	8700 4850 8950 4850
+Wire Wire Line
+	9250 4850 9400 4850
+Text Label 10700 750  3    50   ~ 0
+PEnvelope
+Wire Wire Line
+	9600 2800 9700 2800
+Wire Wire Line
+	9700 2800 9700 2650
+Wire Wire Line
+	9700 2650 10100 2650
+Connection ~ 9700 2800
+Wire Wire Line
+	9700 2800 9800 2800
+Text Label 10100 2650 2    50   ~ 0
+PEnvelope
 $EndSCHEMATC

Commit message: ADSR done !
Parts:
- added LOGO1: Logo_telec, logo:telec-8, symbol logo:Logo_telec
Other:
- note added: "Buffer +\ncompensate for the\nvoltage drop of D7/D8"
- note added: "Hysteresis circuit\nwith reset input"
- note added: "Output buffer"
- note added: "Overidable\nsustain level"
- note added: "Simple comparators"
Changed lines of the file:
@@
 Text Notes 7550 2250 0    50   ~ 0
 Attack
-Text Notes 4650 2200 0    50   ~ 0
+Text Notes 4800 2700 0    50   ~ 0
 Sustain
 Text Notes 7550 2750 0    50   ~ 0
 Decay
-Text Notes 8200 2600 0    50   ~ 0
+Text Notes 8300 3200 0    50   ~ 0
 Release
 $Comp
@@
 Text Label 10100 2650 2    50   ~ 0
 PEnvelope
+Text Notes 3350 3950 0    50   ~ 0
+Simple comparators
+Text Notes 3800 1600 0    50   ~ 0
+Hysteresis circuit\nwith reset input
+Text Notes 4650 2100 0    50   ~ 0
+Overidable\nsustain level
+Text Notes 5650 2150 0    50   ~ 0
+Buffer +\ncompensate for the\nvoltage drop of D7/D8
+Text Notes 9650 3300 0    50   ~ 0
+Output buffer
+$Comp
+L logo:Logo_telec LOGO1
+U 1 1 605DA57A
+P 1900 6950
+F 0 "LOGO1" H 1890 7247 50  0001 C CNN
+F 1 "Logo_telec" H 1897 7174 50  0001 C CNN
+F 2 "logo:telec-8" H 1900 7350 50  0001 C CNN
+F 3 "" H 1900 7350 50  0001 C CNN
+	1    1900 6950
+	1    0    0    -1
+$EndComp
 $EndSCHEMATC

Commit message: updated footprints on ADSR
Parts:
- J2, J3, J4: footprint telec:JackHole -> telec:Jack_Hole_Square; symbol Connector:AudioJack3_Switch -> Connector:AudioJack3_SwitchTR
Connections:
- no-connect marks 21 -> 18
Changed lines of the file:
@@
 $EndComp
 $Comp
-L Connector:AudioJack3_Switch J2
+L Connector:AudioJack3_SwitchTR J2
 U 1 1 5F0BD040
 P 2200 4850
-F 0 "J2" H 2182 5275 50  0000 C CNN
-F 1 "GATE" H 2182 5184 50  0000 C CNN
-F 2 "telec:JackHole" H 2200 4850 50  0001 C CNN
+F 0 "J2" H 2150 5150 50  0000 C CNN
+F 1 "GATE" H 2150 5050 50  0000 C CNN
+F 2 "telec:Jack_Hole_Square" H 2200 4850 50  0001 C CNN
 F 3 "~" H 2200 4850 50  0001 C CNN
 	1    2200 4850
@@
 $EndComp
 $Comp
-L Connector:AudioJack3_Switch J4
+L Connector:AudioJack3_SwitchTR J4
 U 1 1 5F0C1568
 P 9600 5600
 F 0 "J4" H 9320 5600 50  0000 R CNN
 F 1 "Envelope" H 9320 5509 50  0000 R CNN
-F 2 "telec:JackHole" H 9600 5600 50  0001 C CNN
+F 2 "telec:Jack_Hole_Square" H 9600 5600 50  0001 C CNN
 F 3 "~" H 9600 5600 50  0001 C CNN
 	1    9600 5600
@@
 $EndComp
 $Comp
-L Connector:AudioJack3_Switch J3
+L Connector:AudioJack3_SwitchTR J3
 U 1 1 5F0C434F
 P 9600 4650
 F 0 "J3" H 9320 4650 50  0000 R CNN
 F 1 "Hard Envelope" H 9320 4559 50  0000 R CNN
-F 2 "telec:JackHole" H 9600 4650 50  0001 C CNN
+F 2 "telec:Jack_Hole_Square" H 9600 4650 50  0001 C CNN
 F 3 "~" H 9600 4650 50  0001 C CNN
 	1    9600 4650
@@
 Wire Wire Line
 	1650 1050 1650 1150
-NoConn ~ 2400 4750
 NoConn ~ 2400 4850
 NoConn ~ 2400 4950
@@
 L power:GND #PWR07
 U 1 1 5F0D2E83
-P 2500 4700
-F 0 "#PWR07" H 2500 4450 50  0001 C CNN
-F 1 "GND" H 2505 4527 50  0000 C CNN
-F 2 "" H 2500 4700 50  0001 C CNN
-F 3 "" H 2500 4700 50  0001 C CNN
-	1    2500 4700
-	1    0    0    -1
-$EndComp
-Wire Wire Line
-	2400 4650 2500 4650
-Wire Wire Line
-	2500 4650 2500 4700
+P 2500 4750
+F 0 "#PWR07" H 2500 4500 50  0001 C CNN
+F 1 "GND" H 2505 4577 50  0000 C CNN
+F 2 "" H 2500 4750 50  0001 C CNN
+F 3 "" H 2500 4750 50  0001 C CNN
+	1    2500 4750
+	1    0    0    -1
+$EndComp
+Wire Wire Line
+	2400 4750 2500 4750
 $Comp
 L power:+12V #PWR014
@@
 NoConn ~ 9400 5700
 NoConn ~ 9400 5600
-NoConn ~ 9400 5500
 $Comp
 L power:GND #PWR033
 U 1 1 5F2725F7
-P 9300 5450
-F 0 "#PWR033" H 9300 5200 50  0001 C CNN
-F 1 "GND" H 9305 5277 50  0000 C CNN
-F 2 "" H 9300 5450 50  0001 C CNN
-F 3 "" H 9300 5450 50  0001 C CNN
-	1    9300 5450
+P 9300 5550
+F 0 "#PWR033" H 9300 5300 50  0001 C CNN
+F 1 "GND" H 9305 5377 50  0000 C CNN
+F 2 "" H 9300 5550 50  0001 C CNN
+F 3 "" H 9300 5550 50  0001 C CNN
+	1    9300 5550
 	-1   0    0    -1
 $EndComp
 Wire Wire Line
-	9400 5400 9300 5400
-Wire Wire Line
-	9300 5400 9300 5450
+	9400 5500 9300 5500
+Wire Wire Line
+	9300 5500 9300 5550
 Text Label 8700 4850 0    50   ~ 0
 Hard
@@
 NoConn ~ 9400 4750
 NoConn ~ 9400 4650
-NoConn ~ 9400 4550
 $Comp
 L power:GND #PWR032
 U 1 1 5F275C32
-P 9300 4500
-F 0 "#PWR032" H 9300 4250 50  0001 C CNN
-F 1 "GND" H 9305 4327 50  0000 C CNN
-F 2 "" H 9300 4500 50  0001 C CNN
-F 3 "" H 9300 4500 50  0001 C CNN
-	1    9300 4500
+P 9300 4600
+F 0 "#PWR032" H 9300 4350 50  0001 C CNN
+F 1 "GND" H 9305 4427 50  0000 C CNN
+F 2 "" H 9300 4600 50  0001 C CNN
+F 3 "" H 9300 4600 50  0001 C CNN
+	1    9300 4600
 	-1   0    0    -1
 $EndComp
 Wire Wire Line
-	9400 4450 9300 4450
-Wire Wire Line
-	9300 4450 9300 4500
+	9400 4550 9300 4550
+Wire Wire Line
+	9300 4550 9300 4600
 Wire Wire Line
 	3500 2700 3300 2700

Commit message: ADSR ready for prod
Parts:
- R1: value 10k -> 47k
- R2: value 5k -> 15k
Other:
- moved on the sheet: J2
Changed lines of the file:
@@
 P 3050 4900
 F 0 "R1" H 3120 4946 50  0000 L CNN
-F 1 "10k" H 3120 4855 50  0000 L CNN
+F 1 "47k" H 3120 4855 50  0000 L CNN
 F 2 "Resistor_THT:R_Axial_DIN0204_L3.6mm_D1.6mm_P7.62mm_Horizontal" V 2980 4900 50  0001 C CNN
 F 3 "~" H 3050 4900 50  0001 C CNN
@@
 L Connector:AudioJack3_SwitchTR J2
 U 1 1 5F0BD040
-P 2200 4850
-F 0 "J2" H 2150 5150 50  0000 C CNN
-F 1 "GATE" H 2150 5050 50  0000 C CNN
-F 2 "telec:Jack_Hole_Square" H 2200 4850 50  0001 C CNN
-F 3 "~" H 2200 4850 50  0001 C CNN
-	1    2200 4850
+P 2200 4900
+F 0 "J2" H 2150 5200 50  0000 C CNN
+F 1 "GATE" H 2150 5100 50  0000 C CNN
+F 2 "telec:Jack_Hole_Square" H 2200 4900 50  0001 C CNN
+F 3 "~" H 2200 4900 50  0001 C CNN
+	1    2200 4900
 	1    0    0    -1
 $EndComp
@@
 Wire Wire Line
 	1650 1050 1650 1150
-NoConn ~ 2400 4850
-NoConn ~ 2400 4950
+NoConn ~ 2400 4900
+NoConn ~ 2400 5000
 $Comp
 L power:GND #PWR07
 U 1 1 5F0D2E83
-P 2500 4750
-F 0 "#PWR07" H 2500 4500 50  0001 C CNN
-F 1 "GND" H 2505 4577 50  0000 C CNN
-F 2 "" H 2500 4750 50  0001 C CNN
-F 3 "" H 2500 4750 50  0001 C CNN
-	1    2500 4750
-	1    0    0    -1
-$EndComp
-Wire Wire Line
-	2400 4750 2500 4750
+P 2500 4800
+F 0 "#PWR07" H 2500 4550 50  0001 C CNN
+F 1 "GND" H 2505 4627 50  0000 C CNN
+F 2 "" H 2500 4800 50  0001 C CNN
+F 3 "" H 2500 4800 50  0001 C CNN
+	1    2500 4800
+	1    0    0    -1
+$EndComp
+Wire Wire Line
+	2400 4800 2500 4800
 $Comp
 L power:+12V #PWR014
@@
 P 3050 5300
 F 0 "R2" H 3120 5346 50  0000 L CNN
-F 1 "5k" H 3120 5255 50  0000 L CNN
+F 1 "15k" H 3120 5255 50  0000 L CNN
 F 2 "Resistor_THT:R_Axial_DIN0204_L3.6mm_D1.6mm_P7.62mm_Horizontal" V 2980 5300 50  0001 C CNN
 F 3 "~" H 3050 5300 50  0001 C CNN
@@
 	3350 4450 2900 4450
 Wire Wire Line
-	2900 4450 2900 5050
-Wire Wire Line
 	2900 5750 3350 5750
 Wire Wire Line
-	2400 5050 2900 5050
-Connection ~ 2900 5050
-Wire Wire Line
-	2900 5050 2900 5750
-Text Label 2600 5050 0    50   ~ 0
+	2400 5100 2900 5100
+Text Label 2600 5100 0    50   ~ 0
 GATE
 $Comp
 L power:GND #PWR08
 U 1 1 5F0E8429
-P 2500 5200
-F 0 "#PWR08" H 2500 4950 50  0001 C CNN
-F 1 "GND" H 2505 5027 50  0000 C CNN
-F 2 "" H 2500 5200 50  0001 C CNN
-F 3 "" H 2500 5200 50  0001 C CNN
-	1    2500 5200
-	1    0    0    -1
-$EndComp
-Wire Wire Line
-	2400 5150 2500 5150
-Wire Wire Line
-	2500 5150 2500 5200
+P 2500 5250
+F 0 "#PWR08" H 2500 5000 50  0001 C CNN
+F 1 "GND" H 2505 5077 50  0000 C CNN
+F 2 "" H 2500 5250 50  0001 C CNN
+F 3 "" H 2500 5250 50  0001 C CNN
+	1    2500 5250
+	1    0    0    -1
+$EndComp
+Wire Wire Line
+	2400 5200 2500 5200
+Wire Wire Line
+	2500 5200 2500 5250
 $Comp
 L Device:R R5
@@
 	1    0    0    -1
 $EndComp
+Connection ~ 2900 5100
+Wire Wire Line
+	2900 5100 2900 5750
+Wire Wire Line
+	2900 4450 2900 5100
 $EndSCHEMATC
