File: ADSR/ADSR.sch (KiCad schematic (older format))
At the start: 52 parts, among them J1 EuroPower, J2 GATE, J3 Hard Envelope, J4 Envelope, Q1 BC557, Q2 BC547, Q3 BC547, Q4 BC547, U1 LM741, U2 LM741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

Commit message: More clearance
Parts:
- J3: footprint telec:Jack_Hole_Square -> Connector_PinSocket_2.54mm:PinSocket_1x01_P2.54mm_Vertical; symbol Connector:AudioJack3_SwitchTR -> Connector:Conn_01x01_Female
Connections:
- net GND: no longer J3.S
- net at R18.2: now also J3.1 (Pin_1); no longer J3.T
Other:
- note added: "Not enough room\nfor that..."
Changed lines of the file:
@@
 $EndComp
 $Comp
-L Connector:AudioJack3_SwitchTR J3
+L Connector:Conn_01x01_Female J3
 U 1 1 5F0C434F
-P 9600 4650
-F 0 "J3" H 9320 4650 50  0000 R CNN
-F 1 "Hard Envelope" H 9320 4559 50  0000 R CNN
-F 2 "telec:Jack_Hole_Square" H 9600 4650 50  0001 C CNN
-F 3 "~" H 9600 4650 50  0001 C CNN
-	1    9600 4650
-	-1   0    0    -1
+P 9600 4850
+F 0 "J3" H 9750 4800 50  0000 R CNN
+F 1 "Hard Envelope" H 10200 4900 50  0000 R CNN
+F 2 "Connector_PinSocket_2.54mm:PinSocket_1x01_P2.54mm_Vertical" H 9600 4850 50  0001 C CNN
+F 3 "~" H 9600 4850 50  0001 C CNN
+	1    9600 4850
+	1    0    0    1
 $EndComp
 Wire Wire Line
@@
 Wire Wire Line
 	2900 4450 2900 5100
+Text Notes 9650 4550 0    50   ~ 0
+Not enough room\nfor that...
 $EndSCHEMATC
