File: Lights/Lights.kicad_pcb (KiCad board)
At the start: 2 copper layers, 102.5 x 200 mm, 127 parts, among them J101 chain_in, J102 chain_out, J103 Input1, J104 Input2, J105 Input3, J106 THRU, J107 OUT, J108 IN, J109 EuroPower, J110 ExternalPower, J111 Programming, J112 chain_power, J401 Light, J701 Light, J801 Light, Q401 PN2222A, Q402 IRF540N, Q701 PN2222A, Q702 IRF540N, Q801 PN2222A, Q802 IRF540N, SW101 MIDI_settings, U101 L7805, U102 L7805, U103 ATmega328P-PU, U201 TL074, U301 74LS04, U302 6N138, U401 6N138, U501 TL074, U601 TL074, U701 6N138, U801 6N138, Y101 16MHz

Commit message: Small fixes+firmware
Parts:
- moved J110 10.1 mm to (111.1, 29.0), turned to 180 degrees
Connections:
- D101 pad 2: -VDC -> Net-(D101-Pad2)
- D101 pad 3: Net-(D101-Pad3) -> -VDC
- J110 pad 1: Net-(D101-Pad4) -> Net-(D101-Pad2)
- J110 pad 3: Net-(D101-Pad3) -> Net-(D101-Pad4)
- R101 pad 1: +12V -> +5V
- R102 pad 1: +12V -> +5V
Routing:
- net +12V: track 299.3 -> 275.4 mm
- net -VDC: track 97.7 -> 89.6 mm
- net Net-(D101-Pad3): track 6.60 -> 0.00 mm

Commit message: Switched to kicad 7 + small fixes
Parts:
- H112, H113, H114: footprint MountingHole:MountingHole_6mm_Pad -> Kosmo_panel:Kosmo_Jack_Hole
- R306: value 220 -> 2k2
- moved D102 26.2 mm to (94.2, 173.2)
- moved D103 26.2 mm to (94.2, 147.0)
- moved R101 26.2 mm to (101.5, 173.2)
- moved R102 26.2 mm to (101.5, 147.0)
- moved SW101 10.7 mm to (73.1, 94.7), turned to 0 degrees
- moved D101 5.06 mm to (103.2, 34.5), turned to 0 degrees
Connections:
- net /~RESET renamed /~{RESET}
- D101 pad 2: Net-(D101-Pad2) -> Net-(J110-Pin_3)
- D101 pad 4: Net-(D101-Pad4) -> Net-(J110-Pin_1)
- J103 pad R: Net-(J103-PadR) -> unconnected-(J103-PadR)
- J103 pad RN: Net-(J103-PadRN) -> unconnected-(J103-PadRN)
- J104 pad R: Net-(J104-PadR) -> unconnected-(J104-PadR)
- J104 pad RN: Net-(J104-PadRN) -> unconnected-(J104-PadRN)
- J105 pad R: Net-(J105-PadR) -> unconnected-(J105-PadR)
- J105 pad RN: Net-(J105-PadRN) -> unconnected-(J105-PadRN)
- J108 pad S: Net-(J108-PadS) -> unconnected-(J108-PadS)
- J110 pad 1: Net-(D101-Pad2) -> Net-(J110-Pin_1)
- J110 pad 3: Net-(D101-Pad4) -> Net-(J110-Pin_3)
- SW101 pad 1: Net-(SW101-Pad1) -> GND
- SW101 pad 2: Net-(SW101-Pad2) -> GND
- SW101 pad 3: Net-(SW101-Pad3) -> GND
- SW101 pad 4: Net-(SW101-Pad4) -> GND
- SW101 pad 5: GND -> Net-(U103-PD7)
- SW101 pad 6: GND -> Net-(U103-PD6)
- SW101 pad 7: GND -> Net-(U103-PD5)
- SW101 pad 8: GND -> Net-(U103-PD4)
- U103 pad 11: Net-(SW101-Pad3) -> Net-(U103-PD5)
- U103 pad 12: Net-(SW101-Pad2) -> Net-(U103-PD6)
- U103 pad 13: Net-(SW101-Pad1) -> Net-(U103-PD7)
- U103 pad 14: Net-(U103-Pad14) -> unconnected-(U103-PB0-Pad14)
- U103 pad 26: Net-(U103-Pad26) -> unconnected-(U103-PC3-Pad26)
- U103 pad 27: Net-(U103-Pad27) -> unconnected-(U103-PC4-Pad27)
- U103 pad 28: Net-(U103-Pad28) -> unconnected-(U103-PC5-Pad28)
- U103 pad 4: Net-(U103-Pad4) -> unconnected-(U103-PD2-Pad4)
- U103 pad 6: Net-(SW101-Pad4) -> Net-(U103-PD4)
Routing:
- net +5V: track 140.6 -> 276.1 mm, vias 4 -> 11
- net /MIDI_OUT: track 90.3 -> 138.2 mm, vias 4 -> 6
- net Net-(U103-PD6): track 0.00 -> 36.8 mm
- net Net-(U103-PD5): track 0.00 -> 36.8 mm
- net Net-(SW101-Pad3): track 36.8 -> 0.00 mm
- net Net-(SW101-Pad2): track 36.8 -> 0.00 mm
- net Net-(U103-PD7): track 0.00 -> 36.8 mm
- net Net-(SW101-Pad1): track 36.8 -> 0.00 mm
- net Net-(U103-PD4): track 0.00 -> 26.6 mm
- net Net-(SW101-Pad4): track 26.6 -> 0.00 mm
- net /MIDI_IN: track 128.7 -> 106.8 mm, vias 6 -> 3
- net Net-(J110-Pin_3): track 0.00 -> 11.5 mm
- net -VDC: track 89.6 -> 97.5 mm
- net +VDC: track 80.2 -> 87.6 mm
- net Net-(J110-Pin_1): track 0.00 -> 6.69 mm
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Other:
- net class Default removed
- board text added: "2k2"
- board text added: "~ 0 ~"
- board text removed: "~~ 0 ~~"
