File: Lights/Lights_back.kicad_pcb (KiCad board)
At the start: 2 copper layers, 102.5 x 200 mm, 127 parts, among them J101 chain_in, J102 chain_out, J103 Input1, J104 Input2, J105 Input3, J106 THRU, J107 OUT, J108 IN, J109 EuroPower, J110 ExternalPower, J111 Programming, J112 chain_power, J401 Light, J701 Light, J801 Light, Q401 PN2222A, Q402 IRF540N, Q701 PN2222A, Q702 IRF540N, Q801 PN2222A, Q802 IRF540N, SW101 MIDI_settings, U101 L7805, U102 L7805, U103 ATmega328P-PU, U201 TL074, U301 74LS04, U302 6N138, U401 6N138, U501 TL074, U601 TL074, U701 6N138, U801 6N138, Y101 16MHz

Commit message: Split PCB
Parts:
- removed the G*** at (49.2, 112.7)
- removed the G*** at (49.2, 53.1)
- removed the G*** at (24.6, 111.7)
- removed the G*** at (24.6, 52.1)
- removed the G*** at (36.7, 25.8)
- removed the G*** at (24.6, 81.9)
- removed the G*** at (38.1, 173.5)
- removed the G*** at (49.2, 82.9)
- removed H101, H108: Mounting_Holes, Kosmo_panel:Kosmo_Panel_Dual_Mounting_Holes
- removed H102: Gain1, Kosmo_panel:Kosmo_Pot_Hole
- removed H103: Gain2, Kosmo_panel:Kosmo_Pot_Hole
- removed H104: Gain3, Kosmo_panel:Kosmo_Pot_Hole
- removed H105: Input1, Kosmo_panel:Kosmo_Jack_Hole
- removed H106: Input2, Kosmo_panel:Kosmo_Jack_Hole
- removed H107: Input3, Kosmo_panel:Kosmo_Jack_Hole
- removed H109: Offset1, Kosmo_panel:Kosmo_Pot_Hole
- removed H110: Offset2, Kosmo_panel:Kosmo_Pot_Hole
- removed H111: Offset3, Kosmo_panel:Kosmo_Pot_Hole
- removed H112: IN, MountingHole:MountingHole_6mm_Pad
- removed H113: THRU, MountingHole:MountingHole_6mm_Pad
- removed H114: OUT, MountingHole:MountingHole_6mm_Pad
- removed H115, H116: Led_Hole, Kosmo_panel:Kosmo_LED_Hole
- removed LOGO101: telec, logo:telec-8
- added G***: LOGO, logo:sloth-4, B.Cu at (86.3, 124.4)
- added G***: LOGO, logo:ski-4, F.Cu at (86.6, 88.0)
Routing:
- net GND: track 234.8 -> 254.1 mm, vias 18 -> 19
Other:
- board size 102.5 x 200 mm -> 50 x 174 mm
- board text added: "&"
- board text added: "Light control"
- board text added: "MIDI"
- board text added: "PWM"
- board text added: "feb 2020"
- board text added: "telec"
- board text removed: "12"
- board text removed: "D"
- board text removed: "I"
- board text removed: "IN"
- board text removed: "Light Control"
- board text removed: "M"
- board text removed: "OUT"
- board text removed: "THRU"
