File: Lights/Lights.sch (KiCad schematic (older format))
At the start: 45 parts, among them J101 chain_in, J102 chain_out, J103 Input1, J104 Input1, J105 Input1, J106 THRU, J107 OUT, J108 IN, J109 EuroPower, J110 ExternalPower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

Commit message: Finished schematic and routing
Parts:
- removed C? (x3): 1u, Capacitor_SMD:C_0805_2012Metric, symbol Device:C
- removed C?: 100n, Capacitor_SMD:C_0805_2012Metric, symbol Device:C
- removed C? (x2): 10p, Capacitor_SMD:C_0603_1608Metric, symbol Device:C_Small
- removed Y?: X322516MLB4SI, Crystal:Crystal_SMD_3225-4Pin_3.2x2.5mm, symbol Device:Crystal_GND24_Small
- added C105: 100n, Capacitor_THT:C_Disc_D7.0mm_W2.5mm_P5.00mm, symbol Device:C
- added C106, C108, C109: 1u, Capacitor_THT:CP_Radial_D5.0mm_P2.50mm, symbol Device:C
- added C107: 10u, Capacitor_THT:CP_Radial_D5.0mm_P2.50mm, symbol Device:C
- added D103: LED, LED_THT:LED_D3.0mm_FlatTop, symbol Device:LED
- added J112: chain_power, Connector_PinHeader_2.54mm:PinHeader_1x04_P2.54mm_Vertical, symbol Connector:Conn_01x04_Male
- added R101, R102: 1K, Resistor_THT:R_Axial_DIN0204_L3.6mm_D1.6mm_P2.54mm_Vertical, symbol Device:R
- added Y1: 16MHz, Crystal:Resonator-3Pin_W6.0mm_H3.0mm, symbol Device:Resonator_Small
- C103: renamed from C?; footprint Capacitor_SMD:C_0805_2012Metric -> Capacitor_THT:CP_Radial_D5.0mm_P2.50mm; LCSC C28323 -> (none)
- D102: renamed from D?; footprint (none) -> LED_THT:LED_D3.0mm_FlatTop
- H112, H113, H114: footprint Kosmo_panel:Kosmo_Jack_Hole -> MountingHole:MountingHole_6mm_Pad
- J104: value Input1 -> Input2
- J105: value Input1 -> Input3
- J111: renamed from J?; footprint telec:Pogo_02x03_2.54mm -> Connector_IDC:IDC-Header_2x03_P2.54mm_Vertical
- R103: renamed from R?; footprint Resistor_SMD:R_0805_2012Metric -> Resistor_THT:R_Axial_DIN0204_L3.6mm_D1.6mm_P2.54mm_Vertical; LCSC C17560 -> (none)
- gave numbers to parts that had none: 4
Connections:
- net VCC is gone; now on net +5V: J111.2 (Pin_2), R103.1
- net +12V: now also R101.1, R102.1
- net +5V: now also C106.1
- net +5VP: now also C109.1, J112.4 (Pin_4)
- net +VDC: now also C107.1, J112.1 (Pin_1)
- net -VDC: now also C107.2, C108.2, C109.2, J112.2 (Pin_2)
- net ADC1: now also U103.25 (PC2)
- net ADC2: now also U103.24 (PC1)
- net ADC3: now also U103.23 (PC0)
- net GND: now also C105.1, C106.2, Y1.2
- net GNDPWR: now also C108.1, J112.3 (Pin_3)
- net MIDI_IN: now also U103.2 (PD0), D103.1 (K)
- net MIDI_OUT: now also D102.1 (K), U103.3 (PD1)
- net PWM1: now also U103.15 (PB1)
- net PWM2: now also U103.16 (PB2)
- net PWM3: now also U103.5 (PD3)
- net ~RESET: now also C105.2
- net at U103.10 (XTAL2/PB7): now also Y1.1
- net at U103.9 (XTAL1/PB6): now also Y1.3
- net at D102.2 (A): now also R101.2
- new net: D103.2 (A), R102.2
- no-connect marks 1 -> 16
Other:
- moved on the sheet: C101, C102, C103, C104, D101, D102, J101, J102, J103, J104, J105, J106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

Commit message: Finished artwork
Parts:
- added SW101: MIDI_settings, Button_Switch_THT:SW_DIP_SPSTx04_Slide_9.78x12.34mm_W7.62mm_P2.54mm, symbol Switch:SW_DIP_x04
- renumbered Y1 to Y101
Connections:
- net GND: now also SW101.5, SW101.6, SW101.7, SW101.8
- net at U103.11 (PD5): now also SW101.3
- net at U103.12 (PD6): now also SW101.2
- net at U103.13 (PD7): now also SW101.1
- net at U103.6 (PD4): now also SW101.4
- no-connect marks 16 -> 12
Changed lines of the file:
@@
 $EndComp
 $Comp
-L Device:Resonator_Small Y1
+L Device:Resonator_Small Y101
 U 1 1 60986D66
 P 6450 3700
-F 0 "Y1" V 6775 3650 50  0000 C CNN
+F 0 "Y101" V 6775 3650 50  0000 C CNN
 F 1 "16MHz" V 6684 3650 50  0000 C CNN
 F 2 "Crystal:Resonator-3Pin_W6.0mm_H3.0mm" H 6425 3700 50  0001 C CNN
@@
 NoConn ~ 5950 4450
 NoConn ~ 5950 4950
-NoConn ~ 5950 5150
-NoConn ~ 5950 5250
-NoConn ~ 5950 5350
-NoConn ~ 5950 5450
 $Comp
 L power:+12V #PWR0141
@@
 Wire Wire Line
 	8800 1150 9300 1150
+$Comp
+L Switch:SW_DIP_x04 SW101
+U 1 1 60D7D4D8
+P 6800 5250
+F 0 "SW101" H 6800 4883 50  0000 C CNN
+F 1 "MIDI_settings" H 6800 4974 50  0000 C CNN
+F 2 "Button_Switch_THT:SW_DIP_SPSTx04_Slide_9.78x12.34mm_W7.62mm_P2.54mm" H 6800 5250 50  0001 C CNN
+F 3 "~" H 6800 5250 50  0001 C CNN
+	1    6800 5250
+	1    0    0    1
+$EndComp
+$Comp
+L power:GND #PWR0168
+U 1 1 60D80B9E
+P 7150 5550
+AR Path="/60D80B9E" Ref="#PWR0168"  Part="1"
+AR Path="/5F345A0C/60D80B9E" Ref="#PWR?"  Part="1"
+F 0 "#PWR0168" H 7150 5300 50  0001 C CNN
+F 1 "GND" H 7155 5377 50  0000 C CNN
+F 2 "" H 7150 5550 50  0001 C CNN
+F 3 "" H 7150 5550 50  0001 C CNN
+	1    7150 5550
+	1    0    0    -1
+$EndComp
+Wire Wire Line
+	7150 5550 7150 5450
+Wire Wire Line
+	7150 5150 7100 5150
+Wire Wire Line
+	7100 5250 7150 5250
+Connection ~ 7150 5250
+Wire Wire Line
+	7150 5250 7150 5150
+Wire Wire Line
+	7100 5350 7150 5350
+Connection ~ 7150 5350
+Wire Wire Line
+	7150 5350 7150 5250
+Wire Wire Line
+	7100 5450 7150 5450
+Connection ~ 7150 5450
+Wire Wire Line
+	7150 5450 7150 5350
+Wire Wire Line
+	6500 5450 5950 5450
+Wire Wire Line
+	6500 5350 5950 5350
+Wire Wire Line
+	5950 5250 6500 5250
+Wire Wire Line
+	6500 5150 5950 5150
 $EndSCHEMATC

Commit message: Small fixes+firmware
Parts:
- C103, C106, C107, C108, C109: symbol Device:C -> Device:CP
- D101: symbol Device:D_Bridge_+-AA -> Device:D_Bridge_+A-A
Connections:
- net +12V: no longer R101.1, R102.1
- net +5V: now also R101.1, R102.1
- net -VDC: now also D101.3 (-); no longer D101.2 (-)
- net at J110.3 (Pin_3): now also D101.4 (~~); no longer D101.3 (~~)
- net at J110.1 (Pin_1): now also D101.2 (~~); no longer D101.4 (~~)
Changed lines of the file:
@@
 $EndSheet
 $Comp
-L Device:D_Bridge_+-AA D101
+L Device:D_Bridge_+A-A D101
 U 1 1 60633939
 P 5550 1150
@@
 $EndComp
 $Comp
-L Device:C C103
+L Device:CP C103
 U 1 1 607B2A8D
 P 2750 1200
@@
 Connection ~ 2750 1050
 $Comp
-L Device:C C106
+L Device:CP C106
 U 1 1 60A02392
 P 3650 1200
@@
 Connection ~ 3650 1050
 $Comp
-L Device:C C108
+L Device:CP C108
 U 1 1 60A03514
 P 7150 1200
@@
 $EndComp
 $Comp
-L Device:C C109
+L Device:CP C109
 U 1 1 60A03CC6
 P 8000 1200
@@
 $EndComp
 $Comp
-L Device:C C107
+L Device:CP C107
 U 1 1 60A2A522
 P 6300 1200
@@
 NoConn ~ 5950 4950
 $Comp
-L power:+12V #PWR0141
-U 1 1 60BD4C9C
-P 3500 6850
-F 0 "#PWR0141" H 3500 6700 50  0001 C CNN
-F 1 "+12V" H 3515 7023 50  0000 C CNN
-F 2 "" H 3500 6850 50  0001 C CNN
-F 3 "" H 3500 6850 50  0001 C CNN
-	1    3500 6850
-	1    0    0    -1
-$EndComp
-$Comp
-L power:+12V #PWR0142
-U 1 1 60BD5F5C
-P 3850 6850
-F 0 "#PWR0142" H 3850 6700 50  0001 C CNN
-F 1 "+12V" H 3865 7023 50  0000 C CNN
-F 2 "" H 3850 6850 50  0001 C CNN
-F 3 "" H 3850 6850 50  0001 C CNN
-	1    3850 6850
-	1    0    0    -1
-$EndComp
-$Comp
 L Connector:Conn_01x04_Male J112
 U 1 1 60C47075
@@
 Wire Wire Line
 	6500 5150 5950 5150
+$Comp
+L power:+5V #PWR?
+U 1 1 6044F4BA
+P 3500 6850
+F 0 "#PWR?" H 3500 6700 50  0001 C CNN
+F 1 "+5V" H 3515 7023 50  0000 C CNN
+F 2 "" H 3500 6850 50  0001 C CNN
+F 3 "" H 3500 6850 50  0001 C CNN
+	1    3500 6850
+	1    0    0    -1
+$EndComp
+$Comp
+L power:+5V #PWR?
+U 1 1 6044FC04
+P 3850 6850
+F 0 "#PWR?" H 3850 6700 50  0001 C CNN
+F 1 "+5V" H 3865 7023 50  0000 C CNN
+F 2 "" H 3850 6850 50  0001 C CNN
+F 3 "" H 3850 6850 50  0001 C CNN
+	1    3850 6850
+	1    0    0    -1
+$EndComp
 $EndSCHEMATC
