File: Lights/Normalize.sch (KiCad schematic (older format))
At the start: 13 parts, among them U201 TL074

Commit message: Finished schematic and routing
Parts:
- D201, D202: footprint Diode_THT:D_DO-35_SOD27_P7.62mm_Horizontal -> Diode_THT:D_DO-35_SOD27_P2.54mm_Vertical_KathodeUp
- R201, R202, R203, R204, R205, R207, R208: footprint Resistor_THT:R_Axial_DIN0204_L3.6mm_D1.6mm_P7.62mm_Horizontal -> Resistor_THT:R_Axial_DIN0204_L3.6mm_D1.6mm_P2.54mm_Vertical
- U201: footprint Package_DIP:DIP-16_W7.62mm_LongPads -> Package_DIP:DIP-14_W7.62mm_LongPads
Changed lines of the file:
@@
 $Descr A4 11693 8268
 encoding utf-8
-Sheet 2 8
+Sheet 5 8
 Title ""
 Date ""
@@
 F 0 "U601" H 2150 2500 50  0000 C CNN
 F 1 "TL074" H 2200 2400 50  0000 C CNN
-F 2 "Package_DIP:DIP-16_W7.62mm_LongPads" H 2000 2350 50  0001 C CNN
+F 2 "Package_DIP:DIP-14_W7.62mm_LongPads" H 2000 2350 50  0001 C CNN
 F 3 "http://www.ti.com/lit/ds/symlink/tl071.pdf" H 2100 2450 50  0001 C CNN
 	1    2050 2250
@@
 F 0 "U601" H 4550 3017 50  0000 C CNN
 F 1 "TL074" H 4550 2926 50  0000 C CNN
-F 2 "Package_DIP:DIP-16_W7.62mm_LongPads" H 4500 2750 50  0001 C CNN
+F 2 "Package_DIP:DIP-14_W7.62mm_LongPads" H 4500 2750 50  0001 C CNN
 F 3 "http://www.ti.com/lit/ds/symlink/tl071.pdf" H 4600 2850 50  0001 C CNN
 	3    4550 2650
@@
 F 0 "U601" H 3400 3117 50  0000 C CNN
 F 1 "TL074" H 3400 3026 50  0000 C CNN
-F 2 "Package_DIP:DIP-16_W7.62mm_LongPads" H 3350 2850 50  0001 C CNN
+F 2 "Package_DIP:DIP-14_W7.62mm_LongPads" H 3350 2850 50  0001 C CNN
 F 3 "http://www.ti.com/lit/ds/symlink/tl071.pdf" H 3450 2950 50  0001 C CNN
 	2    3400 2750
@@
 F 0 "U601" H 2150 3150 50  0000 C CNN
 F 1 "TL074" H 2200 3050 50  0000 C CNN
-F 2 "Package_DIP:DIP-16_W7.62mm_LongPads" H 2000 3000 50  0001 C CNN
+F 2 "Package_DIP:DIP-14_W7.62mm_LongPads" H 2000 3000 50  0001 C CNN
 F 3 "http://www.ti.com/lit/ds/symlink/tl071.pdf" H 2100 3100 50  0001 C CNN
 	4    2050 2900
@@
 F 0 "U601" H 1408 1146 50  0000 L CNN
 F 1 "TL074" H 1408 1055 50  0000 L CNN
-F 2 "Package_DIP:DIP-16_W7.62mm_LongPads" H 1400 1200 50  0001 C CNN
+F 2 "Package_DIP:DIP-14_W7.62mm_LongPads" H 1400 1200 50  0001 C CNN
 F 3 "http://www.ti.com/lit/ds/symlink/tl071.pdf" H 1500 1300 50  0001 C CNN
 	5    1450 1100
@@
 F 0 "R602" V 1950 3100 50  0000 L CNN
 F 1 "100k" V 2050 3100 50  0000 L CNN
-F 2 "Resistor_THT:R_Axial_DIN0204_L3.6mm_D1.6mm_P7.62mm_Horizontal" V 1980 3200 50  0001 C CNN
+F 2 "Resistor_THT:R_Axial_DIN0204_L3.6mm_D1.6mm_P2.54mm_Vertical" V 1980 3200 50  0001 C CNN
 F 3 "~" H 2050 3200 50  0001 C CNN
 	1    2050 3200
@@
 F 0 "R601" V 1350 3100 50  0000 L CNN
 F 1 "100k" V 1450 3100 50  0000 L CNN
-F 2 "Resistor_THT:R_Axial_DIN0204_L3.6mm_D1.6mm_P7.62mm_Horizontal" V 1380 3200 50  0001 C CNN
+F 2 "Resistor_THT:R_Axial_DIN0204_L3.6mm_D1.6mm_P2.54mm_Vertical" V 1380 3200 50  0001 C CNN
 F 3 "~" H 1450 3200 50  0001 C CNN
 	1    1450 3200
@@
 F 0 "R603" V 2900 3200 50  0000 L CNN
 F 1 "100k" V 3000 3200 50  0000 L CNN
-F 2 "Resistor_THT:R_Axial_DIN0204_L3.6mm_D1.6mm_P7.62mm_Horizontal" V 2930 3300 50  0001 C CNN
+F 2 "Resistor_THT:R_Axial_DIN0204_L3.6mm_D1.6mm_P2.54mm_Vertical" V 2930 3300 50  0001 C CNN
 F 3 "~" H 3000 3300 50  0001 C CNN
 	1    3000 3300
@@
 F 0 "R604" V 3300 2950 50  0000 L CNN
 F 1 "200k" V 3400 2950 50  0000 L CNN
-F 2 "Resistor_THT:R_Axial_DIN0204_L3.6mm_D1.6mm_P7.62mm_Horizontal" V 3330 3050 50  0001 C CNN
+F 2 "Resistor_THT:R_Axial_DIN0204_L3.6mm_D1.6mm_P2.54mm_Vertical" V 3330 3050 50  0001 C CNN
 F 3 "~" H 3400 3050 50  0001 C CNN
 	1    3400 3050
@@
 F 0 "R607" V 4400 2900 50  0000 L CNN
 F 1 "100k" V 4500 2900 50  0000 L CNN
-F 2 "Resistor_THT:R_Axial_DIN0204_L3.6mm_D1.6mm_P7.62mm_Horizontal" V 4430 3000 50  0001 C CNN
+F 2 "Resistor_THT:R_Axial_DIN0204_L3.6mm_D1.6mm_P2.54mm_Vertical" V 4430 3000 50  0001 C CNN
 F 3 "~" H 4500 3000 50  0001 C CNN
 	1    4500 3000
@@
 F 0 "R608" V 5100 2550 50  0000 L CNN
 F 1 "1k" V 5200 2600 50  0000 L CNN
-F 2 "Resistor_THT:R_Axial_DIN0204_L3.6mm_D1.6mm_P7.62mm_Horizontal" V 5130 2650 50  0001 C CNN
+F 2 "Resistor_THT:R_Axial_DIN0204_L3.6mm_D1.6mm_P2.54mm_Vertical" V 5130 2650 50  0001 C CNN
 F 3 "~" H 5200 2650 50  0001 C CNN
 	1    5200 2650
@@
 F 0 "D601" H 5450 2616 50  0000 C CNN
 F 1 "1N4148" H 5450 2525 50  0000 C CNN
-F 2 "Diode_THT:D_DO-35_SOD27_P7.62mm_Horizontal" H 5450 2225 50  0001 C CNN
+F 2 "Diode_THT:D_DO-35_SOD27_P2.54mm_Vertical_KathodeUp" H 5450 2225 50  0001 C CNN
 F 3 "https://assets.nexperia.com/documents/data-sheet/1N4148_1N4448.pdf" H 5450 2400 50  0001 C CNN
 	1    5450 2400
@@
 F 0 "D602" H 5450 3116 50  0000 C CNN
 F 1 "1N4148" H 5450 3025 50  0000 C CNN
-F 2 "Diode_THT:D_DO-35_SOD27_P7.62mm_Horizontal" H 5450 2725 50  0001 C CNN
+F 2 "Diode_THT:D_DO-35_SOD27_P2.54mm_Vertical_KathodeUp" H 5450 2725 50  0001 C CNN
 F 3 "https://assets.nexperia.com/documents/data-sheet/1N4148_1N4448.pdf" H 5450 2900 50  0001 C CNN
 	1    5450 2900
@@
 F 0 "R605" V 3550 1800 50  0000 L CNN
 F 1 "100k" V 3650 1800 50  0000 L CNN
-F 2 "Resistor_THT:R_Axial_DIN0204_L3.6mm_D1.6mm_P7.62mm_Horizontal" V 3580 1900 50  0001 C CNN
+F 2 "Resistor_THT:R_Axial_DIN0204_L3.6mm_D1.6mm_P2.54mm_Vertical" V 3580 1900 50  0001 C CNN
 F 3 "~" H 3650 1900 50  0001 C CNN
 	1    3650 1900

Commit message: Small fixes+firmware
Changed lines of the file:
@@
 AR Path="/606D25B5/6054FDCA" Ref="U501"  Part="1"
 AR Path="/606D67CF/6054FDCA" Ref="U601"  Part="1"
-F 0 "U601" H 2150 2500 50  0000 C CNN
+F 0 "U201" H 2150 2500 50  0000 C CNN
 F 1 "TL074" H 2200 2400 50  0000 C CNN
 F 2 "Package_DIP:DIP-14_W7.62mm_LongPads" H 2000 2350 50  0001 C CNN
@@
 AR Path="/606D25B5/6054FDD0" Ref="U501"  Part="3"
 AR Path="/606D67CF/6054FDD0" Ref="U601"  Part="3"
-F 0 "U601" H 4550 3017 50  0000 C CNN
+F 0 "U201" H 4550 3017 50  0000 C CNN
 F 1 "TL074" H 4550 2926 50  0000 C CNN
 F 2 "Package_DIP:DIP-14_W7.62mm_LongPads" H 4500 2750 50  0001 C CNN
@@
 AR Path="/606D25B5/6054FDD6" Ref="U501"  Part="2"
 AR Path="/606D67CF/6054FDD6" Ref="U601"  Part="2"
-F 0 "U601" H 3400 3117 50  0000 C CNN
+F 0 "U201" H 3400 3117 50  0000 C CNN
 F 1 "TL074" H 3400 3026 50  0000 C CNN
 F 2 "Package_DIP:DIP-14_W7.62mm_LongPads" H 3350 2850 50  0001 C CNN
@@
 AR Path="/606D25B5/6054FDDC" Ref="U501"  Part="4"
 AR Path="/606D67CF/6054FDDC" Ref="U601"  Part="4"
-F 0 "U601" H 2150 3150 50  0000 C CNN
+F 0 "U201" H 2150 3150 50  0000 C CNN
 F 1 "TL074" H 2200 3050 50  0000 C CNN
 F 2 "Package_DIP:DIP-14_W7.62mm_LongPads" H 2000 3000 50  0001 C CNN
@@
 AR Path="/606D25B5/6054FDE2" Ref="U501"  Part="5"
 AR Path="/606D67CF/6054FDE2" Ref="U601"  Part="5"
-F 0 "U601" H 1408 1146 50  0000 L CNN
+F 0 "U201" H 1408 1146 50  0000 L CNN
 F 1 "TL074" H 1408 1055 50  0000 L CNN
 F 2 "Package_DIP:DIP-14_W7.62mm_LongPads" H 1400 1200 50  0001 C CNN
@@
 AR Path="/606D25B5/6054FDE8" Ref="R502"  Part="1"
 AR Path="/606D67CF/6054FDE8" Ref="R602"  Part="1"
-F 0 "R602" V 1950 3100 50  0000 L CNN
+F 0 "R202" V 1950 3100 50  0000 L CNN
 F 1 "100k" V 2050 3100 50  0000 L CNN
 F 2 "Resistor_THT:R_Axial_DIN0204_L3.6mm_D1.6mm_P2.54mm_Vertical" V 1980 3200 50  0001 C CNN
@@
 AR Path="/606D25B5/6054FDF3" Ref="#PWR0503"  Part="1"
 AR Path="/606D67CF/6054FDF3" Ref="#PWR0603"  Part="1"
-F 0 "#PWR0603" H 1750 2550 50  0001 C CNN
+F 0 "#PWR0203" H 1750 2550 50  0001 C CNN
 F 1 "GND" H 1755 2627 50  0000 C CNN
 F 2 "" H 1750 2800 50  0001 C CNN
@@
 AR Path="/606D25B5/6054FDF9" Ref="R501"  Part="1"
 AR Path="/606D67CF/6054FDF9" Ref="R601"  Part="1"
-F 0 "R601" V 1350 3100 50  0000 L CNN
+F 0 "R201" V 1350 3100 50  0000 L CNN
 F 1 "100k" V 1450 3100 50  0000 L CNN
 F 2 "Resistor_THT:R_Axial_DIN0204_L3.6mm_D1.6mm_P2.54mm_Vertical" V 1380 3200 50  0001 C CNN
@@
 AR Path="/606D25B5/6054FE0A" Ref="RV501"  Part="1"
 AR Path="/606D67CF/6054FE0A" Ref="RV601"  Part="1"
-F 0 "RV601" H 2681 2696 50  0000 R CNN
+F 0 "RV201" H 2681 2696 50  0000 R CNN
 F 1 "100k" H 2681 2605 50  0000 R CNN
 F 2 "Connector_PinHeader_2.54mm:PinHeader_1x03_P2.54mm_Vertical" H 2750 2650 50  0001 C CNN
@@
 AR Path="/606D25B5/6054FE19" Ref="R503"  Part="1"
 AR Path="/606D67CF/6054FE19" Ref="R603"  Part="1"
-F 0 "R603" V 2900 3200 50  0000 L CNN
+F 0 "R203" V 2900 3200 50  0000 L CNN
 F 1 "100k" V 3000 3200 50  0000 L CNN
 F 2 "Resistor_THT:R_Axial_DIN0204_L3.6mm_D1.6mm_P2.54mm_Vertical" V 2930 3300 50  0001 C CNN
@@
 AR Path="/606D25B5/6054FE1F" Ref="R504"  Part="1"
 AR Path="/606D67CF/6054FE1F" Ref="R604"  Part="1"
-F 0 "R604" V 3300 2950 50  0000 L CNN
+F 0 "R204" V 3300 2950 50  0000 L CNN
 F 1 "200k" V 3400 2950 50  0000 L CNN
 F 2 "Resistor_THT:R_Axial_DIN0204_L3.6mm_D1.6mm_P2.54mm_Vertical" V 3330 3050 50  0001 C CNN
@@
 AR Path="/606D25B5/6054FE25" Ref="#PWR0504"  Part="1"
 AR Path="/606D67CF/6054FE25" Ref="#PWR0604"  Part="1"
-F 0 "#PWR0604" H 3000 3200 50  0001 C CNN
+F 0 "#PWR0204" H 3000 3200 50  0001 C CNN
 F 1 "GND" H 3005 3277 50  0000 C CNN
 F 2 "" H 3000 3450 50  0001 C CNN
@@
 AR Path="/606D25B5/6054FE34" Ref="RV502"  Part="1"
 AR Path="/606D67CF/6054FE34" Ref="RV602"  Part="1"
-F 0 "RV602" H 3781 2146 50  0000 R CNN
+F 0 "RV202" H 3781 2146 50  0000 R CNN
 F 1 "100k" H 3781 2055 50  0000 R CNN
 F 2 "Connector_PinHeader_2.54mm:PinHeader_1x03_P2.54mm_Vertical" H 3850 2100 50  0001 C CNN
@@
 AR Path="/606D25B5/6054FE3A" Ref="#PWR0506"  Part="1"
 AR Path="/606D67CF/6054FE3A" Ref="#PWR0606"  Part="1"
-F 0 "#PWR0606" H 3850 2000 50  0001 C CNN
+F 0 "#PWR0206" H 3850 2000 50  0001 C CNN
 F 1 "GND" H 3855 2077 50  0000 C CNN
 F 2 "" H 3850 2250 50  0001 C CNN
@@
 AR Path="/606D25B5/6054FE43" Ref="R506"  Part="1"
 AR Path="/606D67CF/6054FE43" Ref="R606"  Part="1"
-F 0 "R606" V 3900 2650 50  0000 L CNN
+F 0 "R206" V 3900 2650 50  0000 L CNN
 F 1 "100k" V 4000 2650 50  0000 L CNN
 F 2 "Resistor_THT:R_Axial_DIN0204_L3.6mm_D1.6mm_P7.62mm_Horizontal" V 3930 2750 50  0001 C CNN
@@
 AR Path="/606D25B5/6054FE49" Ref="R507"  Part="1"
 AR Path="/606D67CF/6054FE49" Ref="R607"  Part="1"
-F 0 "R607" V 4400 2900 50  0000 L CNN
+F 0 "R207" V 4400 2900 50  0000 L CNN
 F 1 "100k" V 4500 2900 50  0000 L CNN
 F 2 "Resistor_THT:R_Axial_DIN0204_L3.6mm_D1.6mm_P2.54mm_Vertical" V 4430 3000 50  0001 C CNN
@@
 AR Path="/606D25B5/6054FE59" Ref="R508"  Part="1"
 AR Path="/606D67CF/6054FE59" Ref="R608"  Part="1"
-F 0 "R608" V 5100 2550 50  0000 L CNN
+F 0 "R208" V 5100 2550 50  0000 L CNN
 F 1 "1k" V 5200 2600 50  0000 L CNN
 F 2 "Resistor_THT:R_Axial_DIN0204_L3.6mm_D1.6mm_P2.54mm_Vertical" V 5130 2650 50  0001 C CNN
@@
 AR Path="/606D25B5/6054FE5F" Ref="D501"  Part="1"
 AR Path="/606D67CF/6054FE5F" Ref="D601"  Part="1"
-F 0 "D601" H 5450 2616 50  0000 C CNN
+F 0 "D201" H 5450 2616 50  0000 C CNN
 F 1 "1N4148" H 5450 2525 50  0000 C CNN
 F 2 "Diode_THT:D_DO-35_SOD27_P2.54mm_Vertical_KathodeUp" H 5450 2225 50  0001 C CNN
@@
 AR Path="/606D25B5/6054FE65" Ref="D502"  Part="1"
 AR Path="/606D67CF/6054FE65" Ref="D602"  Part="1"
-F 0 "D602" H 5450 3116 50  0000 C CNN
+F 0 "D202" H 5450 3116 50  0000 C CNN
 F 1 "1N4148" H 5450 3025 50  0000 C CNN
 F 2 "Diode_THT:D_DO-35_SOD27_P2.54mm_Vertical_KathodeUp" H 5450 2725 50  0001 C CNN
@@
 AR Path="/606D25B5/6054FE6B" Ref="#PWR0507"  Part="1"
 AR Path="/606D67CF/6054FE6B" Ref="#PWR0607"  Part="1"
-F 0 "#PWR0607" H 5450 2100 50  0001 C CNN
+F 0 "#PWR0207" H 5450 2100 50  0001 C CNN
 F 1 "+5V" H 5465 2423 50  0000 C CNN
 F 2 "" H 5450 2250 50  0001 C CNN
@@
 AR Path="/606D25B5/6054FE71" Ref="#PWR0508"  Part="1"
 AR Path="/606D67CF/6054FE71" Ref="#PWR0608"  Part="1"
-F 0 "#PWR0608" H 5450 2800 50  0001 C CNN
+F 0 "#PWR0208" H 5450 2800 50  0001 C CNN
 F 1 "GND" H 5455 2877 50  0000 C CNN
 F 2 "" H 5450 3050 50  0001 C CNN
@@
 AR Path="/606D25B5/6054FE7F" Ref="R505"  Part="1"
 AR Path="/606D67CF/6054FE7F" Ref="R605"  Part="1"
-F 0 "R605" V 3550 1800 50  0000 L CNN
+F 0 "R205" V 3550 1800 50  0000 L CNN
 F 1 "100k" V 3650 1800 50  0000 L CNN
 F 2 "Resistor_THT:R_Axial_DIN0204_L3.6mm_D1.6mm_P2.54mm_Vertical" V 3580 1900 50  0001 C CNN
@@
 AR Path="/606D25B5/6054FE85" Ref="#PWR0502"  Part="1"
 AR Path="/606D67CF/6054FE85" Ref="#PWR0602"  Part="1"
-F 0 "#PWR0602" H 1350 1500 50  0001 C CNN
+F 0 "#PWR0202" H 1350 1500 50  0001 C CNN
 F 1 "-12V" H 1365 1573 50  0000 C CNN
 F 2 "" H 1350 1400 50  0001 C CNN
@@
 AR Path="/606D25B5/6054FE8B" Ref="#PWR0505"  Part="1"
 AR Path="/606D67CF/6054FE8B" Ref="#PWR0605"  Part="1"
-F 0 "#PWR0605" H 3450 1700 50  0001 C CNN
+F 0 "#PWR0205" H 3450 1700 50  0001 C CNN
 F 1 "+12V" H 3465 2023 50  0000 C CNN
 F 2 "" H 3450 1850 50  0001 C CNN
@@
 AR Path="/606D25B5/6054FE91" Ref="#PWR0501"  Part="1"
 AR Path="/606D67CF/6054FE91" Ref="#PWR0601"  Part="1"
-F 0 "#PWR0601" H 1350 650 50  0001 C CNN
+F 0 "#PWR0201" H 1350 650 50  0001 C CNN
 F 1 "+12V" H 1365 973 50  0000 C CNN
 F 2 "" H 1350 800 50  0001 C CNN
